File: 1.hardware/interface.kicad_sch (KiCad schematic)
At the start: 0 parts

Commit message: 중간 저장
Other:
- note added: "CAN"
- note added: "I2C"
- note added: "UART"
- note added: "USB"
Changed lines of the file:
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@@
 	(generator_version "9.0")
 	(paper "A4")
+	(text "I2C"
+		(exclude_from_sim no)
+		(at 58.674 71.628 0)
+		(effects
+			(font
+				(size 1.27 1.27)
+			)
+		)
+	)
+	(text "CAN"
+		(exclude_from_sim no)
+		(at 58.674 73.66 0)
+		(effects
+			(font
+				(size 1.27 1.27)
+			)
+		)
+	)
+	(text "UART"
+		(exclude_from_sim no)
+		(at 58.674 75.692 0)
+		(effects
+			(font
+				(size 1.27 1.27)
+			)
+		)
+	)
+	(text "USB"
+		(exclude_from_sim no)
+		(at 58.674 69.596 0)
+		(effects
+			(font
+				(size 1.27 1.27)
+			)
+		)
+	)
 	(global_label "USB_DP"
 		(shape passive)

Commit message: 중간 저장2
Parts:
- added C21, C22: 0.1uF/16V, Capacitor_SMD:C_0402_1005Metric, symbol Device:C_Small_US
- added C23: 2.2uF/6.3V, Capacitor_SMD:C_0603_1608Metric, symbol Device:C_Small_US
- added D4: PRTR5V0U2X, Package_TO_SOT_SMD:SOT-143, symbol Power_Protection:PRTR5V0U2X
- added J7: Connector_USB_C_Receptacle_USB2.0, Connector_USB:USB_C_Receptacle_HRO_TYPE-C-31-M-12, symbol USB-C-USB-2.0-cache:Connector_USB_C_Receptacle_USB2.0
- added J8: uart_comm, symbol Connector_Generic:Conn_01x04
- added R79: 4.7K, symbol Device:R_Small_US
- added R80: NC_4.7K, symbol Device:R_Small_US
- added R81, R82: 4.7K/0.063w, symbol Device:R_Small_US
- added U5: ESP32-C3-WROOM-02, RF_Module:ESP32-C3-WROOM-02, symbol RF_Module:ESP32-C3-WROOM-02
Connections:
- net USB_DM: now also D4.3 (I/O2), J7.A7 (D-), J7.B7 (D-)
- net USB_DP: now also D4.2 (I/O1), J7.A6 (D+), J7.B6 (D+)
- new net: J7.A5 (CC1), J7.B5 (CC2), R79.1, R80.2
- new net 3V3_MCU: C21.1, C22.1, C23.1, R81.1, R82.1, U5.1 (3V3)
- new net GND: C21.2, C22.2, C23.2, D4.1 (GND), J7.A1 (GND), J7.A12 (GND), J7.B1 (GND), J7.B12 (GND), J7.S1 (SHIELD), J8.4 (Pin_4), R79.2, U5.19 (GND), U5.9 (GND)
- new net UART_RX: J8.3 (Pin_3), R82.2
- new net UART_TX: J8.2 (Pin_2), R81.2
- new net VBUS: D4.4 (VCC), J7.A4 (VBUS), J7.A9 (VBUS), J7.B4 (VBUS), J7.B9 (VBUS), R80.1
- no-connect marks 0 -> 2
Other:
- note added: "BLE/WIFI"

Commit message: 중간 저장
Connections:
- no-connect marks 2 -> 3
Changed lines of the file:
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@@
 		(at 49.53 54.61)
+	)
+	(no_connect
+		(at 31.75 87.63)
 	)
 	(wire

Commit message: 중간 저장
Parts:
- added C62: 0.1uF/16V, Capacitor_SMD:C_0402_1005Metric, symbol Device:C_Small_US
- added J1, J12, J13: Conn_01x02, symbol Connector_Generic:Conn_01x02
- added J14: Conn_01x03, symbol Connector_Generic:Conn_01x03
- added LED3: LED_0603_Red_WIFI, PCM_LED_SMD_AKL:LED_0603_1608Metric, symbol PCM_LED_AKL:LED_0603_Red
- added LED4: LED_0603_Blue_BLE, PCM_LED_SMD_AKL:LED_0603_1608Metric, symbol PCM_LED_AKL:LED_0603_Blue
- added LED5: LED_0603_Green_PWR, PCM_LED_SMD_AKL:LED_0603_1608Metric, symbol PCM_LED_AKL:LED_0603_Green
- added R101, R102, R103, R104, R105, R106, R107: 4.7K/0.063w, symbol Device:R_Small_US
- added SW1: Reset_Btn, symbol Switch:SW_Push
- renumbered C21 to C50, C22 to C51, C23 to C52, D4 to D9, J8 to J7, J7 to J8, R81 to R90, R82 to R91, R80 to R92, R79 to R93
Connections:
- net 3V3_MCU: now also J1.2 (Pin_2); no longer U5.1 (3V3)
- net GND: now also U5.15 (IO3), C62.2, J14.3 (Pin_3), LED5.1 (K), SW1.1
- net USB_DM: now also J12.1 (Pin_1)
- net USB_DP: now also J13.2 (Pin_2)
- net FSPICSO: now reaches U5.10 (IO10)
- net at U5.11 (IO20/RXD): now also J14.1 (Pin_1), R103.2
- net at U5.12 (IO21/TXD): now also J14.2 (Pin_2), R104.2
- net at U5.13 (IO18): now also J12.2 (Pin_2)
- net at U5.14 (IO19): now also J13.1 (Pin_1)
- net FSPIQ: now reaches U5.16 (IO2)
- net ESP32_UART_TX: now reaches U5.17 (IO1)
- net ESP32_UART_RX: now reaches U5.18 (IO0)
- net at U5.2 (EN): now also R101.2
- net FSPIHD: now reaches U5.3 (IO4)
- net FSPIWP: now reaches U5.4 (IO5)
- net FSPICLK: now reaches U5.5 (IO6)
- net FSPID: now reaches U5.6 (IO7)
- net at U5.7 (IO8): now also LED4.1 (K)
- net at U5.8 (IO9): now also LED3.1 (K)
- new net: J1.1 (Pin_1), R101.1, R102.1, R103.1, R104.1, R105.1, R106.1, R107.1, U5.1 (3V3)
- new net: C62.1, R107.2, SW1.2
- new net: LED5.2 (A), R102.2
- new net: LED3.2 (A), R105.2
- new net: LED4.2 (A), R106.2
Other:
- moved on the sheet: C50, C51, C52, U5

Commit message: 중간 저장
Parts:
- added J15: I2C_conn, symbol Connector_Generic:Conn_01x02
- added J16: Can_conn, symbol Connector_Generic:Conn_01x02
- J8: value Connector_USB_C_Receptacle_USB2.0 -> USB_C
- R101, R102, R103, R104, R105, R106, R107, R90, R91, R92, R93: footprint (none) -> Resistor_SMD:R_0402_1005Metric
Connections:
- net FSPICLK is gone; now on net ESP32_SPI2_SCK: U5.5 (IO6)
- net FSPICSO is gone; now on net ESP32_SPI2_NSS: U5.10 (IO10)
- net FSPID is gone; now on net ESP32_SPI2_MOSI: U5.6 (IO7)
- net FSPIQ is gone; now on net ESP32_SPI2_MISO: U5.16 (IO2)
Changed lines of the file:
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@@
 	(text "I2C"
 		(exclude_from_sim no)
-		(at 176.276 45.72 0)
+		(at 112.268 19.558 0)
 		(effects
 			(font
@@
 	(text "CAN"
 		(exclude_from_sim no)
-		(at 176.276 47.752 0)
+		(at 112.522 53.848 0)
 		(effects
 			(font
@@
 	(text "USB"
 		(exclude_from_sim no)
-		(at 34.036 18.796 0)
+		(at 30.48 18.796 0)
 		(effects
 			(font
@@
 	(wire
 		(pts
+			(xy 152.4 142.24) (xy 161.29 142.24)
+		)
+		(stroke
+			(width 0)
+			(type default)
+		)
+	)
+	(wire
+		(pts
 			(xy 54.61 113.03) (xy 64.77 113.03)
 		)
@@
 	(wire
 		(pts
+			(xy 152.4 139.7) (xy 161.29 139.7)
+		)
+		(stroke
+			(width 0)
+			(type default)
+		)
+	)
+	(wire
+		(pts
 			(xy 68.58 24.13) (xy 72.39 24.13)
 		)
@@
 	(wire
 		(pts
+			(xy 152.4 144.78) (xy 161.29 144.78)
+		)
+		(stroke
+			(width 0)
+			(type default)
+		)
+	)
+	(wire
+		(pts
 			(xy 76.2 127) (xy 76.2 123.19)
 		)
@@
 	(wire
 		(pts
+			(xy 152.4 147.32) (xy 161.29 147.32)
+		)
+		(stroke
+			(width 0)
+			(type default)
+		)
+	)
+	(wire
+		(pts
 			(xy 22.86 157.48) (xy 27.94 157.48)
 		)
@@
 	(global_label "FSPID"
 		(shape passive)
-		(at 170.18 154.94 180)
+		(at 152.4 147.32 180)
 		(fields_autoplaced yes)
 		(effects
@@
 		)
 		(property "Intersheetrefs" "${INTERSHEET_REFS}"
-			(at 162.8632 154.94 0)
+			(at 145.0832 147.32 0)
 			(effects
 				(font
@@
 	(global_label "FSPICSO"
 		(shape passive)
-		(at 170.18 162.56 180)
+		(at 152.4 139.7 180)
 		(fields_autoplaced yes)
 		(effects
@@
 		)
 		(property "Intersheetrefs" "${INTERSHEET_REFS}"
-			(at 160.3232 162.56 0)
+			(at 142.5432 139.7 0)
 			(effects
 				(font
@@
 	(global_label "ESP32_SPI2_MISO"
 		(shape passive)
-		(at 181.61 146.05 0)
+		(at 161.29 144.78 0)
 		(fields_autoplaced yes)
 		(effects
@@
 		)
 		(property "Intersheetrefs" "${INTERSHEET_REFS}"
-			(at 200.3566 146.05 0)
+			(at 180.0366 144.78 0)
 			(effects
 				(font
@@
 	(global_label "FSPICLK"
 		(shape passive)
-		(at 170.18 152.4 180)
+		(at 152.4 142.24 180)
 		(fields_autoplaced yes)
 		(effects
@@
 		)
 		(property "Intersheetrefs" "${INTERSHEET_REFS}"
-			(at 160.5651 152.4 0)
+			(at 142.7851 142.24 0)
 			(effects
 				(font
@@
 	(global_label "ESP32_SPI2_MOSI"
 		(shape passive)
-		(at 173.99 148.59 0)
+		(at 161.29 147.32 0)
 		(fields_autoplaced yes)
 		(effects
@@
 		)
 		(property "Intersheetrefs" "${INTERSHEET_REFS}"
-			(at 192.7366 148.59 0)
+			(at 180.0366 147.32 0)
 			(effects
 				(font
@@
 	(global_label "ESP32_SPI2_SCK"
 		(shape passive)
-		(at 181.61 143.51 0)
+		(at 161.29 142.24 0)
 		(fields_autoplaced yes)
 		(effects
@@
 		)
 		(property "Intersheetrefs" "${INTERSHEET_REFS}"
-			(at 199.5099 143.51 0)
+			(at 179.1899 142.24 0)
 			(effects
 				(font
@@
 	(global_label "ESP32_SPI2_NSS"
 		(shape passive)
-		(at 181.61 140.97 0)
+		(at 161.29 139.7 0)
 		(fields_autoplaced yes)
 		(effects
@@
 		)
 		(property "Intersheetrefs" "${INTERSHEET_REFS}"
-			(at 199.5099 140.97 0)
+			(at 179.1899 139.7 0)
 			(effects
 				(font
@@
 	(global_label "FSPIQ"
 		(shape passive)
-		(at 168.91 148.59 180)
+		(at 152.4 144.78 180)
 		(fields_autoplaced yes)
 		(effects
@@
 		)
 		(property "Intersheetrefs" "${INTERSHEET_REFS}"
-			(at 161.5327 148.59 0)
+			(at 145.0227 144.78 0)
 			(effects
 				(font
@@
 			)
 		)
-		(property "Footprint" ""
+		(property "Footprint" "Resistor_SMD:R_0402_1005Metric"
 			(at 161.29 118.11 0)
 			(effects
@@
 			)
 		)
-		(property "Footprint" ""
+		(property "Footprint" "Resistor_SMD:R_0402_1005Metric"
 			(at 49.53 82.55 0)
 			(effects
@@
 		(dnp no)
 		(property "Reference" "LED5"
-			(at 22.86 125.7299 90)
+			(at 18.034 124.714 90)
 			(effects
 				(font
@@
 			)
 		)
-		(property "Value" "Connector_USB_C_Receptacle_USB2.0"
+		(property "Value" "USB_C"
 			(at 34.29 21.59 0)
 			(effects
@@
 			)
 		)
-		(property "Footprint" ""
+		(property "Footprint" "Resistor_SMD:R_0402_1005Metric"
 			(at 157.48 118.11 0)
 			(effects
@@
 			)
 		)
-		(property "Footprint" ""
+		(property "Footprint" "Resistor_SMD:R_0402_1005Metric"
 			(at 36.83 82.55 0)
 			(effects
@@
 	)
 	(symbol
+		(lib_id "Connector_Generic:Conn_01x02")
+		(at 109.22 64.77 180)
+		(unit 1)
+		(exclude_from_sim no)
+		(in_bom yes)
+		(on_board yes)
+		(dnp no)
+		(fields_autoplaced yes)
+		(property "Reference" "J16"
+			(at 109.22 55.88 0)
+			(effects
+				(font
+					(size 1.27 1.27)
+				)
+			)
+		)
+		(property "Value" "Can_conn"
+			(at 109.22 58.42 0)
+			(effects
+				(font
+					(size 1.27 1.27)
+				)
+			)
+		)
+		(property "Footprint" ""
+			(at 109.22 64.77 0)
+			(effects
+				(font
+					(size 1.27 1.27)
+				)
+				(hide yes)
+			)
+		)
+		(property "Datasheet" "~"
+			(at 109.22 64.77 0)
+			(effects
+				(font
+					(size 1.27 1.27)
+				)
+				(hide yes)
+			)
+		)
+		(property "Description" "Generic connector, single row, 01x02, script generated (kicad-library-utils/schlib/autogen/connector/)"
+			(at 109.22 64.77 0)
+			(effects
+				(font
+					(size 1.27 1.27)
+				)
+				(hide yes)
+			)
+		)
+		(pin "1"
+		)
+		(pin "2"
+		)
+		(instances
+			(project "bldc_motor_controller"
+				(path "/a25adab6-a8c3-4e0e-8ba9-baac00aaa394/430b6e73-4ab5-4f88-adfd-520e070c0b15"
+					(reference "J16")
+					(unit 1)
+				)
+			)
+		)
+	)
+	(symbol
 		(lib_id "Device:R_Small_US")
 		(at 40.64 123.19 0)
@@
 		)
 		(property "Value" "4.7K/0.063w"
-			(at 47.752 125.222 0)
+			(at 34.036 125.73 0)
 			(effects
 				(font
@@
 			)
 		)
-		(property "Footprint" ""
+		(property "Footprint" "Resistor_SMD:R_0402_1005Metric"
 			(at 40.64 123.19 0)
 			(effects
@@
 		)
 		(property "Value" "4.7K/0.063w"
-			(at 60.198 124.968 0)
+			(at 48.26 125.984 0)
 			(effects
 				(font
@@
 			)
 		)
-		(property "Footprint" ""
+		(property "Footprint" "Resistor_SMD:R_0402_1005Metric"
 			(at 54.61 123.19 0)
 			(effects
@@
 			)
 		)
-		(property "Footprint" ""
+		(property "Footprint" "Resistor_SMD:R_0402_1005Metric"
 			(at 17.78 118.11 0)
 			(effects
@@
 			)
 		)
-		(property "Footprint" ""
+		(property "Footprint" "Resistor_SMD:R_0402_1005Metric"
 			(at 81.28 118.11 0)
 			(effects
@@
 	)
 	(symbol
+		(lib_id "Connector_Generic:Conn_01x02")
+		(at 109.22 30.48 180)
+		(unit 1)
+		(exclude_from_sim no)
+		(in_bom yes)
+		(on_board yes)
+		(dnp no)
+		(fields_autoplaced yes)
+		(property "Reference" "J15"
+			(at 109.22 21.59 0)
+			(effects
+				(font
+					(size 1.27 1.27)
+				)
+			)
+		)
+		(property "Value" "I2C_conn"
+			(at 109.22 24.13 0)
+			(effects
+				(font
+					(size 1.27 1.27)
+				)
+			)
+		)
+		(property "Footprint" ""
+			(at 109.22 30.48 0)
+			(effects
+				(font
+					(size 1.27 1.27)
+				)
+				(hide yes)
+			)
+		)
+		(property "Datasheet" "~"
+			(at 109.22 30.48 0)
+			(effects
+				(font
+					(size 1.27 1.27)
+				)
+				(hide yes)
+			)
+		)
+		(property "Description" "Generic connector, single row, 01x02, script generated (kicad-library-utils/schlib/autogen/connector/)"
+			(at 109.22 30.48 0)
+			(effects
+				(font
+					(size 1.27 1.27)
+				)
+				(hide yes)
+			)
+		)
+		(pin "1"
+		)
+		(pin "2"
+		)
+		(instances
+			(project ""
+				(path "/a25adab6-a8c3-4e0e-8ba9-baac00aaa394/430b6e73-4ab5-4f88-adfd-520e070c0b15"
+					(reference "J15")
+					(unit 1)
+				)
+			)
+		)
+	)
+	(symbol
 		(lib_id "Device:R_Small_US")
 		(at 72.39 34.29 0)
@@
 			)
 		)
-		(property "Footprint" ""
+		(property "Footprint" "Resistor_SMD:R_0402_1005Metric"
 			(at 72.39 34.29 0)
 			(effects
@@
 		)
 		(property "Value" "4.7K/0.063w"
-			(at 70.358 120.396 0)
+			(at 71.12 120.396 0)
 			(effects
 				(font
@@
 			)
 		)
-		(property "Footprint" ""
+		(property "Footprint" "Resistor_SMD:R_0402_1005Metric"
 			(at 64.77 118.11 0)
 			(effects
@@
 			)
 		)
-		(property "Footprint" ""
+		(property "Footprint" "Resistor_SMD:R_0402_1005Metric"
 			(at 72.39 27.94 0)
 			(effects

Commit message: 중간 저장
Parts:
- SW1: value Reset_Btn -> Esp32_Btn
Changed lines of the file:
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@@
 			)
 		)
-		(property "Value" "Reset_Btn"
+		(property "Value" "Esp32_Btn"
 			(at 66.04 130.8099 90)
 			(effects

Commit message: 중간저장
Parts:
- removed J15: I2C_conn, symbol Connector_Generic:Conn_01x02
- added JP1: IF_CAN_END, Jumper:SolderJumper-2_P1.3mm_Open_RoundedPad1.0x1.5mm, symbol Jumper:SolderJumper_2_Open
- added R115: 120R, symbol Device:R_Small_US
- added U11: SN65HVD230, Package_SO:SOIC-8_3.9x4.9mm_P1.27mm, symbol Interface_CAN_LIN:SN65HVD230
Connections:
- net GND: now also U11.2 (GND); no longer D9.1 (GND)
- net CANH: now reaches J16.1 (Pin_1)
- net CANH: now also R115.1, U11.7 (CANH)
- net CANL: now reaches J16.2 (Pin_2)
- net CANL: now also JP1.2 (B), U11.6 (CANL)
- new net: JP1.1 (A), R115.2
- new net +3.3V: U11.3 (VCC)
- new net CAN_RXD: U11.4 (R)
- new net CAN_TXD: U11.1 (D)
- no-connect marks 3 -> 5
Other:
- note removed: "I2C"
- moved on the sheet: J16

Commit message: 중간 저장
Parts:
- added C70, C71: 0.1uF/16V, Capacitor_SMD:C_0402_1005Metric, symbol Device:C_Small_US
- added D11, D12: WS2812B, LED_SMD:LED_WS2812B_PLCC4_5.0x5.0mm_P3.2mm, symbol LED:WS2812B
- added R118: 1k/0.063w, symbol Device:R_Small_US
Connections:
- net GND: now also C70.2, C71.2, D11.3 (VSS), D12.3 (VSS)
- new net: D11.2 (DOUT), D12.4 (DIN)
- new net 5V: C70.1, C71.1, D11.1 (VDD), D12.1 (VDD), R118.1
- new net WS2812_PWM: D11.4 (DIN), R118.2
- no-connect marks 5 -> 6
