File: 1.hardware/mcu.kicad_sch (KiCad schematic)
At the start: 29 parts, among them J1 Debug, J2 usb_pwr, J3 vat_pwr, J4 ext_pwr, SW1 reset_btn, U1 STM32H743BITx, X1 SMD3225-4

Commit message: 중간 저장
Connections:
- net LTDC_B6: no longer names the net of U1.188 (PK5)
- net LTDC_B7: no longer names the net of U1.189 (PK6)
- net LTDC_G6: no longer names the net of U1.13 (PI11)
- net LTDC_G7: no longer names the net of U1.128 (PK2)
- net LTDC_R6: no longer names the net of U1.62 (PB1)
- net LTDC_R7: no longer names the net of U1.65 (PJ0)
Changed lines of the file:
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@@
 	(wire
 		(pts
-			(xy 238.76 195.58) (xy 245.11 195.58)
-		)
-		(stroke
-			(width 0)
-			(type default)
-		)
-	)
-	(wire
-		(pts
 			(xy 257.81 66.04) (xy 262.89 66.04)
 		)
@@
 	(wire
 		(pts
-			(xy 237.49 124.46) (xy 245.11 124.46)
-		)
-		(stroke
-			(width 0)
-			(type default)
-		)
-	)
-	(wire
-		(pts
 			(xy 265.43 71.12) (xy 265.43 66.04)
 		)
@@
 	(wire
 		(pts
-			(xy 237.49 114.3) (xy 245.11 114.3)
-		)
-		(stroke
-			(width 0)
-			(type default)
-		)
-	)
-	(wire
-		(pts
 			(xy 321.31 109.22) (xy 328.93 109.22)
 		)
@@
 	(wire
 		(pts
-			(xy 237.49 106.68) (xy 245.11 106.68)
-		)
-		(stroke
-			(width 0)
-			(type default)
-		)
-	)
-	(wire
-		(pts
 			(xy 293.37 66.04) (xy 290.83 66.04)
 		)
@@
 	(wire
 		(pts
-			(xy 237.49 116.84) (xy 245.11 116.84)
-		)
-		(stroke
-			(width 0)
-			(type default)
-		)
-	)
-	(wire
-		(pts
 			(xy 77.47 175.26) (xy 82.55 175.26)
 		)
@@
 	(wire
 		(pts
-			(xy 321.31 127) (xy 328.93 127)
-		)
-		(stroke
-			(width 0)
-			(type default)
-		)
-	)
-	(wire
-		(pts
 			(xy 238.76 167.64) (xy 245.11 167.64)
 		)
@@
 		)
 	)
-	(global_label "LTDC_R7"
-		(shape passive)
-		(at 237.49 124.46 180)
-		(fields_autoplaced yes)
-		(effects
-			(font
-				(size 1.27 1.27)
-			)
-			(justify right)
-		)
-		(property "Intersheetrefs" "${INTERSHEET_REFS}"
-			(at 227.6333 124.46 0)
-			(effects
-				(font
-					(size 1.27 1.27)
-				)
-				(justify right)
-				(hide yes)
-			)
-		)
-	)
 	(global_label "FMC_D17"
 		(shape passive)
@@
 		)
 	)
-	(global_label "LTDC_B6"
-		(shape passive)
-		(at 237.49 114.3 180)
-		(fields_autoplaced yes)
-		(effects
-			(font
-				(size 1.27 1.27)
-			)
-			(justify right)
-		)
-		(property "Intersheetrefs" "${INTERSHEET_REFS}"
-			(at 227.6333 114.3 0)
-			(effects
-				(font
-					(size 1.27 1.27)
-				)
-				(justify right)
-				(hide yes)
-			)
-		)
-	)
 	(global_label "FMC_D9"
 		(shape passive)
@@
 		)
 	)
-	(global_label "LTDC_G7"
-		(shape passive)
-		(at 237.49 106.68 180)
-		(fields_autoplaced yes)
-		(effects
-			(font
-				(size 1.27 1.27)
-			)
-			(justify right)
-		)
-		(property "Intersheetrefs" "${INTERSHEET_REFS}"
-			(at 227.6333 106.68 0)
-			(effects
-				(font
-					(size 1.27 1.27)
-				)
-				(justify right)
-				(hide yes)
-			)
-		)
-	)
 	(global_label "LTDC_G4"
 		(shape passive)
@@
 		)
 	)
-	(global_label "LTDC_G6"
-		(shape passive)
-		(at 238.76 195.58 180)
-		(fields_autoplaced yes)
-		(effects
-			(font
-				(size 1.27 1.27)
-			)
-			(justify right)
-		)
-		(property "Intersheetrefs" "${INTERSHEET_REFS}"
-			(at 228.9033 195.58 0)
-			(effects
-				(font
-					(size 1.27 1.27)
-				)
-				(justify right)
-				(hide yes)
-			)
-		)
-	)
 	(global_label "DEBUG_JTDO_SWO"
 		(shape passive)
@@
 		)
 	)
-	(global_label "LTDC_B7"
-		(shape passive)
-		(at 237.49 116.84 180)
-		(fields_autoplaced yes)
-		(effects
-			(font
-				(size 1.27 1.27)
-			)
-			(justify right)
-		)
-		(property "Intersheetrefs" "${INTERSHEET_REFS}"
-			(at 227.6333 116.84 0)
-			(effects
-				(font
-					(size 1.27 1.27)
-				)
-				(justify right)
-				(hide yes)
-			)
-		)
-	)
 	(global_label "FMC_A3"
 		(shape passive)
@@
 				(hide yes)
 			)
-		)
-	)
-	(global_label "LTDC_R6"
-		(shape passive)
-		(at 328.93 127 0)
-		(fields_autoplaced yes)
-		(effects
-			(font
-				(size 1.27 1.27)
-			)
-			(justify left)
-		)
-		(property "Intersheetrefs" "${INTERSHEET_REFS}"
-			(at 338.7867 127 0)
-			(effects
-				(font
-					(size 1.27 1.27)
-				)
-				(justify left)
-				(hide yes)
-			)

Commit message: 중간 저장2
Connections:
- net USB_ID: no longer names the net of U1.144 (PA10)
Changed lines of the file:
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@@
-	(wire
-		(pts
-			(xy 321.31 106.68) (xy 328.93 106.68)
-		)
-		(stroke
-			(width 0)
-			(type default)
-		)
-	)
 	(wire
 		(pts
@@
 		)
 	)
+	(global_label "FMC_SDNWE"
+		(shape passive)
+		(at 238.76 223.52 180)
+		(fields_autoplaced yes)
+		(effects
+			(font
+				(size 1.27 1.27)
+			)
+			(justify right)
+		)
+		(property "Intersheetrefs" "${INTERSHEET_REFS}"
+			(at 225.6981 223.52 0)
+			(effects
+				(font
+					(size 1.27 1.27)
+				)
+				(justify right)
+				(hide yes)
+			)
+		)
+	)
 	(global_label "FMC_D17"
 		(shape passive)
@@
 			(effects
 				(font
-					(size 1.27 1.27)
-				)
-				(justify left)
-				(hide yes)
-			)
-		)
-	)
-	(global_label "USB_ID"
-		(shape passive)
-		(at 328.93 106.68 0)
-		(fields_autoplaced yes)
-		(effects
-			(font
-				(size 1.27 1.27)
-			)
-			(justify left)
-		)
-		(property "Intersheetrefs" "${INTERSHEET_REFS}"
-			(at 337.4563 106.68 0)
-			(effects
-				(font

Commit message: 중간저장
Parts:
- added C28: 0.1uF/16V, symbol Device:C_Small_US
- added R85: 2K/0.063w, symbol Device:R_Small_US
Connections:
- net 3V3_MCU: now also R85.1
- net GND: now also SW1.1, C28.2
- net at SW1.2: now also C28.1, R85.2
Other:
- moved on the sheet: SW1

Commit message: 중간 저장
Parts:
- removed J2: usb_pwr, symbol Connector_Generic:Conn_01x02
- added Q3: PMOS, symbol Simulation_SPICE:PMOS
Changed lines of the file:
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@@
+	)
+	(symbol
+		(lib_id "Simulation_SPICE:PMOS")
+		(at 90.17 101.6 270)
+		(mirror x)
+		(unit 1)
+		(exclude_from_sim no)
+		(in_bom yes)
+		(on_board yes)
+		(dnp no)
+		(property "Reference" "Q3"
+			(at 90.17 92.71 90)
+			(effects
+				(font
+					(size 1.27 1.27)
+				)
+			)
+		)
+		(property "Value" "PMOS"
+			(at 90.17 95.25 90)
+			(effects
+				(font
+					(size 1.27 1.27)
+				)
+			)
+		)
+		(property "Footprint" ""
+			(at 92.71 96.52 0)
+			(effects
+				(font
+					(size 1.27 1.27)
+				)
+				(hide yes)
+			)
+		)
+		(property "Datasheet" "https://ngspice.sourceforge.io/docs/ngspice-html-manual/manual.xhtml#cha_MOSFETs"
+			(at 77.47 101.6 0)
+			(effects
+				(font
+					(size 1.27 1.27)
+				)
+				(hide yes)
+			)
+		)
+		(property "Description" "P-MOSFET transistor, drain/source/gate"
+			(at 90.17 101.6 0)
+			(effects
+				(font
+					(size 1.27 1.27)
+				)
+				(hide yes)
+			)
+		)
+		(property "Sim.Device" "PMOS"
+			(at 73.025 101.6 0)
+			(effects
+				(font
+					(size 1.27 1.27)
+				)
+				(hide yes)
+			)
+		)
+		(property "Sim.Type" "VDMOS"
+			(at 71.12 101.6 0)
+			(effects
+				(font
+					(size 1.27 1.27)
+				)
+				(hide yes)
+			)
+		)
+		(property "Sim.Pins" "1=D 2=G 3=S"
+			(at 74.93 101.6 0)
+			(effects
+				(font
+					(size 1.27 1.27)
+				)
+				(hide yes)
+			)
+		)
+		(pin "3"
+		)
+		(pin "1"
+		)
+		(pin "2"
+		)
+		(instances
+			(project "bldc_motor_controller"
+				(path "/a25adab6-a8c3-4e0e-8ba9-baac00aaa394/f1d28d97-f090-4298-9a06-d9576d5adbbf"
+					(reference "Q3")
+					(unit 1)
+				)
+			)
+		)
 	)
 	(symbol
@@
 					(unit 1)
 				)
-			)
-		)
-	)
-	(symbol
-		(lib_id "Connector_Generic:Conn_01x02")
-		(at 72.39 115.57 180)
-		(unit 1)
-		(exclude_from_sim no)
-		(in_bom yes)
-		(on_board yes)
-		(dnp no)
-		(fields_autoplaced yes)
-		(property "Reference" "J2"
-			(at 72.39 106.68 0)
-			(effects
-				(font
-					(size 1.27 1.27)
-				)
-			)
-		)
-		(property "Value" "usb_pwr"
-			(at 72.39 109.22 0)
-			(effects
-				(font
-					(size 1.27 1.27)
-				)
-			)
-		)
-		(property "Footprint" ""
-			(at 72.39 115.57 0)
-			(effects
-				(font
-					(size 1.27 1.27)
-				)
-				(hide yes)
-			)
-		)
-		(property "Datasheet" "~"
-			(at 72.39 115.57 0)
-			(effects
-				(font
-					(size 1.27 1.27)
-				)
-				(hide yes)
-			)
-		)
-		(property "Description" "Generic connector, single row, 01x02, script generated (kicad-library-utils/schlib/autogen/connector/)"
-			(at 72.39 115.57 0)
-			(effects
-				(font
-					(size 1.27 1.27)
-				)
-				(hide yes)
-			)
-		)
-		(pin "1"
-		)
-		(pin "2"
-		)
-		(instances
-			(project ""
-				(path "/a25adab6-a8c3-4e0e-8ba9-baac00aaa394/f1d28d97-f090-4298-9a06-d9576d5adbbf"
-					(reference "J2")
-					(unit 1)
-				)

Commit message: 중간 저장
Parts:
- removed C28: 0.1uF/16V, symbol Device:C_Small_US
- removed J3: vat_pwr, symbol Connector_Generic:Conn_01x02
- removed J4: ext_pwr, symbol Connector_Generic:Conn_01x02
- removed Q3: PMOS, symbol Simulation_SPICE:PMOS
- removed R85: 2K/0.063w, symbol Device:R_Small_US
- removed SW1: reset_btn, Button_Switch_THT:SW_PUSH_6mm, symbol PCM_SL_Devices:Push_Button
- added C60, C61: 0.1uF/16V, symbol Device:C_Small_US
- added D10: LL4148, PCM_Diode_SMD_AKL:D_MiniMELF, symbol PCM_Diode_AKL:LL4148
- added IC3: STWD100NXWY3F, SOT95P280X145-5N, symbol SamacSys_Parts:STWD100NXWY3F
- added J2: Conn_01x02, symbol Connector_Generic:Conn_01x02
- added R94, R96: 10K/0.063w, symbol Device:R_Small_US
- added R95: 100/0.063w, symbol Device:R_Small_US
- added SW2: SW_DPDT_x2, symbol Switch:SW_DPDT_x2
- added SW3: Reset_Btn, symbol Switch:SW_Push
- renumbered C6 to C1, C8 to C10, C9 to C11, C10 to C12, C11 to C13, C12 to C14, C13 to C15, C14 to C16, C15 to C19, C1 to C2, C17 to C20, C16 to C21, C2 to C3, C3 to C4, C19 to C5, C4 to C6, C20 to C7, C5 to C8, C7 to C9, J1 to J3
Connections:
- net 3V3_MCU: now also C60.1, IC3.5 (VCC), J2.1 (Pin_1), R94.1, R96.1; no longer C1.1, C10.1, C11.1, C12.1, C13.1, C14.1, C15.1, C16.1, C19.1, C2.1, C21.1, C3.1, C4.1, C6.1, C8.1, C9.1, U1.103 (VDD), U1.115 (VDD), U1.124 (VDD), U1.15 (VDD), U1.150 (VDD), U1.158 (VDD), U1.171 (VDD), U1.185 (VDD), U1.204 (VDD), U1.26 (VDD), U1.39 (VDD), U1.52 (VDD), U1.59 (VDD), U1.73 (VDD), U1.83 (VDD), U1.94 (VDD)
- net GND: now also C60.2, C61.2, IC3.2 (GND), SW2.3 (C), SW3.1
- net ESP32_SPI2_NSS: now reaches U1.104 (PB12)
- net ESP32_SPI2_SCK: now reaches U1.105 (PB13)
- net ESP32_SPI2_MISO: now reaches U1.106 (PB14)
- net W25q_FLASH_SPI1_MISO: now reaches U1.178 (PG9)
- net W25q_FLASH_SPI1_NSS: now reaches U1.179 (PG10)
- net W25q_FLASH_SPI1_SCK: now reaches U1.180 (PG11)
- net WATCHDOG_OUT: now reaches U1.34 (NRST)
- net WATCHDOG_OUT: now also C61.1, D10.2 (A), IC3.1 (~{WDO}), R96.2
- net ESP32_SPI2_MOSI: now reaches U1.36 (PC1)
- net W25q_FLASH_SPI1_MOSI: now reaches U1.56 (PA7)
- new net: IC3.3 (~{EN}), R94.2, SW2.1 (A), SW2.2 (B)
- new net: D10.1 (K), R95.1
- new net: R95.2, SW3.2
- new net MCU_VDD: C1.1, C10.1, C11.1, C12.1, C13.1, C14.1, C15.1, C16.1, C19.1, C2.1, C21.1, C3.1, C4.1, C6.1, C8.1, C9.1, J2.2 (Pin_2), U1.103 (VDD), U1.115 (VDD), U1.124 (VDD), U1.15 (VDD), U1.150 (VDD), U1.158 (VDD), U1.171 (VDD), U1.185 (VDD), U1.204 (VDD), U1.26 (VDD), U1.39 (VDD), U1.52 (VDD), U1.59 (VDD), U1.73 (VDD), U1.83 (VDD), U1.94 (VDD)
- new net WATCHDOG_PWM: IC3.4 (WDI)

Commit message: 중간 저장
Parts:
- added Q1: PMOS, symbol Simulation_SPICE:PMOS
- added R110: 0R/0.063w, Resistor_SMD:R_0402_1005Metric, symbol Device:R_Small_US
- added R111: 4.7k/0.063w, Resistor_SMD:R_0402_1005Metric, symbol Device:R_Small_US
- IC3: footprint SOT95P280X145-5N -> SamacSys_Parts:SOT95P280X145-5N
- R94: value 10K/0.063w -> 4.7K/0.063w; footprint (none) -> Resistor_SMD:R_0402_1005Metric
- R95, R96: footprint (none) -> Resistor_SMD:R_0402_1005Metric
Connections:
- net 3V3_MCU: no longer J3.1 (Pin_1)
- net GND: now also R110.2, R111.2
- net at IC3.3 (~{EN}), R94.2, SW2.1 (A)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: now also Q1.3 (S)
- new net: Q1.1 (D), R110.1
- new net DEBUG_3V3: J3.1 (Pin_1), Q1.2 (G), R111.1
Other:
- moved on the sheet: SW2A

Commit message: 중간 저장
Parts:
- added C68, C69: 12pF/50V, symbol Device:C_Small_US
- added Q5, Q6, Q7: NMOS, symbol Simulation_SPICE:NMOS
- added R116, R117, R119, R120, R121, R122, R123, R124: 2K/0.063w, Resistor_SMD:R_0402_1005Metric, symbol Device:R_Small_US
- added Y1: X161032768KGD2SI, symbol Device:Crystal
Connections:
- net 3V3_MCU: now also Q5.2 (G), Q6.2 (G), Q7.2 (G), R116.1, R117.1, R120.1, R121.1, R123.1
- net GND: now also C68.2, C69.2
- net LTDC_R4: now also U1.68 (PJ3); no longer U1.54 (PA5)
- net BLUE_LED2: now reaches LED2.1 (K)
- net at LED2.2 (A): now also R117.2
- net BLUE_LED1: now reaches LED1.1 (K)
- net at LED1.2 (A): now also R116.2
- net OSC_32_OUT: now reaches U1.10 (PC15)
- net OSC_32_OUT: now also C69.1, Y1.2
- net I2C1_SCL: now reaches U1.195 (PB6)
- net I2C1_SDA: now reaches U1.196 (PB7)
- net CAN_RXD: now reaches U1.198 (PB8)
- net CAN_TXD: now reaches U1.199 (PB9)
- net OSC_32_IN: now reaches U1.9 (PC14)
- net OSC_32_IN: now also C68.1, Y1.1
- new net 5V: R119.1, R122.1, R124.1
- new net HALL_A: Q5.1 (D), R119.2
- new net HALL_A_INTR: Q5.3 (S), R120.2
- new net HALL_B: Q6.1 (D), R122.2
- new net HALL_B_INTR: Q6.3 (S), R121.2
- new net HALL_C: Q7.1 (D), R124.2
- new net HALL_C_INTR: Q7.3 (S), R123.2

Commit message: 중간 수정
Parts:
- C68, C69: footprint (none) -> Capacitor_SMD:C_0402_1005Metric
Changed lines of the file:
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@@
 			)
 		)
-		(property "Footprint" ""
+		(property "Footprint" "Capacitor_SMD:C_0402_1005Metric"
 			(at 378.46 209.55 0)
 			(effects
@@
 			)
 		)
-		(property "Footprint" ""
+		(property "Footprint" "Capacitor_SMD:C_0402_1005Metric"
 			(at 391.16 209.55 0)
 			(effects
