File: 1.hardware/mcu.kicad_sch (KiCad schematic)
At the start: 50 parts, among them J3 DEBUG_CONN, U1 TL431AIDBZR, U2 STM32H743BITx, U3 TXS0104EPW, X1 SMD3225-4, Y1 X1A0000610002

Commit message: 중간 저장
Connections:
- net 3V3_MCU: now also U2.137 (VDD33_USB)
Changed lines of the file:
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@@
+	)
+	(junction
+		(at 300.99 66.04)
+		(diameter 0)
+		(color 0 0 0 0)
 	)
 	(junction
@@
 	(wire
 		(pts
+			(xy 303.53 66.04) (xy 300.99 66.04)
+		)
+		(stroke
+			(width 0)
+			(type default)
+		)
+	)
+	(wire
+		(pts
 			(xy 121.92 119.38) (xy 119.38 119.38)
 		)
@@
 		)
 		(stroke
+			(width 0)
+			(type default)
+		)
+	)
+	(wire
+		(pts
+			(xy 303.53 71.12) (xy 303.53 66.04)
+		)
+		(stroke
