File: 1.hardware/bldc_motor_controller.kicad_pcb (KiCad board)
At the start: 2 copper layers, 2 parts, among them U1 STM32H743BITx, X1 SMD3225-4

Commit message: 중간 저장2
Parts:
- added AC1: BNO085, SamacSys_Parts:BNO085, F.Cu at (73.8, 83.7)
- added SW1: reset_btn, Button_Switch_THT:SW_PUSH_6mm, F.Cu at (73.5, 72.0)
Connections:
- U1 pad 100: unconnected-(U1-PH10-Pad100) -> FMC_D18
- U1 pad 101: unconnected-(U1-PH11-Pad101) -> FMC_D19
- U1 pad 102: unconnected-(U1-PH12-Pad102) -> FMC_D20
- U1 pad 103: unconnected-(U1-VDD-Pad103) -> 3V3_MCU
- U1 pad 108: unconnected-(U1-PD8-Pad108) -> FMC_D13
- U1 pad 109: unconnected-(U1-PD9-Pad109) -> FMC_D14
- U1 pad 11: unconnected-(U1-PI9-Pad11) -> FMC_D30
- U1 pad 110: unconnected-(U1-PD10-Pad110) -> FMC_D15
- U1 pad 115: unconnected-(U1-VDD-Pad115) -> 3V3_MCU
- U1 pad 116: unconnected-(U1-PD14-Pad116) -> FMC_D0
- U1 pad 117: unconnected-(U1-PD15-Pad117) -> FMC_D1
- U1 pad 12: unconnected-(U1-PI10-Pad12) -> FMC_D31
- U1 pad 122: unconnected-(U1-PJ10-Pad122) -> LTDC_G3
- U1 pad 124: unconnected-(U1-VDD-Pad124) -> 3V3_MCU
- U1 pad 131: unconnected-(U1-PG4-Pad131) -> FMC_BA0
- U1 pad 132: unconnected-(U1-PG5-Pad132) -> FMC_BA1
- U1 pad 135: unconnected-(U1-PG8-Pad135) -> FMC_SDCLK
- U1 pad 141: unconnected-(U1-PC9-Pad141) -> LTDC_B2
- U1 pad 142: unconnected-(U1-PA8-Pad142) -> LTDC_B3
- U1 pad 144: unconnected-(U1-PA10-Pad144) -> USB_ID
- U1 pad 145: unconnected-(U1-PA11-Pad145) -> USB_DM
- U1 pad 146: unconnected-(U1-PA12-Pad146) -> USB_DP
- U1 pad 147: unconnected-(U1-PA13-Pad147) -> DEBUG_SWDIO
- U1 pad 148: unconnected-(U1-VCAP-Pad148) -> Net-(C17-Pad1)
- U1 pad 15: unconnected-(U1-VDD-Pad15) -> 3V3_MCU
- U1 pad 150: unconnected-(U1-VDD-Pad150) -> 3V3_MCU
- U1 pad 151: unconnected-(U1-PH13-Pad151) -> FMC_D21
- U1 pad 152: unconnected-(U1-PH14-Pad152) -> FMC_D22
- U1 pad 153: unconnected-(U1-PH15-Pad153) -> FMC_D23
- U1 pad 154: unconnected-(U1-PI0-Pad154) -> FMC_D24
- U1 pad 155: unconnected-(U1-PI1-Pad155) -> FMC_D25
- U1 pad 156: unconnected-(U1-PI2-Pad156) -> FMC_D26
- U1 pad 157: unconnected-(U1-PI3-Pad157) -> FMC_D27
- U1 pad 158: unconnected-(U1-VDD-Pad158) -> 3V3_MCU
- U1 pad 159: unconnected-(U1-PA14-Pad159) -> DEBUG_SWCLK
- U1 pad 16: unconnected-(U1-PF0-Pad16) -> FMC_A0
- U1 pad 160: unconnected-(U1-PA15-Pad160) -> DEBUG_JTDI
- U1 pad 164: unconnected-(U1-PD0-Pad164) -> FMC_D2
- U1 pad 165: unconnected-(U1-PD1-Pad165) -> FMC_D3
- U1 pad 17: unconnected-(U1-PF1-Pad17) -> FMC_A1
- U1 pad 171: unconnected-(U1-VDD-Pad171) -> 3V3_MCU
- U1 pad 175: unconnected-(U1-PJ13-Pad175) -> LTDC_B1
- U1 pad 18: unconnected-(U1-PF2-Pad18) -> FMC_A2
- U1 pad 181: unconnected-(U1-PG12-Pad181) -> LTDC_B4
- U1 pad 185: unconnected-(U1-VDD-Pad185) -> 3V3_MCU
- U1 pad 191: unconnected-(U1-PG15-Pad191) -> FMC_SDNCAS
- U1 pad 192: unconnected-(U1-PB3-Pad192) -> DEBUG_JTDO_SWO
- U1 pad 193: unconnected-(U1-PB4-Pad193) -> DEBUG_RESET
- U1 pad 200: unconnected-(U1-PE0-Pad200) -> FMC_NBL0
- U1 pad 201: unconnected-(U1-PE1-Pad201) -> FMC_NBL1
- U1 pad 204: unconnected-(U1-VDD-Pad204) -> 3V3_MCU
- U1 pad 205: unconnected-(U1-PI4-Pad205) -> FMC_NBL2
- U1 pad 206: unconnected-(U1-PI5-Pad206) -> FMC_NBL3
- U1 pad 207: unconnected-(U1-PI6-Pad207) -> FMC_D28
- U1 pad 208: unconnected-(U1-PI7-Pad208) -> FMC_D29
- U1 pad 22: unconnected-(U1-PF3-Pad22) -> LTDC_HSYNC
- U1 pad 23: unconnected-(U1-PF4-Pad23) -> LTDC_VSYNC
- U1 pad 24: unconnected-(U1-PF5-Pad24) -> LTDC_CLK
- U1 pad 26: unconnected-(U1-VDD-Pad26) -> 3V3_MCU
- U1 pad 27: unconnected-(U1-PF6-Pad27) -> FMC_A3
- U1 pad 28: unconnected-(U1-PF7-Pad28) -> FMC_A4
- U1 pad 29: unconnected-(U1-PF8-Pad29) -> FMC_A5
- U1 pad 3: unconnected-(U1-PE4-Pad3) -> LTDC_B0
- U1 pad 31: unconnected-(U1-PF10-Pad31) -> LTDC_DE
- U1 pad 32: unconnected-(U1-PH0-Pad32) -> RCC_IN
- U1 pad 33: unconnected-(U1-PH1-Pad33) -> RCC_OUT
- U1 pad 35: unconnected-(U1-PC0-Pad35) -> LTDC_R5
- U1 pad 37: unconnected-(U1-PC2_C-Pad37) -> FMC_SDNE0
- U1 pad 39: unconnected-(U1-VDD-Pad39) -> 3V3_MCU
- U1 pad 4: unconnected-(U1-PE5-Pad4) -> LTDC_G0
- U1 pad 44: unconnected-(U1-PA1-Pad44) -> LTDC_R2
- U1 pad 45: unconnected-(U1-PA2-Pad45) -> LTDC_R1
- U1 pad 46: unconnected-(U1-PH2-Pad46) -> LTDC_R0
- U1 pad 48: unconnected-(U1-PH4-Pad48) -> LTDC_G5
- U1 pad 5: unconnected-(U1-PE6-Pad5) -> LTDC_G1
- U1 pad 50: unconnected-(U1-PA3-Pad50) -> LTDC_B5
- U1 pad 52: unconnected-(U1-VDD-Pad52) -> 3V3_MCU
- U1 pad 53: unconnected-(U1-PA4-Pad53) -> Speaker_DAC
- U1 pad 54: unconnected-(U1-PA5-Pad54) -> LTDC_R4
- U1 pad 58: unconnected-(U1-PC5-Pad58) -> FMC_SDCKE0
- U1 pad 59: unconnected-(U1-VDD-Pad59) -> 3V3_MCU
- U1 pad 61: unconnected-(U1-PB0-Pad61) -> LTDC_R3
- U1 pad 64: unconnected-(U1-PI15-Pad64) -> LTDC_G2
- U1 pad 70: unconnected-(U1-PF11-Pad70) -> FMC_SDNRAS
- U1 pad 71: unconnected-(U1-PF12-Pad71) -> FMC_A6
- U1 pad 73: unconnected-(U1-VDD-Pad73) -> 3V3_MCU
- U1 pad 74: unconnected-(U1-PF13-Pad74) -> FMC_A7
- U1 pad 75: unconnected-(U1-PF14-Pad75) -> FMC_A8
- U1 pad 76: unconnected-(U1-PF15-Pad76) -> FMC_A9
- U1 pad 77: unconnected-(U1-PG0-Pad77) -> FMC_A10
- U1 pad 78: unconnected-(U1-PG1-Pad78) -> FMC_A11
- U1 pad 79: unconnected-(U1-PE7-Pad79) -> FMC_D4
- U1 pad 80: unconnected-(U1-PE8-Pad80) -> FMC_D5
- U1 pad 81: unconnected-(U1-PE9-Pad81) -> FMC_D6
- U1 pad 83: unconnected-(U1-VDD-Pad83) -> 3V3_MCU
- U1 pad 84: unconnected-(U1-PE10-Pad84) -> FMC_D7
- U1 pad 85: unconnected-(U1-PE11-Pad85) -> FMC_D8
- U1 pad 86: unconnected-(U1-PE12-Pad86) -> FMC_D9
- U1 pad 87: unconnected-(U1-PE13-Pad87) -> FMC_D10
- U1 pad 88: unconnected-(U1-PE14-Pad88) -> FMC_D11
- U1 pad 89: unconnected-(U1-PE15-Pad89) -> FMC_D12
- U1 pad 90: unconnected-(U1-PB10-Pad90) -> LTDC_G4
- U1 pad 92: unconnected-(U1-VCAP-Pad92) -> Net-(C18-Pad1)
- U1 pad 94: unconnected-(U1-VDD-Pad94) -> 3V3_MCU
- U1 pad 98: unconnected-(U1-PH8-Pad98) -> FMC_D16
- U1 pad 99: unconnected-(U1-PH9-Pad99) -> FMC_D17
- X1 pad 1: unconnected-(X1-Pad1) -> RCC_IN
- X1 pad 2: unconnected-(X1-Pad2) -> GND
- X1 pad 3: unconnected-(X1-Pad3) -> RCC_OUT
- X1 pad 4: unconnected-(X1-Pad4) -> GND

Commit message: 중간저장
Parts:
- added C21: 0.1uF/16V, Capacitor_SMD:C_0402_1005Metric, F.Cu at (166.0, 93.4)
- added C22: 0.1uF/16V, Capacitor_SMD:C_0402_1005Metric, F.Cu at (166.0, 95.4)
- added C23: 2.2uF/6.3V, Capacitor_SMD:C_0603_1608Metric, F.Cu at (162.4, 98.3)
- added C24: 0.1uF/16V, Capacitor_SMD:C_0402_1005Metric, F.Cu at (195.5, 66.9)
- added C25: 4.7uF/10V, Capacitor_SMD:C_0603_1608Metric, F.Cu at (182.2, 92.6)
- added C26: 1uF/50V, Capacitor_SMD:C_0603_1608Metric, F.Cu at (182.2, 95.1)
- added C27: 1uF/50V, Capacitor_SMD:C_0603_1608Metric, F.Cu at (182.2, 97.6)
- added C52: 0.1uF/16V, Capacitor_SMD:C_0402_1005Metric, F.Cu at (195.5, 68.8)
- added C53: 0.1uF/16V, Capacitor_SMD:C_0402_1005Metric, F.Cu at (195.5, 70.8)
- added C54: 0.1uF/16V, Capacitor_SMD:C_0402_1005Metric, F.Cu at (195.5, 72.8)
- added C55: 2.2uF/6.3V, Capacitor_SMD:C_0603_1608Metric, F.Cu at (198.9, 67.1)
- added C56: 0.1uF/16V, Capacitor_SMD:C_0402_1005Metric, F.Cu at (195.5, 74.7)
- added C57: 0.1uF/16V, Capacitor_SMD:C_0402_1005Metric, F.Cu at (195.5, 76.7)
- added C58: 0.1uF/16V, Capacitor_SMD:C_0402_1005Metric, F.Cu at (195.5, 78.7)
- added C59: 0.1uF/16V, Capacitor_SMD:C_0402_1005Metric, F.Cu at (195.5, 80.7)
- added D1: NSR0240V2, PCM_Diode_SMD_AKL:D_SOD-523, F.Cu at (186.1, 93.0)
- added D2: NSR0240V2, PCM_Diode_SMD_AKL:D_SOD-523, F.Cu at (186.1, 96.2)
- added D4: PRTR5V0U2X, Package_TO_SOT_SMD:SOT-143, F.Cu at (162.5, 94.8)
- added IC1: IS42S32800J-6TLI, SamacSys_Parts:SOP50P1176X120-86N, F.Cu at (187.2, 77.6)
- added J7: Connector_USB_C_Receptacle_USB2.0, Connector_USB:USB_C_Receptacle_HRO_TYPE-C-31-M-12, F.Cu at (154.5, 98.2)
- added LED1: LED_0603_Blue, PCM_LED_SMD_AKL:LED_0603_1608Metric, F.Cu at (196.2, 101.7)
- added LED2: LED_0603_Blue, PCM_LED_SMD_AKL:LED_0603_1608Metric, F.Cu at (196.2, 105.0)
- added PS1: TPS61169DCKR, SamacSys_Parts:SOT65P210X110-5N, F.Cu at (190.1, 93.0)
- added PS2: TPS61169DCKR, SamacSys_Parts:SOT65P210X110-5N, F.Cu at (190.1, 96.0)
- added U4: LM2904AYD, PCM_Package_SO_AKL:SO-8_3.9x4.9mm_P1.27mm, F.Cu at (198.5, 94.7)
- added U5: ESP32-C3-WROOM-02, RF_Module:ESP32-C3-WROOM-02, F.Cu at (163.4, 84.8)
- added U6: W25Q128JVS, Package_SO:SOIC-8_5.3x5.3mm_P1.27mm, F.Cu at (199.2, 85.1)
Connections:
- AC1 pad 2: unconnected-(AC1-GND_1-Pad2) -> GND
- AC1 pad 25: unconnected-(AC1-GND_2-Pad25) -> GND
- U1 pad 144: USB_ID -> unconnected-(U1-PA10-Pad144)

Commit message: 중간 저장
Parts:
- removed AC1: BNO085, SamacSys_Parts:BNO085
- added C22: 30pF/50V, Capacitor_SMD:C_0603_1608Metric, F.Cu at (119.5, 95.0)
- added C23: 0.22uF/50V, Capacitor_SMD:C_0603_1608Metric, F.Cu at (119.5, 97.5)
- added C24: 100uF/50V, Capacitor_THT:CP_Radial_Tantal_D8.0mm_P5.00mm, F.Cu at (110.2, 98.5)
- added C25: 0.1uF/50V, Capacitor_SMD:C_0402_1005Metric, F.Cu at (121.4, 113.8)
- added C26: 0.01uF/50V, Capacitor_SMD:C_0402_1005Metric, F.Cu at (121.4, 115.8)
- added C27: 0.22uF/50V, Capacitor_SMD:C_0603_1608Metric, F.Cu at (119.5, 100.0)
- added C29: 0.01uF/50V, Capacitor_SMD:C_0402_1005Metric, F.Cu at (121.4, 117.7)
- added C30: 0.01uF/50V, Capacitor_SMD:C_0402_1005Metric, F.Cu at (121.4, 119.7)
- added C31: 100uF/50V, Capacitor_THT:CP_Radial_Tantal_D8.0mm_P5.00mm, F.Cu at (110.2, 108.0)
- added C32: 0.22uF/50V, Capacitor_SMD:C_0603_1608Metric, F.Cu at (119.5, 102.5)
- added C33: 0.1uF/50V, Capacitor_SMD:C_0402_1005Metric, F.Cu at (121.4, 121.7)
- added C34: 0.01uF/50V, Capacitor_SMD:C_0402_1005Metric, F.Cu at (121.4, 123.6)
- added C35: 0.1uF/50V, Capacitor_SMD:C_0402_1005Metric, F.Cu at (121.4, 125.6)
- added C36: 0.1uF/50V, Capacitor_SMD:C_0402_1005Metric, F.Cu at (121.4, 127.6)
- added C37: 10uF/25V, Capacitor_SMD:C_1206_3216Metric, F.Cu at (120.0, 131.0)
- added D1: LL4148, PCM_Diode_SMD_AKL:D_MiniMELF, F.Cu at (111.0, 131.4)
- added D4: Green_Led, LED_SMD:LED_0603_1608Metric, F.Cu at (119.2, 134.0)
- added D5: WS2812B, LED_SMD:LED_WS2812B_PLCC4_5.0x5.0mm_P3.2mm, F.Cu at (128.9, 97.0)
- added D6: WS2812B, LED_SMD:LED_WS2812B_PLCC4_5.0x5.0mm_P3.2mm, F.Cu at (128.9, 103.6)
- added J5: Barrel_Jack_Switch_Pin3Ring, Connector_BarrelJack:BarrelJack_Wuerth_6941xx301002, F.Cu at (113.3, 114.7)
- added L1: 60R_100Mhz, Inductor_SMD:L_0603_1608Metric, F.Cu at (119.5, 105.0)
- added L2: 60R_100Mhz, Inductor_SMD:L_0603_1608Metric, F.Cu at (119.5, 107.5)
- added L3: 60R_100Mhz, Inductor_SMD:L_0603_1608Metric, F.Cu at (119.5, 110.0)
- added L4: 47uH/1.55A, Inductor_SMD:L_12x12mm_H6mm, F.Cu at (100.4, 100.8)
- added L5: 47uH/1.55A, Inductor_SMD:L_12x12mm_H6mm, F.Cu at (100.4, 115.1)
- added L6: 3.3uH/1.6A, Inductor_SMD:L_12x12mm_H6mm, F.Cu at (100.4, 129.3)
- added R7: 0R/0.063w, Resistor_SMD:R_0402_1005Metric, F.Cu at (115.7, 130.3)
- added R8: 0R/0.063w, Resistor_SMD:R_0402_1005Metric, F.Cu at (115.7, 132.3)
- added R9: 3.3K/0.063w, Resistor_SMD:R_0402_1005Metric, F.Cu at (115.7, 134.3)
- renumbered C25 to C38, C26 to C39, C27 to C40, C24 to C41, C52 to C42, C56 to C43, C53 to C44, C57 to C45, C54 to C46, C58 to C47, C55 to C48, C59 to C49, C21 to C50, C22 to C51, C23 to C52, D1 to D7, D2 to D8, D4 to D9, IC1 to IC2, J7 to J8, U6 to U3
Connections:
- SW1 pad 1: unconnected-(SW1-Pad1) -> GND
- SW1 pad 2: unconnected-(SW1-Pad2) -> Net-(C17-Pad1)

Commit message: 중간 저장
Parts:
- added C53: 100uF/16V, Capacitor_THT:CP_Radial_Tantal_D8.0mm_P5.00mm, F.Cu at (242.1, 107.9)
- added C54: 0.1uF/50V, Capacitor_SMD:C_0402_1005Metric, F.Cu at (250.8, 104.1)
- added C55: 0.1uF/50V, Capacitor_SMD:C_0402_1005Metric, F.Cu at (250.8, 106.1)
- added C56: 0.22uF/50V, Capacitor_SMD:C_0603_1608Metric, F.Cu at (250.1, 113.9)
- added C57: 0.1uF/16V, Capacitor_SMD:C_0402_1005Metric, F.Cu at (235.1, 106.6)
- added C58: 0.1uF/16V, Capacitor_SMD:C_0402_1005Metric, F.Cu at (235.1, 108.6)
- added C59: 2.2uF/6.3V, Capacitor_SMD:C_0603_1608Metric, F.Cu at (235.7, 104.4)
- added C62: 0.1uF/16V, Capacitor_SMD:C_0402_1005Metric, F.Cu at (261.5, 128.0)
- added D10: LL4148, PCM_Diode_SMD_AKL:D_MiniMELF, F.Cu at (262.6, 82.2)
- added IC3: STWD100NXWY3F, SamacSys_Parts:SOT95P280X145-5N, F.Cu at (261.8, 78.1)
- added L9: 60R_100Mhz, Inductor_SMD:L_0603_1608Metric, F.Cu at (250.1, 116.4)
- added LED3: LED_0603_Red_WIFI, PCM_LED_SMD_AKL:LED_0603_1608Metric, F.Cu at (262.1, 118.7)
- added LED4: LED_0603_Blue_BLE, PCM_LED_SMD_AKL:LED_0603_1608Metric, F.Cu at (262.1, 122.0)
- added LED5: LED_0603_Green_PWR, PCM_LED_SMD_AKL:LED_0603_1608Metric, F.Cu at (262.1, 125.4)
- added R100: 10k/0.063w, Resistor_SMD:R_0402_1005Metric, F.Cu at (232.2, 118.0)
- added R101: 4.7K/0.063w, Resistor_SMD:R_0402_1005Metric, F.Cu at (255.7, 126.0)
- added R102: 4.7K/0.063w, Resistor_SMD:R_0402_1005Metric, F.Cu at (255.7, 128.0)
- added R103: 4.7K/0.063w, Resistor_SMD:R_0402_1005Metric, F.Cu at (258.6, 118.0)
- added R104: 4.7K/0.063w, Resistor_SMD:R_0402_1005Metric, F.Cu at (258.6, 120.0)
- added R105: 4.7K/0.063w, Resistor_SMD:R_0402_1005Metric, F.Cu at (258.6, 122.0)
- added R106: 4.7K/0.063w, Resistor_SMD:R_0402_1005Metric, F.Cu at (258.6, 124.0)
- added R107: 4.7K/0.063w, Resistor_SMD:R_0402_1005Metric, F.Cu at (258.6, 126.0)
- added R108: 4.7k/0.063w, Resistor_SMD:R_0402_1005Metric, F.Cu at (217.6, 100.1)
- added R12: 22R/0.063w, Resistor_SMD:R_0402_1005Metric, F.Cu at (255.7, 104.1)
- added R13: 22R/0.063w, Resistor_SMD:R_0402_1005Metric, F.Cu at (255.7, 106.1)
- added R14: 22R/0.063w, Resistor_SMD:R_0402_1005Metric, F.Cu at (255.7, 108.1)
- added R15: 22R/0.063w, Resistor_SMD:R_0402_1005Metric, F.Cu at (255.7, 110.1)
- added R16: 22R/0.063w, Resistor_SMD:R_0402_1005Metric, F.Cu at (255.7, 112.1)
- added R17: 22R/0.063w, Resistor_SMD:R_0402_1005Metric, F.Cu at (255.7, 114.1)
- added R18: 22R/0.063w, Resistor_SMD:R_0402_1005Metric, F.Cu at (258.6, 104.1)
- added R19: 22R/0.063w, Resistor_SMD:R_0402_1005Metric, F.Cu at (258.6, 106.1)
- added R20: 22R/0.063w, Resistor_SMD:R_0402_1005Metric, F.Cu at (258.6, 108.1)
- added R21: 22R/0.063w, Resistor_SMD:R_0402_1005Metric, F.Cu at (258.6, 110.1)
- added R22: 22R/0.063w, Resistor_SMD:R_0402_1005Metric, F.Cu at (258.6, 112.1)
- added R23: 22R/0.063w, Resistor_SMD:R_0402_1005Metric, F.Cu at (258.6, 114.1)
- added R24: 22R/0.063w, Resistor_SMD:R_0402_1005Metric, F.Cu at (261.5, 104.1)
- added R25: 22R/0.063w, Resistor_SMD:R_0402_1005Metric, F.Cu at (261.5, 106.1)
- added R26: 22R/0.063w, Resistor_SMD:R_0402_1005Metric, F.Cu at (261.5, 108.1)
- added R27: 22R/0.063w, Resistor_SMD:R_0402_1005Metric, F.Cu at (261.5, 110.1)
- added R28: 22R/0.063w, Resistor_SMD:R_0402_1005Metric, F.Cu at (261.5, 112.1)
- added R29: 22R/0.063w, Resistor_SMD:R_0402_1005Metric, F.Cu at (261.5, 114.1)
- added R30: 22R/0.063w, Resistor_SMD:R_0402_1005Metric, F.Cu at (264.4, 104.1)
- added R31: 22R/0.063w, Resistor_SMD:R_0402_1005Metric, F.Cu at (264.4, 106.1)
- added R32: 22R/0.063w, Resistor_SMD:R_0402_1005Metric, F.Cu at (264.4, 108.1)
- added R33: 22R/0.063w, Resistor_SMD:R_0402_1005Metric, F.Cu at (264.4, 110.1)
- added R34: 33R/0.063w, Resistor_SMD:R_0402_1005Metric, F.Cu at (217.6, 104.1)
- added R35: 33R/0.063w, Resistor_SMD:R_0402_1005Metric, F.Cu at (217.6, 106.1)
- added R36: 33R/0.063w, Resistor_SMD:R_0402_1005Metric, F.Cu at (217.6, 108.1)
- added R37: 33R/0.063w, Resistor_SMD:R_0402_1005Metric, F.Cu at (217.6, 110.1)
- added R38: 33R/0.063w, Resistor_SMD:R_0402_1005Metric, F.Cu at (217.6, 112.1)
- added R39: 33R/0.063w, Resistor_SMD:R_0402_1005Metric, F.Cu at (217.6, 114.1)
- added R40: 33R/0.063w, Resistor_SMD:R_0402_1005Metric, F.Cu at (217.6, 116.0)
- added R41: 33R/0.063w, Resistor_SMD:R_0402_1005Metric, F.Cu at (217.6, 118.0)
- added R42: 33R/0.063w, Resistor_SMD:R_0402_1005Metric, F.Cu at (217.6, 120.0)
- added R43: 33R/0.063w, Resistor_SMD:R_0402_1005Metric, F.Cu at (217.6, 122.0)
- added R44: 33R/0.063w, Resistor_SMD:R_0402_1005Metric, F.Cu at (220.6, 104.1)
- added R45: 33R/0.063w, Resistor_SMD:R_0402_1005Metric, F.Cu at (220.6, 106.1)
- added R46: 33R/0.063w, Resistor_SMD:R_0402_1005Metric, F.Cu at (220.6, 108.1)
- added R47: 33R/0.063w, Resistor_SMD:R_0402_1005Metric, F.Cu at (220.6, 110.1)
- added R48: 33R/0.063w, Resistor_SMD:R_0402_1005Metric, F.Cu at (220.6, 112.1)
- added R49: 33R/0.063w, Resistor_SMD:R_0402_1005Metric, F.Cu at (220.6, 114.1)
- added R50: 33R/0.063w, Resistor_SMD:R_0402_1005Metric, F.Cu at (220.6, 116.0)
- added R51: 33R/0.063w, Resistor_SMD:R_0402_1005Metric, F.Cu at (220.6, 118.0)
- added R52: 33R/0.063w, Resistor_SMD:R_0402_1005Metric, F.Cu at (220.6, 120.0)
- added R53: 33R/0.063w, Resistor_SMD:R_0402_1005Metric, F.Cu at (220.6, 122.0)
- added R54: 33R/0.063w, Resistor_SMD:R_0402_1005Metric, F.Cu at (223.5, 104.1)
- added R55: 33R/0.063w, Resistor_SMD:R_0402_1005Metric, F.Cu at (223.5, 106.1)
- added R56: 33R/0.063w, Resistor_SMD:R_0402_1005Metric, F.Cu at (223.5, 108.1)
- added R57: 33R/0.063w, Resistor_SMD:R_0402_1005Metric, F.Cu at (223.5, 110.1)
- added R58: 33R/0.063w, Resistor_SMD:R_0402_1005Metric, F.Cu at (223.5, 112.1)
- added R59: 33R/0.063w, Resistor_SMD:R_0402_1005Metric, F.Cu at (223.5, 114.1)
- added R60: 33R/0.063w, Resistor_SMD:R_0402_1005Metric, F.Cu at (223.5, 116.0)
- added R61: 33R/0.063w, Resistor_SMD:R_0402_1005Metric, F.Cu at (223.5, 118.0)
- added R62: 33R/0.063w, Resistor_SMD:R_0402_1005Metric, F.Cu at (223.5, 120.0)
- added R63: 33R/0.063w, Resistor_SMD:R_0402_1005Metric, F.Cu at (223.5, 122.0)
- added R64: 33R/0.063w, Resistor_SMD:R_0402_1005Metric, F.Cu at (226.4, 104.1)
- added R65: 33R/0.063w, Resistor_SMD:R_0402_1005Metric, F.Cu at (226.4, 106.1)
- added R66: 33R/0.063w, Resistor_SMD:R_0402_1005Metric, F.Cu at (226.4, 108.1)
- added R67: 33R/0.063w, Resistor_SMD:R_0402_1005Metric, F.Cu at (226.4, 110.1)
- added R68: 33R/0.063w, Resistor_SMD:R_0402_1005Metric, F.Cu at (226.4, 112.1)
- added R69: 33R/0.063w, Resistor_SMD:R_0402_1005Metric, F.Cu at (226.4, 114.1)
- added R70: 33R/0.063w, Resistor_SMD:R_0402_1005Metric, F.Cu at (226.4, 116.0)
- added R71: 33R/0.063w, Resistor_SMD:R_0402_1005Metric, F.Cu at (226.4, 118.0)
- added R72: 33R/0.063w, Resistor_SMD:R_0402_1005Metric, F.Cu at (226.4, 120.0)
- added R73: 33R/0.063w, Resistor_SMD:R_0402_1005Metric, F.Cu at (226.4, 122.0)
- added R74: 33R/0.063w, Resistor_SMD:R_0402_1005Metric, F.Cu at (229.3, 104.1)
- added R75: 33R/0.063w, Resistor_SMD:R_0402_1005Metric, F.Cu at (229.3, 106.1)
- added R76: 33R/0.063w, Resistor_SMD:R_0402_1005Metric, F.Cu at (229.3, 108.1)
- added R77: 33R/0.063w, Resistor_SMD:R_0402_1005Metric, F.Cu at (229.3, 110.1)
- added R78: 33R/0.063w, Resistor_SMD:R_0402_1005Metric, F.Cu at (229.3, 112.1)
- added R79: 33R/0.063w, Resistor_SMD:R_0402_1005Metric, F.Cu at (229.3, 114.1)
- added R80: 33R/0.063w, Resistor_SMD:R_0402_1005Metric, F.Cu at (229.3, 116.0)
- added R81: 33R/0.063w, Resistor_SMD:R_0402_1005Metric, F.Cu at (229.3, 118.0)
- added R82: 33R/0.063w, Resistor_SMD:R_0402_1005Metric, F.Cu at (229.3, 120.0)
- added R83: 33R/0.063w, Resistor_SMD:R_0402_1005Metric, F.Cu at (229.3, 122.0)
- added R84: 33R/0.063w, Resistor_SMD:R_0402_1005Metric, F.Cu at (232.2, 104.1)
- added R85: 33R/0.063w, Resistor_SMD:R_0402_1005Metric, F.Cu at (232.2, 106.1)
- added R86: 33R/0.063w, Resistor_SMD:R_0402_1005Metric, F.Cu at (232.2, 108.1)
- added R87: 33R/0.063w, Resistor_SMD:R_0402_1005Metric, F.Cu at (232.2, 110.1)
- added R88: 33R/0.063w, Resistor_SMD:R_0402_1005Metric, F.Cu at (232.2, 112.1)
- added R89: 33R/0.063w, Resistor_SMD:R_0402_1005Metric, F.Cu at (232.2, 114.1)
- added R90: 4.7K/0.063w, Resistor_SMD:R_0402_1005Metric, F.Cu at (255.7, 118.0)
- added R91: 4.7K/0.063w, Resistor_SMD:R_0402_1005Metric, F.Cu at (255.7, 120.0)
- added R92: NC_4.7K, Resistor_SMD:R_0402_1005Metric, F.Cu at (255.7, 122.0)
- added R93: 4.7K, Resistor_SMD:R_0402_1005Metric, F.Cu at (255.7, 124.0)
- added R94: 10K/0.063w, Resistor_SMD:R_0402_1005Metric, F.Cu at (257.8, 77.0)
- added R95: 100/0.063w, Resistor_SMD:R_0402_1005Metric, F.Cu at (257.8, 79.0)
- added R96: 10K/0.063w, Resistor_SMD:R_0402_1005Metric, F.Cu at (257.8, 81.0)
- added R99: 10k/0.063w, Resistor_SMD:R_0402_1005Metric, F.Cu at (232.2, 116.0)
- added U10: Hall_Analog_Joystick, New_Footprints:Hall_Analog_Joystick, F.Cu at (245.6, 88.3)
- added U6: LM2931-5.0_SO8, Package_SO:SOIC-8_3.9x4.9mm_P1.27mm, F.Cu at (243.9, 116.0)
- added U7: LM2904D, PCM_Package_SO_AKL:SO-8_3.9x4.9mm_P1.27mm, F.Cu at (260.7, 89.6)
- added U8: LM2904D, PCM_Package_SO_AKL:SO-8_3.9x4.9mm_P1.27mm, F.Cu at (260.7, 96.4)
- added U9: Hall_Analog_Joystick, New_Footprints:Hall_Analog_Joystick, F.Cu at (226.5, 88.3)
- J5: value Barrel_Jack_Switch_Pin3Ring -> 12V-24V Jack
- J8: value Connector_USB_C_Receptacle_USB2.0 -> USB_C
Connections:
- net /power/12V_1 renamed Net-(C23-Pad1)
- net Net-(IC1-EN) renamed PWR_INPUT(5V~24V)
- C22 pad 2: GND -> GNDPWR
- C23 pad 2: GND -> GNDPWR
- C24 pad 2: GND -> GNDPWR
- C25 pad 2: GND -> GNDPWR
- C26 pad 2: GND -> GNDPWR
- J5 pad 2: GND -> GNDPWR
- J5 pad 3: GND -> GNDPWR
- U1 pad 103: 3V3_MCU -> MCU_VDD
- U1 pad 104: unconnected-(U1-PB12-Pad104) -> ESP32_SPI2_NSS
- U1 pad 105: unconnected-(U1-PB13-Pad105) -> ESP32_SPI2_SCK
- U1 pad 106: unconnected-(U1-PB14-Pad106) -> ESP32_SPI2_MISO
- U1 pad 115: 3V3_MCU -> MCU_VDD
- U1 pad 124: 3V3_MCU -> MCU_VDD
- U1 pad 15: 3V3_MCU -> MCU_VDD
- U1 pad 150: 3V3_MCU -> MCU_VDD
- U1 pad 158: 3V3_MCU -> MCU_VDD
- U1 pad 171: 3V3_MCU -> MCU_VDD
- U1 pad 178: unconnected-(U1-PG9-Pad178) -> W25q_FLASH_SPI1_MISO
- U1 pad 179: unconnected-(U1-PG10-Pad179) -> W25q_FLASH_SPI1_NSS
- U1 pad 180: unconnected-(U1-PG11-Pad180) -> W25q_FLASH_SPI1_SCK
- U1 pad 185: 3V3_MCU -> MCU_VDD
- U1 pad 204: 3V3_MCU -> MCU_VDD
- U1 pad 26: 3V3_MCU -> MCU_VDD
- U1 pad 34: unconnected-(U1-NRST-Pad34) -> WATCHDOG_OUT
- U1 pad 36: unconnected-(U1-PC1-Pad36) -> ESP32_SPI2_MOSI
- U1 pad 39: 3V3_MCU -> MCU_VDD
- U1 pad 52: 3V3_MCU -> MCU_VDD
- U1 pad 56: unconnected-(U1-PA7-Pad56) -> W25q_FLASH_SPI1_MOSI
- U1 pad 59: 3V3_MCU -> MCU_VDD
- U1 pad 73: 3V3_MCU -> MCU_VDD
- U1 pad 83: 3V3_MCU -> MCU_VDD
- U1 pad 94: 3V3_MCU -> MCU_VDD
- U3 pad 1: unconnected-(U3-~{CS}-Pad1) -> W25q_FLASH_SPI1_NSS
- U3 pad 2: unconnected-(U3-DO/IO_{1}-Pad2) -> W25q_FLASH_SPI1_MISO
- U3 pad 3: unconnected-(U3-~{WP}/IO_{2}-Pad3) -> Net-(U3-~{WP}/IO_{2})
- U3 pad 5: unconnected-(U3-DI/IO_{0}-Pad5) -> W25q_FLASH_SPI1_MOSI
- U3 pad 6: unconnected-(U3-CLK-Pad6) -> W25q_FLASH_SPI1_SCK
- U3 pad 7: unconnected-(U3-~{HOLD}/~{RESET}/IO_{3}-Pad7) -> Net-(U3-~{HOLD}/~{RESET}/IO_{3})
- U5 pad 1: 3V3_MCU -> Net-(J1-Pin_1)
- U5 pad 10: unconnected-(U5-IO10-Pad10) -> ESP32_SPI2_NSS
- U5 pad 11: unconnected-(U5-IO20/RXD-Pad11) -> Net-(J14-Pin_1)
- U5 pad 12: unconnected-(U5-IO21/TXD-Pad12) -> Net-(J14-Pin_2)
- U5 pad 13: unconnected-(U5-IO18-Pad13) -> Net-(J12-Pin_2)
- U5 pad 14: unconnected-(U5-IO19-Pad14) -> Net-(J13-Pin_1)
- U5 pad 15: unconnected-(U5-IO3-Pad15) -> GND
- U5 pad 16: unconnected-(U5-IO2-Pad16) -> ESP32_SPI2_MISO
- U5 pad 17: unconnected-(U5-IO1-Pad17) -> ESP32_UART_TX
- U5 pad 18: unconnected-(U5-IO0-Pad18) -> ESP32_UART_RX
- U5 pad 2: unconnected-(U5-EN-Pad2) -> Net-(U5-EN)
- U5 pad 3: unconnected-(U5-IO4-Pad3) -> FSPIHD
- U5 pad 4: unconnected-(U5-IO5-Pad4) -> FSPIWP
- U5 pad 5: unconnected-(U5-IO6-Pad5) -> ESP32_SPI2_SCK
- U5 pad 6: unconnected-(U5-IO7-Pad6) -> ESP32_SPI2_MOSI
- U5 pad 7: unconnected-(U5-IO8-Pad7) -> Net-(LED4-K)
- U5 pad 8: unconnected-(U5-IO9-Pad8) -> Net-(LED3-K)

Commit message: 중간 저장
Parts:
- added C63: 0.1uF/50V, Capacitor_SMD:C_0402_1005Metric, F.Cu at (177.5, 107.1)
- added C64: 0.1uF/50V, Capacitor_SMD:C_0402_1005Metric, F.Cu at (177.5, 109.1)
- added C65: 1uF/16V, Capacitor_SMD:C_0402_1005Metric, F.Cu at (177.5, 111.1)
- added C66: 1uF/16V, Capacitor_SMD:C_0402_1005Metric, F.Cu at (177.5, 113.0)
- added C67: 0.1uF/50V, Capacitor_SMD:C_0603_1608Metric, F.Cu at (172.0, 107.4)
- added IC4: TPS7A2018PDBVR, SamacSys_Parts:SOT95P280X145-5N, F.Cu at (181.4, 108.2)
- added R109: 4.7k/0.063w, Resistor_SMD:R_0402_1005Metric, F.Cu at (168.6, 107.1)
- added R110: 0R/0.063w, Resistor_SMD:R_0402_1005Metric, F.Cu at (177.5, 117.0)
- added R111: 4.7k/0.063w, Resistor_SMD:R_0402_1005Metric, F.Cu at (177.5, 119.0)
- added R112: 10k/0.063w, Resistor_SMD:R_0402_1005Metric, F.Cu at (168.6, 109.1)
- added R113: 10k/0.063w, Resistor_SMD:R_0402_1005Metric, F.Cu at (168.6, 111.1)
- added R114: 10k/0.063w, Resistor_SMD:R_0402_1005Metric, F.Cu at (168.6, 113.1)
- R94: value 10K/0.063w -> 4.7K/0.063w
Connections:
- R108 pad 1: unconnected-(R108-Pad1) -> +3.3V
- R108 pad 2: unconnected-(R108-Pad2) -> Joystick1_Sel
- U10 pad 1: unconnected-(U10-H+-Pad1) -> 1V8
- U10 pad 2: unconnected-(U10-H-Pad2) -> Joystick2_H
- U10 pad 3: unconnected-(U10-H--Pad3) -> GND
- U10 pad 4: unconnected-(U10-V+-Pad4) -> 1V8
- U10 pad 5: unconnected-(U10-V-Pad5) -> Joystick2_V
- U10 pad 6: unconnected-(U10-V--Pad6) -> GND
- U10 pad 7: unconnected-(U10-SEL+-Pad7) -> Joystick2_Sel
- U10 pad 8: unconnected-(U10-SEL--Pad8) -> GND
- U9 pad 1: unconnected-(U9-H+-Pad1) -> 1V8
- U9 pad 2: unconnected-(U9-H-Pad2) -> Joystick1_H
- U9 pad 3: unconnected-(U9-H--Pad3) -> GND
- U9 pad 4: unconnected-(U9-V+-Pad4) -> 1V8
- U9 pad 5: unconnected-(U9-V-Pad5) -> Joystick1_V
- U9 pad 6: unconnected-(U9-V--Pad6) -> GND
- U9 pad 7: unconnected-(U9-SEL+-Pad7) -> Joystick1_Sel
- U9 pad 8: unconnected-(U9-SEL--Pad8) -> GND

Commit message: 중간 수정
Parts:
- added C68: 12pF/50V, Capacitor_SMD:C_0402_1005Metric, F.Cu at (32.8, 112.7)
- added C69: 12pF/50V, Capacitor_SMD:C_0402_1005Metric, F.Cu at (32.8, 114.6)
- added C70: 0.1uF/16V, Capacitor_SMD:C_0402_1005Metric, F.Cu at (23.8, 119.2)
- added C71: 0.1uF/16V, Capacitor_SMD:C_0402_1005Metric, F.Cu at (23.8, 121.2)
- added D11: WS2812B, LED_SMD:LED_WS2812B_PLCC4_5.0x5.0mm_P3.2mm, F.Cu at (13.9, 115.0)
- added D12: WS2812B, LED_SMD:LED_WS2812B_PLCC4_5.0x5.0mm_P3.2mm, F.Cu at (13.9, 121.6)
- added D13: B540C-13-F, SamacSys_Parts:DIOM7959X250N, F.Cu at (76.5, 122.9)
- added D14: B540C-13-F, SamacSys_Parts:DIOM7959X250N, F.Cu at (76.5, 130.0)
- added D2: SS2H10-E3_52T, SamacSys_Parts:DIOM5436X244N, F.Cu at (47.8, 120.0)
- added IC1: TLE8366E_V33, SamacSys_Parts:SOIC127P600X170-9N, F.Cu at (40.3, 114.9)
- added JP1: IF_CAN_END, Jumper:SolderJumper-2_P1.3mm_Open_RoundedPad1.0x1.5mm, F.Cu at (20.2, 120.0)
- added Q10: IRFZ44NSTRLPBF, SamacSys_Parts:IRFZ44NSTRLPBF, F.Cu at (41.0, 99.5)
- added Q11: IRFZ44NSTRLPBF, SamacSys_Parts:IRFZ44NSTRLPBF, F.Cu at (53.4, 99.5)
- added Q12: IRFZ44NSTRLPBF, SamacSys_Parts:IRFZ44NSTRLPBF, F.Cu at (65.8, 99.5)
- added Q13: IRFZ44NSTRLPBF, SamacSys_Parts:IRFZ44NSTRLPBF, F.Cu at (78.2, 99.5)
- added Q8: IRFZ44NSTRLPBF, SamacSys_Parts:IRFZ44NSTRLPBF, F.Cu at (16.1, 99.5)
- added Q9: IRFZ44NSTRLPBF, SamacSys_Parts:IRFZ44NSTRLPBF, F.Cu at (28.5, 99.5)
- added R116: 2K/0.063w, Resistor_SMD:R_0402_1005Metric, F.Cu at (29.9, 112.7)
- added R117: 2K/0.063w, Resistor_SMD:R_0402_1005Metric, F.Cu at (29.9, 114.7)
- added R119: 2K/0.063w, Resistor_SMD:R_0402_1005Metric, F.Cu at (29.9, 116.7)
- added R120: 2K/0.063w, Resistor_SMD:R_0402_1005Metric, F.Cu at (29.9, 118.6)
- added R121: 2K/0.063w, Resistor_SMD:R_0402_1005Metric, F.Cu at (29.9, 120.6)
- added R122: 2K/0.063w, Resistor_SMD:R_0402_1005Metric, F.Cu at (29.9, 122.6)
- added R123: 2K/0.063w, Resistor_SMD:R_0402_1005Metric, F.Cu at (29.9, 124.6)
- added R124: 2K/0.063w, Resistor_SMD:R_0402_1005Metric, F.Cu at (29.9, 126.6)
- added U11: SN65HVD230, Package_SO:SOIC-8_3.9x4.9mm_P1.27mm, F.Cu at (22.2, 115.0)
- added Z1: SZ1SMB5915BT3G, SamacSys_Parts:DIOM5436X247N, F.Cu at (40.1, 120.0)
- L4, L5: footprint Inductor_SMD:L_12x12mm_H6mm -> Inductor_SMD:L_SXN_SMDRI127
- L6: value 3.3uH/1.6A -> SWPA5040S3R3MT; footprint Inductor_SMD:L_12x12mm_H6mm -> Inductor_SMD:L_Sunlord_SWPA5040S
- moved J5 69.6 mm to (60.0, 70.0), turned to -90 degrees
- moved J8 45.1 mm to (145.7, 54.0)
Connections:
- D9 pad 1: GND -> unconnected-(D9-GND-Pad1)
- IC4 pad 2: unconnected-(IC4-GND-Pad2) -> GND
- LED1 pad 1: unconnected-(LED1-K-Pad1) -> BLUE_LED1
- LED1 pad 2: unconnected-(LED1-A-Pad2) -> Net-(LED1-A)
- LED2 pad 1: unconnected-(LED2-K-Pad1) -> BLUE_LED2
- LED2 pad 2: unconnected-(LED2-A-Pad2) -> Net-(LED2-A)
- R113 pad 2: TEMP_I2C_SCL -> I2C1_SCL
- R114 pad 2: TEMP_I2C_SDA -> I2C1_SDA
- U1 pad 10: unconnected-(U1-PC15-Pad10) -> OSC_32_OUT
- U1 pad 195: unconnected-(U1-PB6-Pad195) -> I2C1_SCL
- U1 pad 196: unconnected-(U1-PB7-Pad196) -> I2C1_SDA
- U1 pad 198: unconnected-(U1-PB8-Pad198) -> CAN_RXD
- U1 pad 199: unconnected-(U1-PB9-Pad199) -> CAN_TXD
- U1 pad 54: LTDC_R4 -> unconnected-(U1-PA5-Pad54)
- U1 pad 68: unconnected-(U1-PJ3-Pad68) -> LTDC_R4
- U1 pad 9: unconnected-(U1-PC14-Pad9) -> OSC_32_IN
- U7 pad 1: unconnected-(U7-Pad1) -> Net-(R127-Pad2)
- U7 pad 2: unconnected-(U7A---Pad2) -> Net-(U7A--)
- U7 pad 3: unconnected-(U7A-+-Pad3) -> Net-(U7A-+)
- U7 pad 4: unconnected-(U7A-V--Pad4) -> GND
- U7 pad 5: unconnected-(U7B-+-Pad5) -> Net-(U7B-+)
- U7 pad 6: unconnected-(U7B---Pad6) -> Net-(U7B--)
- U7 pad 7: unconnected-(U7-Pad7) -> Net-(R128-Pad2)
- U7 pad 8: unconnected-(U7A-V+-Pad8) -> +3.3V
- U8 pad 1: unconnected-(U8-Pad1) -> Net-(R131-Pad2)
- U8 pad 2: unconnected-(U8A---Pad2) -> Net-(U8A--)
- U8 pad 3: unconnected-(U8A-+-Pad3) -> Net-(U8A-+)
- U8 pad 4: unconnected-(U8A-V--Pad4) -> GND
- U8 pad 8: unconnected-(U8A-V+-Pad8) -> +3.3V
Other:
- board outline added: 150 x 100 mm
