File: 1.hardware/bldc_motor_controller.kicad_pcb (KiCad board)
At the start: 2 copper layers, 150 x 150 mm, 191 parts, among them IC1 UCC27712QDRQ1, IC3 STWD100NXWY3F, IC4 SN74HC266D, J5 12V-48V Jack, J8 USB_C, Q10 STL130N6F7, Q2 STL130N6F7, Q3 STL130N6F7, Q4 STL130N6F7, Q8 STL130N6F7, Q9 STL130N6F7, U1 STM32H743BITx, U11 SN65HVD230, U3 W25Q128JVS, U5 ESP32-C3-WROOM-02

Commit message: 중간 저장
Parts:
- added C100: 33pF/50V, Capacitor_SMD:C_0402_1005Metric, F.Cu at (188.1, 34.9)
- added C101: 33pF/50V, Capacitor_SMD:C_0402_1005Metric, F.Cu at (188.1, 36.8)
- added C102: 33pF/50V, Capacitor_SMD:C_0402_1005Metric, F.Cu at (188.1, 38.8)
- added C103: 0.22uF/50V, Capacitor_SMD:C_0603_1608Metric, F.Cu at (170.0, 63.7)
- added C104: 0.22uF/50V, Capacitor_SMD:C_0603_1608Metric, F.Cu at (170.0, 66.2)
- added C105: 0.22uF/50V, Capacitor_SMD:C_0603_1608Metric, F.Cu at (174.0, 53.7)
- added C106: 0.22uF/50V, Capacitor_SMD:C_0603_1608Metric, F.Cu at (174.0, 56.2)
- added C107: 0.22uF/50V, Capacitor_SMD:C_0603_1608Metric, F.Cu at (174.0, 58.7)
- added C108: 0.22uF/50V, Capacitor_SMD:C_0603_1608Metric, F.Cu at (174.0, 61.2)
- added C109: 22uF/100V, Capacitor_SMD:C_Elec_8x10.2, F.Cu at (153.8, 32.9)
- added C110: 22uF/100V, Capacitor_SMD:C_Elec_8x10.2, F.Cu at (153.8, 42.7)
- added C111: 22uF/100V, Capacitor_SMD:C_Elec_8x10.2, F.Cu at (153.8, 52.6)
- added C112: 0.22uF/50V, Capacitor_SMD:C_0603_1608Metric, F.Cu at (160.8, 83.6)
- added C113: 0.1uF/50V, Capacitor_SMD:C_0603_1608Metric, F.Cu at (160.8, 86.1)
- added C114: 0.1uF/50V, Capacitor_SMD:C_0603_1608Metric, F.Cu at (160.8, 88.7)
- added C115: 0.1uF/50V, Capacitor_SMD:C_0603_1608Metric, F.Cu at (160.8, 91.2)
- added C116: 0.1uF/50V, Capacitor_SMD:C_0603_1608Metric, F.Cu at (160.8, 93.7)
- added C117: 0.1uF/50V, Capacitor_SMD:C_0603_1608Metric, F.Cu at (164.8, 83.6)
- added C118: 0.1uF/50V, Capacitor_SMD:C_0603_1608Metric, F.Cu at (164.8, 86.1)
- added C119: 0.1uF/50V, Capacitor_SMD:C_0603_1608Metric, F.Cu at (164.8, 88.7)
- added C120: 0.1uF/50V, Capacitor_SMD:C_0603_1608Metric, F.Cu at (164.8, 91.2)
- added C121: 0.1uF/50V, Capacitor_SMD:C_0603_1608Metric, F.Cu at (164.8, 93.7)
- added C122: 39nF/50V, Capacitor_SMD:C_0402_1005Metric, F.Cu at (164.8, 75.3)
- added C123: 39nF/50V, Capacitor_SMD:C_0402_1005Metric, F.Cu at (164.8, 77.2)
- added C124: 39nF/50V, Capacitor_SMD:C_0402_1005Metric, F.Cu at (164.8, 79.2)
- added C2: 2.2uF/100V, Capacitor_SMD:C_Elec_6.3x5.4, F.Cu at (213.0, 55.6)
- added C29: 4.7uF/10V, Capacitor_SMD:C_0603_1608Metric, F.Cu at (194.1, 65.1)
- added C30: 20pF/50V, Capacitor_SMD:C_0402_1005Metric, F.Cu at (212.4, 64.8)
- added C32: 0.1uF/50V, Capacitor_SMD:C_0603_1608Metric, F.Cu at (194.1, 67.6)
- added C34: 20pF/50V, Capacitor_SMD:C_0402_1005Metric, F.Cu at (212.4, 66.8)
- added C35: 0.1uF/50V, Capacitor_SMD:C_0603_1608Metric, F.Cu at (194.1, 70.1)
- added C36: 0.1uF/50V, Capacitor_SMD:C_0603_1608Metric, F.Cu at (194.1, 72.7)
- added C37: 0.1uF/50V, Capacitor_SMD:C_0603_1608Metric, F.Cu at (194.1, 75.2)
- added C38: 0.1uF/50V, Capacitor_SMD:C_0603_1608Metric, F.Cu at (194.1, 77.7)
- added C39: 1uF/16V, Capacitor_SMD:C_0603_1608Metric, F.Cu at (198.1, 65.1)
- added C40: 0.1uF/50V, Capacitor_SMD:C_0603_1608Metric, F.Cu at (198.1, 67.6)
- added C41: 0.1uF/50V, Capacitor_SMD:C_0603_1608Metric, F.Cu at (198.1, 70.1)
- added C42: 0.1uF/50V, Capacitor_SMD:C_0603_1608Metric, F.Cu at (198.1, 72.7)
- added C43: 0.1uF/50V, Capacitor_SMD:C_0603_1608Metric, F.Cu at (198.1, 75.2)
- added C44: 0.1uF/50V, Capacitor_SMD:C_0603_1608Metric, F.Cu at (198.1, 77.7)
- added C45: 0.1uF/50V, Capacitor_SMD:C_0603_1608Metric, F.Cu at (202.1, 65.1)
- added C46: 0.1uF/50V, Capacitor_SMD:C_0603_1608Metric, F.Cu at (202.1, 67.6)
- added C47: 0.1uF/50V, Capacitor_SMD:C_0603_1608Metric, F.Cu at (202.1, 70.1)
- added C48: 0.1uF/50V, Capacitor_SMD:C_0603_1608Metric, F.Cu at (202.1, 72.7)
- added C49: 0.1uF/50V, Capacitor_SMD:C_0603_1608Metric, F.Cu at (202.1, 75.2)
- added C5: 22uF/25V, Capacitor_SMD:C_Elec_5x5.8, F.Cu at (215.1, 31.4)
- added C50: 0.1uF/50V, Capacitor_SMD:C_0603_1608Metric, F.Cu at (202.1, 77.7)
- added C51: 2.2uF/10V, Capacitor_SMD:C_0603_1608Metric, F.Cu at (206.1, 65.1)
- added C52: 0.1uF/50V, Capacitor_SMD:C_0603_1608Metric, F.Cu at (206.1, 67.6)
- added C53: 2.2uF/10V, Capacitor_SMD:C_0603_1608Metric, F.Cu at (206.1, 70.1)
- added C54: 0.1uF/50V, Capacitor_SMD:C_0603_1608Metric, F.Cu at (206.1, 72.7)
- added C55: 0.1uF/50V, Capacitor_SMD:C_0603_1608Metric, F.Cu at (206.1, 75.2)
- added C56: 1uF/16V, Capacitor_SMD:C_0603_1608Metric, F.Cu at (206.1, 77.7)
- added C6: 22uF/25V, Capacitor_SMD:C_Elec_5x5.8, F.Cu at (215.1, 38.2)
- added C77: 0.1uF/50V, Capacitor_SMD:C_0603_1608Metric, F.Cu at (187.5, 81.4)
- added C78: 1uF/10V, Capacitor_SMD:C_0603_1608Metric, F.Cu at (187.5, 83.9)
- added C79: 0.1uF/50V, Capacitor_SMD:C_0603_1608Metric, F.Cu at (174.9, 75.5)
- added C8: 10uF/25V, Capacitor_SMD:C_Elec_4x5.4, F.Cu at (203.8, 58.9)
- added C80: 39nF/50V, Capacitor_SMD:C_0402_1005Metric, F.Cu at (178.3, 75.3)
- added C81: 39nF/50V, Capacitor_SMD:C_0402_1005Metric, F.Cu at (178.3, 77.2)
- added C82: 39nF/50V, Capacitor_SMD:C_0402_1005Metric, F.Cu at (178.3, 79.2)
- added C83: 39nF/50V, Capacitor_SMD:C_0402_1005Metric, F.Cu at (178.3, 81.2)
- added C84: 4.7uF/10V, Capacitor_SMD:C_0603_1608Metric, F.Cu at (170.0, 53.7)
- added C85: 47uF/50V, Capacitor_SMD:C_Elec_6.3x7.7, F.Cu at (172.9, 32.0)
- added C86: 47uF/50V, Capacitor_SMD:C_Elec_6.3x7.7, F.Cu at (172.9, 40.2)
- added C87: 47uF/50V, Capacitor_SMD:C_Elec_6.3x7.7, F.Cu at (172.9, 48.3)
- added C88: 10uF/25V, Capacitor_SMD:C_Elec_4x5.4, F.Cu at (164.2, 30.9)
- added C89: 10uF/25V, Capacitor_SMD:C_Elec_4x5.4, F.Cu at (164.2, 36.7)
- added C90: 10uF/25V, Capacitor_SMD:C_Elec_4x5.4, F.Cu at (164.2, 42.6)
- added C91: 10uF/25V, Capacitor_SMD:C_Elec_4x5.4, F.Cu at (164.2, 48.4)
- added C92: 10uF/25V, Capacitor_SMD:C_Elec_4x5.4, F.Cu at (164.2, 54.3)
- added C93: 10uF/25V, Capacitor_SMD:C_Elec_4x5.4, F.Cu at (164.2, 60.1)
- added C94: 33pF/50V, Capacitor_SMD:C_0402_1005Metric, F.Cu at (188.1, 28.9)
- added C95: 33pF/50V, Capacitor_SMD:C_0402_1005Metric, F.Cu at (188.1, 30.9)
- added C96: 33pF/50V, Capacitor_SMD:C_0402_1005Metric, F.Cu at (188.1, 32.9)
- added C97: 0.22uF/50V, Capacitor_SMD:C_0603_1608Metric, F.Cu at (170.0, 56.2)
- added C98: 0.22uF/50V, Capacitor_SMD:C_0603_1608Metric, F.Cu at (170.0, 58.7)
- added C99: 0.22uF/50V, Capacitor_SMD:C_0603_1608Metric, F.Cu at (170.0, 61.2)
- added D1: SS58c, Diode_SMD:D_SMC, F.Cu at (205.5, 31.8)
- added D12: NSR0240V2, PCM_Diode_SMD_AKL:D_SOD-523, F.Cu at (183.6, 75.9)
- added D13: NSR0240V2, PCM_Diode_SMD_AKL:D_SOD-523, F.Cu at (183.6, 79.2)
- added D2: SS58c, Diode_SMD:D_SMC, F.Cu at (205.5, 39.6)
- added D8: LL4148, PCM_Diode_SMD_AKL:D_MiniMELF, F.Cu at (199.4, 81.0)
- added H1: MountingHole, MountingHole:MountingHole_3.2mm_M3, F.Cu at (196.0, 31.9)
- added H2: MountingHole, MountingHole:MountingHole_3.2mm_M3, F.Cu at (196.0, 39.9)
- added H3: MountingHole, MountingHole:MountingHole_3.2mm_M3, F.Cu at (196.0, 47.8)
- added H4: MountingHole, MountingHole:MountingHole_3.2mm_M3, F.Cu at (196.0, 55.8)
- added LED1: LED_0603_Blue, PCM_LED_SMD_AKL:LED_0603_1608Metric, F.Cu at (194.1, 80.6)
- added LED2: LED_0603_Blue, PCM_LED_SMD_AKL:LED_0603_1608Metric, F.Cu at (194.1, 83.9)
- added LED3: LED_0603_Green_PWR, PCM_LED_SMD_AKL:LED_0603_1608Metric, F.Cu at (194.1, 89.2)
- added LED4: LED_0603_Blue_BLE, PCM_LED_SMD_AKL:LED_0603_1608Metric, F.Cu at (194.1, 92.5)
- added LED5: LED_0603_Red, PCM_LED_SMD_AKL:LED_0603_1608Metric, F.Cu at (194.1, 95.9)
- added R1: 309/0.1w, Resistor_SMD:R_0603_1608Metric, F.Cu at (202.0, 44.7)
- added R10: 10k/0.1w, Resistor_SMD:R_0603_1608Metric, F.Cu at (206.0, 44.7)
- added R106: 10.2R/0.125w, Resistor_SMD:R_0805_2012Metric, F.Cu at (187.7, 75.8)
- added R107: 10.2R/0.125w, Resistor_SMD:R_0805_2012Metric, F.Cu at (187.7, 78.7)
- added R108: 10k/0.063w, Resistor_SMD:R_0402_1005Metric, F.Cu at (183.2, 81.9)
- added R11: 13.7k/0.1w, Resistor_SMD:R_0603_1608Metric, F.Cu at (206.0, 47.2)
- added R12: 10k/0.1w, Resistor_SMD:R_0603_1608Metric, F.Cu at (206.0, 49.7)
- added R13: 13.7k/0.1w, Resistor_SMD:R_0603_1608Metric, F.Cu at (206.0, 52.2)
- added R131: 10k/0.063w, Resistor_SMD:R_0402_1005Metric, F.Cu at (174.3, 87.8)
- added R132: 100/0.1w, Resistor_SMD:R_0603_1608Metric, F.Cu at (174.9, 78.0)
- added R133: 100/0.1w, Resistor_SMD:R_0603_1608Metric, F.Cu at (174.9, 80.5)
- added R136: 100/0.1w, Resistor_SMD:R_0603_1608Metric, F.Cu at (174.9, 83.1)
- added R137: 100/0.1w, Resistor_SMD:R_0603_1608Metric, F.Cu at (174.9, 85.6)
- added R138: 2.2/0.25w, Resistor_SMD:R_1206_3216Metric, F.Cu at (186.8, 54.1)
- added R139: 2.2/0.25w, Resistor_SMD:R_1206_3216Metric, F.Cu at (186.8, 57.4)
- added R14: 10k/0.1w, Resistor_SMD:R_0603_1608Metric, F.Cu at (206.0, 54.8)
- added R140: 2.2/0.25w, Resistor_SMD:R_1206_3216Metric, F.Cu at (186.8, 60.7)
- added R141: 49.9/0.1w, Resistor_SMD:R_0603_1608Metric, F.Cu at (174.0, 63.7)
- added R142: 49.9/0.1w, Resistor_SMD:R_0603_1608Metric, F.Cu at (174.0, 66.2)
- added R143: 49.9/0.1w, Resistor_SMD:R_0603_1608Metric, F.Cu at (178.0, 53.7)
- added R144: 49.9/0.1w, Resistor_SMD:R_0603_1608Metric, F.Cu at (178.0, 56.2)
- added R145: 49.9/0.1w, Resistor_SMD:R_0603_1608Metric, F.Cu at (178.0, 58.7)
- added R146: 49.9/0.1w, Resistor_SMD:R_0603_1608Metric, F.Cu at (178.0, 61.2)
- added R147: 2.2/0.125w, Resistor_SMD:R_0805_2012Metric, F.Cu at (149.4, 59.0)
- added R148: 2.2/0.125w, Resistor_SMD:R_0805_2012Metric, F.Cu at (149.4, 61.9)
- added R149: 2.2/0.125w, Resistor_SMD:R_0805_2012Metric, F.Cu at (149.4, 64.9)
- added R150: 2.2/0.25w, Resistor_SMD:R_1206_3216Metric, F.Cu at (186.8, 64.0)
- added R151: 2.2/0.125w, Resistor_SMD:R_0805_2012Metric, F.Cu at (149.4, 67.8)
- added R152: 2.2/0.25w, Resistor_SMD:R_1206_3216Metric, F.Cu at (186.8, 67.3)
- added R153: 2.2/0.125w, Resistor_SMD:R_0805_2012Metric, F.Cu at (153.8, 59.0)
- added R154: 2.2/0.25w, Resistor_SMD:R_1206_3216Metric, F.Cu at (186.8, 70.6)
- added R155: 2.2/0.125w, Resistor_SMD:R_0805_2012Metric, F.Cu at (153.8, 61.9)
- added R156: 3.3/0.125w, Resistor_SMD:R_0805_2012Metric, F.Cu at (153.8, 64.9)
- added R157: 3.3/0.125w, Resistor_SMD:R_0805_2012Metric, F.Cu at (153.8, 67.8)
- added R158: 3.3/0.125w, Resistor_SMD:R_0805_2012Metric, F.Cu at (158.2, 59.0)
- added R159: 3.3/0.125w, Resistor_SMD:R_0805_2012Metric, F.Cu at (158.2, 61.9)
- added R16: 10k/0.063w, Resistor_SMD:R_0402_1005Metric, F.Cu at (209.6, 64.9)
- added R160: 3.3/0.125w, Resistor_SMD:R_0805_2012Metric, F.Cu at (158.2, 64.9)
- added R161: 3.3/0.125w, Resistor_SMD:R_0805_2012Metric, F.Cu at (158.2, 67.8)
- added R162: 5.1k/0.1w, Resistor_SMD:R_0603_1608Metric, F.Cu at (178.0, 63.7)
- added R163: 5.1k/0.1w, Resistor_SMD:R_0603_1608Metric, F.Cu at (178.0, 66.2)
- added R164: 5.1k/0.1w, Resistor_SMD:R_0603_1608Metric, F.Cu at (182.0, 53.7)
- added R165: 5.1k/0.1w, Resistor_SMD:R_0603_1608Metric, F.Cu at (182.0, 56.2)
- added R166: 5.1k/0.1w, Resistor_SMD:R_0603_1608Metric, F.Cu at (182.0, 58.7)
- added R167: 5.1k/0.1w, Resistor_SMD:R_0603_1608Metric, F.Cu at (182.0, 61.2)
- added R168: 0.01R, Resistor_SMD:R_2512_6332Metric, F.Cu at (182.3, 30.4)
- added R169: 0.01R, Resistor_SMD:R_2512_6332Metric, F.Cu at (182.3, 35.3)
- added R17: 10k/0.063w, Resistor_SMD:R_0402_1005Metric, F.Cu at (209.6, 66.8)
- added R170: 0.01R, Resistor_SMD:R_2512_6332Metric, F.Cu at (182.3, 40.2)
- added R171: 10k/0.063w, Resistor_SMD:R_0402_1005Metric, F.Cu at (148.6, 83.4)
- added R172: 10k/0.063w, Resistor_SMD:R_0402_1005Metric, F.Cu at (148.6, 85.4)
- added R173: 10k/0.063w, Resistor_SMD:R_0402_1005Metric, F.Cu at (148.6, 87.3)
- added R174: 100k/0.063w, Resistor_SMD:R_0402_1005Metric, F.Cu at (148.6, 89.3)
- added R175: 10k/0.063w, Resistor_SMD:R_0402_1005Metric, F.Cu at (148.6, 91.3)
- added R176: 10k/0.063w, Resistor_SMD:R_0402_1005Metric, F.Cu at (148.6, 93.3)
- added R177: 10k/0.063w, Resistor_SMD:R_0402_1005Metric, F.Cu at (148.6, 95.3)
- added R178: 10k/0.063w, Resistor_SMD:R_0402_1005Metric, F.Cu at (151.5, 83.4)
- added R179: 10k/0.063w, Resistor_SMD:R_0402_1005Metric, F.Cu at (151.5, 85.4)
- added R180: 10k/0.063w, Resistor_SMD:R_0402_1005Metric, F.Cu at (151.5, 87.3)
- added R181: 10k/0.063w, Resistor_SMD:R_0402_1005Metric, F.Cu at (151.5, 89.3)
- added R182: 100k/0.063w, Resistor_SMD:R_0402_1005Metric, F.Cu at (151.5, 91.3)
- added R183: 100k/0.063w, Resistor_SMD:R_0402_1005Metric, F.Cu at (151.5, 93.3)
- added R184: 100k/0.063w, Resistor_SMD:R_0402_1005Metric, F.Cu at (151.5, 95.3)
- added R185: 47k/0.125w, Resistor_SMD:R_0402_1005Metric, F.Cu at (154.4, 83.4)
- added R186: 47k/0.125w, Resistor_SMD:R_0402_1005Metric, F.Cu at (154.4, 85.4)
- added R187: 47k/0.125w, Resistor_SMD:R_0402_1005Metric, F.Cu at (154.4, 87.3)
- added R188: 5k/0.063w, Resistor_SMD:R_0402_1005Metric, F.Cu at (154.4, 89.3)
- added R189: 5k/0.063w, Resistor_SMD:R_0402_1005Metric, F.Cu at (154.4, 91.3)
- added R190: 5k/0.063w, Resistor_SMD:R_0402_1005Metric, F.Cu at (154.4, 93.3)
- added R191: 100/0.1w, Resistor_SMD:R_0402_1005Metric, F.Cu at (154.4, 95.3)
- added R192: 100/0.1w, Resistor_SMD:R_0402_1005Metric, F.Cu at (157.3, 83.4)
- added R193: 100/0.1w, Resistor_SMD:R_0402_1005Metric, F.Cu at (157.3, 85.4)
- added R194: 22/0.063w, Resistor_SMD:R_0402_1005Metric, F.Cu at (157.3, 87.3)
- added R195: 22/0.063w, Resistor_SMD:R_0402_1005Metric, F.Cu at (157.3, 89.3)
- added R196: 22/0.063w, Resistor_SMD:R_0402_1005Metric, F.Cu at (157.3, 91.3)
- added R2: 22.1k/0.1w, Resistor_SMD:R_0603_1608Metric, F.Cu at (202.0, 47.2)
- added R26: 0R/0.063w, Resistor_SMD:R_0402_1005Metric, F.Cu at (209.6, 68.8)
- added R27: 0R/0.063w, Resistor_SMD:R_0402_1005Metric, F.Cu at (209.6, 70.8)
- added R3: 360k/0.1w, Resistor_SMD:R_0603_1608Metric, F.Cu at (202.0, 49.7)
- added R31: 2k/0.063w, Resistor_SMD:R_0402_1005Metric, F.Cu at (209.6, 72.8)
- added R35: 2k/0.063w, Resistor_SMD:R_0402_1005Metric, F.Cu at (209.6, 74.8)
- added R39: 10k/0.063w, Resistor_SMD:R_0402_1005Metric, F.Cu at (197.6, 88.6)
- added R4: 30k/0.1w, Resistor_SMD:R_0603_1608Metric, F.Cu at (202.0, 52.2)
- added R44: 0R/0.063w, Resistor_SMD:R_0402_1005Metric, F.Cu at (197.6, 90.5)
- added R45: 0R/0.063w, Resistor_SMD:R_0402_1005Metric, F.Cu at (197.6, 92.5)
- added R46: 120/0.125w, Resistor_SMD:R_0805_2012Metric, F.Cu at (198.4, 97.0)
- added R49: 1k/0.063w, Resistor_SMD:R_0402_1005Metric, F.Cu at (197.6, 94.5)
- added R5: 100k/0.063w, Resistor_SMD:R_0402_1005Metric, F.Cu at (219.4, 52.6)
- added R6: 10k/0.063w, Resistor_SMD:R_0402_1005Metric, F.Cu at (219.4, 54.5)
- added R7: 10k/0.063w, Resistor_SMD:R_0402_1005Metric, F.Cu at (219.4, 56.5)
- added R8: 10k/0.063w, Resistor_SMD:R_0402_1005Metric, F.Cu at (219.4, 58.5)
- added R9: 13.7k/0.1w, Resistor_SMD:R_0603_1608Metric, F.Cu at (202.0, 54.8)
- added TP1: TP_V_input, TestPoint:TestPoint_Pad_D2.0mm, F.Cu at (210.1, 45.5)
- added TP10: TP_JV1, TestPoint:TestPoint_Pad_D2.0mm, F.Cu at (170.8, 84.4)
- added TP11: TP_JV2, TestPoint:TestPoint_Pad_D2.0mm, F.Cu at (170.8, 88.5)
- added TP12: TP_MOTOR_U, TestPoint:TestPoint_Pad_D2.0mm, F.Cu at (179.9, 44.7)
- added TP13: TP_HALL_A, TestPoint:TestPoint_Pad_D2.0mm, F.Cu at (179.9, 48.8)
- added TP14: TP_MOTOR_V, TestPoint:TestPoint_Pad_D2.0mm, F.Cu at (184.0, 44.7)
- added TP15: TP_HALL_B, TestPoint:TestPoint_Pad_D2.0mm, F.Cu at (184.0, 48.8)
- added TP16: TP_MOTOR_W, TestPoint:TestPoint_Pad_D2.0mm, F.Cu at (188.0, 44.7)
- added TP17: TP_HALL_C, TestPoint:TestPoint_Pad_D2.0mm, F.Cu at (188.0, 48.8)
- added TP18: TP_HALL_3x_Sig, TestPoint:TestPoint_Pad_D2.0mm, F.Cu at (149.2, 76.3)
- added TP19: TP_MOTOR1_DIR, TestPoint:TestPoint_Pad_D2.0mm, F.Cu at (149.2, 80.3)
- added TP2: TestPoint, TestPoint:TestPoint_Pad_D2.0mm, F.Cu at (210.1, 49.5)
- added TP20: TP_MOTOR_U_SHUNT_ADC, TestPoint:TestPoint_Pad_D2.0mm, F.Cu at (153.2, 76.3)
- added TP21: TP_MOTOR_V_SHUNT_ADC, TestPoint:TestPoint_Pad_D2.0mm, F.Cu at (153.2, 80.3)
- added TP22: TP_MOTOR_W_SHUNT_ADC, TestPoint:TestPoint_Pad_D2.0mm, F.Cu at (157.3, 76.3)
- added TP23: TP_ZC_UV_1, TestPoint:TestPoint_Pad_D2.0mm, F.Cu at (157.3, 80.3)
- added TP24: TP_ZC_UW_2, TestPoint:TestPoint_Pad_D2.0mm, F.Cu at (161.3, 76.3)
- added TP25: TP_ZC_VW_3, TestPoint:TestPoint_Pad_D2.0mm, F.Cu at (161.3, 80.3)
- added TP3: TP_12V, TestPoint:TestPoint_Pad_D2.0mm, F.Cu at (214.1, 45.5)
- added TP4: TP_1V8, TestPoint:TestPoint_Pad_D2.0mm, F.Cu at (214.1, 49.5)
- added TP5: TP_3V3, TestPoint:TestPoint_Pad_D2.0mm, F.Cu at (218.2, 45.5)
- added TP6: TP_5V, TestPoint:TestPoint_Pad_D2.0mm, F.Cu at (218.2, 49.5)
- added TP7: TP_2V5, TestPoint:TestPoint_Pad_D2.0mm, F.Cu at (210.2, 81.0)
- added TP8: TP_JH2, TestPoint:TestPoint_Pad_D2.0mm, F.Cu at (170.8, 76.3)
- added TP9: TP_JH1, TestPoint:TestPoint_Pad_D2.0mm, F.Cu at (170.8, 80.3)
- added X1: SMD3225-4, PCM_Crystal_AKL:Crystal_SMD_3225-4Pin_3.2x2.5mm, F.Cu at (205.5, 81.3)
- C26: renamed from C27; footprint Capacitor_SMD:C_0402_1005Metric -> Capacitor_SMD:C_0603_1608Metric
- C27: renamed from C35; footprint Capacitor_SMD:C_0402_1005Metric -> Capacitor_SMD:C_0603_1608Metric
- C28: renamed from C66; footprint Capacitor_SMD:C_0402_1005Metric -> Capacitor_SMD:C_0603_1608Metric
- C57: renamed from C50; value 0.1uF/16V -> 0.1uF/50V; footprint Capacitor_SMD:C_0402_1005Metric -> Capacitor_SMD:C_0603_1608Metric
- C58: renamed from C51; value 0.1uF/16V -> 0.1uF/50V; footprint Capacitor_SMD:C_0402_1005Metric -> Capacitor_SMD:C_0603_1608Metric
- C59: renamed from C70; value 0.1uF/16V -> 0.1uF/50V; footprint Capacitor_SMD:C_0402_1005Metric -> Capacitor_SMD:C_0603_1608Metric
- C61: renamed from C71; value 0.1uF/16V -> 0.1uF/50V; footprint Capacitor_SMD:C_0402_1005Metric -> Capacitor_SMD:C_0603_1608Metric
- C62: renamed from C57; value 0.1uF/16V -> 0.1uF/50V; footprint Capacitor_SMD:C_0402_1005Metric -> Capacitor_SMD:C_0603_1608Metric
- C63: renamed from C41; value 0.1uF/16V -> 0.1uF/50V; footprint Capacitor_SMD:C_0402_1005Metric -> Capacitor_SMD:C_0603_1608Metric
- C64: renamed from C58; value 0.1uF/16V -> 0.1uF/50V; footprint Capacitor_SMD:C_0402_1005Metric -> Capacitor_SMD:C_0603_1608Metric
- C66: renamed from C42; value 0.1uF/16V -> 0.1uF/50V; footprint Capacitor_SMD:C_0402_1005Metric -> Capacitor_SMD:C_0603_1608Metric
- C67: renamed from C43; value 0.1uF/16V -> 0.1uF/50V; footprint Capacitor_SMD:C_0402_1005Metric -> Capacitor_SMD:C_0603_1608Metric
- C68: renamed from C44; value 0.1uF/16V -> 0.1uF/50V; footprint Capacitor_SMD:C_0402_1005Metric -> Capacitor_SMD:C_0603_1608Metric
- C69: renamed from C45; value 0.1uF/16V -> 0.1uF/50V; footprint Capacitor_SMD:C_0402_1005Metric -> Capacitor_SMD:C_0603_1608Metric
- C70: renamed from C46; value 0.1uF/16V -> 0.1uF/50V; footprint Capacitor_SMD:C_0402_1005Metric -> Capacitor_SMD:C_0603_1608Metric
- C71: renamed from C47; value 0.1uF/16V -> 0.1uF/50V; footprint Capacitor_SMD:C_0402_1005Metric -> Capacitor_SMD:C_0603_1608Metric
- C73: renamed from C49; value 0.1uF/16V -> 0.1uF/50V; footprint Capacitor_SMD:C_0402_1005Metric -> Capacitor_SMD:C_0603_1608Metric
- R19: renamed from R96; value 10K/0.063w -> 10k/0.063w
- R21: renamed from R94; value 4.7K/0.063w -> 4.7k/0.063w
- R23: renamed from R116; value 2K/0.063w -> 4.7k/0.063w
- R24: renamed from R117; value 2K/0.063w -> 4.7k/0.063w
- R28: renamed from R123; value 2K/0.063w -> 2k/0.063w
- R29: renamed from R121; value 2K/0.063w -> 2k/0.063w
- R30: renamed from R120; value 2K/0.063w -> 2k/0.063w
- R32: renamed from R124; value 2K/0.063w -> 2k/0.063w
- R33: renamed from R122; value 2K/0.063w -> 2k/0.063w
- R34: renamed from R119; value 2K/0.063w -> 2k/0.063w
- R36: renamed from R102; value 4.7K/0.063w -> 4.7k/0.063w
- R37: renamed from R90; value 4.7K/0.063w -> 4.7k/0.063w
- R38: renamed from R91; value 4.7K/0.063w -> 4.7k/0.063w
- R40: renamed from R106; value 4.7K/0.063w -> 4.7k/0.063w
- R41: renamed from R138; value 4.7K/0.063w -> 4.7k/0.063w
- R42: renamed from R92; value NC_4.7K -> NC_4.7k/0.1w
- R43: renamed from R93; value 4.7K -> 4.7k/0.1w
- R47: renamed from R103; value 4.7K/0.063w -> 4.7k/0.063w
- R48: renamed from R104; value 4.7K/0.063w -> 4.7k/0.063w
- renumbered C56 to C1, C26 to C10, C29 to C11, C31 to C12, C33 to C13, C36 to C14, C64 to C15, C72 to C16, C28 to C17, C30 to C18, C34 to C19, C37 to C20, C65 to C21, C76 to C22, C32 to C23, C63 to C24, C77 to C25, C22 to C3, C68 to C31, C69 to C33, C23 to C4, C52 to C60, C59 to C65, C24 to C7, C48 to C72, C38 to C74, C39 to C75, C40 to C76, C25 to C9, D11 to D10, D12 to D11, D3 to D5, D4 to D6, D5 to D7, IC3 to IC2, IC1 to IC4, J5 to J2, J8 to J5, L4 to L2, L1 to L3, L3 to L4, L9 to L5, L5 to L6, L6 to L7, L10 to L8, PS5 to PS1, PS3 to PS2, PS4 to PS3, Q2 to Q6, Q3 to Q7, R84 to R100, R85 to R101, R86 to R102, R87 to R103, R88 to R104, R89 to R105, R12 to R109, R13 to R110, R14 to R111, R15 to R112, R16 to R113, R17 to R114, R18 to R115, R19 to R116, R20 to R117, R21 to R118, R22 to R119, R23 to R120, R24 to R121, R25 to R122, R26 to R123, R27 to R124, R28 to R125, R29 to R126, R30 to R127, R31 to R128, R32 to R129, R33 to R130, R108 to R134, R109 to R135, R111 to R15, R142 to R18, R95 to R20, R110 to R22, R141 to R25, R34 to R50, R35 to R51, R36 to R52, R37 to R53, R38 to R54, R39 to R55, R40 to R56, R41 to R57, R42 to R58, R43 to R59, R44 to R60, R45 to R61, R46 to R62, R47 to R63, R48 to R64, R49 to R65, R50 to R66, R51 to R67, R52 to R68, R53 to R69, R54 to R70, R55 to R71, R56 to R72, R57 to R73, R58 to R74, R59 to R75, R60 to R76, R61 to R77, R62 to R78, R63 to R79, R64 to R80, R65 to R81, R66 to R82, R67 to R83, R68 to R84, R69 to R85, R70 to R86, R71 to R87, R72 to R88, R73 to R89, R74 to R90, R75 to R91, R76 to R92, R77 to R93, R78 to R94, R79 to R95, R80 to R96, R81 to R97, R82 to R98, R83 to R99, U1 to U2, U11 to U3, U5 to U4, U3 to U5
Connections:
- C4 pad 1: Net-(C23-Pad1) -> Net-(C4-Pad1)
- C57 pad 1: 3V3_MCU -> 3V3_ESP32
- C58 pad 1: 3V3_MCU -> 3V3_ESP32
- C60 pad 1: 3V3_MCU -> 3V3_ESP32
- C74 pad 1: 3V3_PWR -> 3V3
- D9 pad 1: unconnected-(D9-GND-Pad1) -> GND
- IC4 pad 1: unconnected-(IC1-LI-Pad1) -> Net-(IC4-LI)
- IC4 pad 2: unconnected-(IC1-HI-Pad2) -> Net-(IC4-HI)
- IC4 pad 3: unconnected-(IC1-VDD-Pad3) -> Net-(IC4-VDD)
- IC4 pad 4: unconnected-(IC1-COM-Pad4) -> GNDPWR
- IC4 pad 5: unconnected-(IC1-LO-Pad5) -> Net-(IC4-LO)
- IC4 pad 6: unconnected-(IC1-HS-Pad6) -> MOTOR_U
- IC4 pad 7: unconnected-(IC1-HO-Pad7) -> Net-(IC4-HO)
- IC4 pad 8: unconnected-(IC1-HB-Pad8) -> Net-(IC4-HB)
- J2 pad 1: Net-(D2-Pad2) -> Net-(D1-A)
- L2 pad 1: Net-(C23-Pad1) -> Net-(C4-Pad1)
- Q6 pad 1: unconnected-(Q2-S_1-Pad1) -> MOTOR_U
- Q6 pad 2: unconnected-(Q2-S_2-Pad2) -> MOTOR_U
- Q6 pad 3: unconnected-(Q2-S_3-Pad3) -> MOTOR_U
- Q6 pad 4: unconnected-(Q2-G-Pad4) -> Net-(Q6-G)
- Q6 pad 5: unconnected-(Q2-D_1-Pad5) -> PWR_INPUT(12V~48V)
- Q6 pad 6: unconnected-(Q2-D_2-Pad6) -> PWR_INPUT(12V~48V)
- Q6 pad 7: unconnected-(Q2-D_3-Pad7) -> PWR_INPUT(12V~48V)
- Q6 pad 8: unconnected-(Q2-D_4-Pad8) -> PWR_INPUT(12V~48V)
- Q6 pad 9: unconnected-(Q2-D_5-Pad9) -> PWR_INPUT(12V~48V)
- Q7 pad 1: unconnected-(Q3-S_1-Pad1) -> Net-(Q7-S_1)
- Q7 pad 2: unconnected-(Q3-S_2-Pad2) -> Net-(Q7-S_1)
- Q7 pad 3: unconnected-(Q3-S_3-Pad3) -> Net-(Q7-S_1)
- Q7 pad 4: unconnected-(Q3-G-Pad4) -> Net-(Q7-G)
- Q7 pad 5: unconnected-(Q3-D_1-Pad5) -> MOTOR_U
- Q7 pad 6: unconnected-(Q3-D_2-Pad6) -> MOTOR_U
- Q7 pad 7: unconnected-(Q3-D_3-Pad7) -> MOTOR_U
- Q7 pad 8: unconnected-(Q3-D_4-Pad8) -> MOTOR_U
- Q7 pad 9: unconnected-(Q3-D_5-Pad9) -> MOTOR_U
- R113 pad 1: LTDC_B0 -> LTDC_B2
- R114 pad 1: LTDC_B1 -> LTDC_B3
- R115 pad 1: LTDC_B2 -> LTDC_B4
- R116 pad 1: LTDC_B3 -> LTDC_B5
- R117 pad 1: LTDC_B4 -> LTDC_B6
- R118 pad 1: LTDC_B5 -> LTDC_B7
- R119 pad 1: LTDC_G0 -> LTDC_G2
- R120 pad 1: LTDC_G1 -> LTDC_G3
- R121 pad 1: LTDC_G2 -> LTDC_G4
- R122 pad 1: LTDC_G3 -> LTDC_G5
- R123 pad 1: LTDC_G4 -> LTDC_G6
- R124 pad 1: LTDC_G5 -> LTDC_G7
- R125 pad 1: LTDC_R0 -> LTDC_R2
- R126 pad 1: LTDC_R1 -> LTDC_R3
- R127 pad 1: LTDC_R2 -> LTDC_R4
- R128 pad 1: LTDC_R3 -> LTDC_R5
- R129 pad 1: LTDC_R4 -> LTDC_R6
- R130 pad 1: LTDC_R5 -> LTDC_R7
- R36 pad 1: Net-(J1-Pin_1) -> 3V3_ESP32
- R37 pad 2: UART_TX -> UART1_TX
- R38 pad 2: UART_RX -> UART1_RX
- R40 pad 1: Net-(J1-Pin_1) -> 3V3_ESP32
- R41 pad 1: Net-(J1-Pin_1) -> 3V3_ESP32
- R47 pad 1: Net-(J1-Pin_1) -> 3V3_ESP32
- R48 pad 1: Net-(J1-Pin_1) -> 3V3_ESP32
- U2 pad 1: unconnected-(U1-PE2-Pad1) -> LED1
- U2 pad 103: MCU_VDD -> 3V3_MCU
- U2 pad 104: ESP32_SPI2_NSS -> unconnected-(U2-PB12-Pad104)
- U2 pad 105: ESP32_SPI2_SCK -> unconnected-(U2-PB13-Pad105)
- U2 pad 106: ESP32_SPI2_MISO -> UART1_TX
- U2 pad 107: unconnected-(U1-PB15-Pad107) -> UART1_RX
- U2 pad 112: unconnected-(U1-PD12-Pad112) -> WS2812_PWM
- U2 pad 115: MCU_VDD -> 3V3_MCU
- U2 pad 118: unconnected-(U1-PJ6-Pad118) -> MOTOR_W_LI
- U2 pad 120: unconnected-(U1-PJ8-Pad120) -> MOTOR_V_LI
- U2 pad 121: unconnected-(U1-PJ9-Pad121) -> MOTOR_W_HI
- U2 pad 123: unconnected-(U1-PJ11-Pad123) -> MOTOR_V_HI
- U2 pad 124: MCU_VDD -> 3V3_MCU
- U2 pad 126: unconnected-(U1-PK0-Pad126) -> MOTOR_U_LI
- U2 pad 127: unconnected-(U1-PK1-Pad127) -> MOTOR_U_HI
- U2 pad 128: unconnected-(U1-PK2-Pad128) -> LTDC_G7
- U2 pad 129: unconnected-(U1-PG2-Pad129) -> HALL_6x_Pulse_Sig
- U2 pad 13: unconnected-(U1-PI11-Pad13) -> LTDC_G6
- U2 pad 130: unconnected-(U1-PG3-Pad130) -> MOTOR_DIR_INTR
- U2 pad 133: unconnected-(U1-PG6-Pad133) -> HALL_C_INTR
- U2 pad 134: unconnected-(U1-PG7-Pad134) -> HALL_B_INTR
- U2 pad 138: unconnected-(U1-PC6-Pad138) -> HALL_A_INTR
- U2 pad 139: unconnected-(U1-PC7-Pad139) -> ZC_VW_3
- U2 pad 140: unconnected-(U1-PC8-Pad140) -> ZC_UW_2
- U2 pad 143: unconnected-(U1-PA9-Pad143) -> ZC_UV_1
- U2 pad 144: unconnected-(U1-PA10-Pad144) -> LTDC_B4
- U2 pad 15: MCU_VDD -> 3V3_MCU
- U2 pad 150: MCU_VDD -> 3V3_MCU
- U2 pad 158: MCU_VDD -> 3V3_MCU
- U2 pad 169: unconnected-(U1-PD5-Pad169) -> ESP32_UART_RX
- U2 pad 171: MCU_VDD -> 3V3_MCU
- U2 pad 172: unconnected-(U1-PD6-Pad172) -> ESP32_UART_TX
- U2 pad 173: unconnected-(U1-PD7-Pad173) -> ESP32_SPI1_MOSI
- U2 pad 175: LTDC_B1 -> unconnected-(U2-PJ13-Pad175)
- U2 pad 178: W25q_FLASH_SPI1_MISO -> ESP32_SPI1_MISO
- U2 pad 179: W25q_FLASH_SPI1_NSS -> ESP32_SPI1_NSS
- U2 pad 180: W25q_FLASH_SPI1_SCK -> ESP32_SPI1_SCK
- U2 pad 181: LTDC_B4 -> unconnected-(U2-PG12-Pad181)
- U2 pad 185: MCU_VDD -> 3V3_MCU
- U2 pad 187: unconnected-(U1-PK4-Pad187) -> TP_RES
- U2 pad 188: unconnected-(U1-PK5-Pad188) -> LTDC_B6
- U2 pad 189: unconnected-(U1-PK6-Pad189) -> LTDC_B7
- U2 pad 19: unconnected-(U1-PI12-Pad19) -> LTDC_HSYNC
- U2 pad 190: unconnected-(U1-PK7-Pad190) -> LTDC_DE
- U2 pad 194: unconnected-(U1-PB5-Pad194) -> TP_INT
- U2 pad 2: unconnected-(U1-PE3-Pad2) -> LED2
- U2 pad 20: unconnected-(U1-PI13-Pad20) -> LTDC_VSYNC
- U2 pad 203: unconnected-(U1-PDR_ON-Pad203) -> GND
- U2 pad 204: MCU_VDD -> 3V3_MCU
- U2 pad 21: unconnected-(U1-PI14-Pad21) -> LTDC_CLK
- U2 pad 22: LTDC_HSYNC -> FMC_A3
- U2 pad 23: LTDC_VSYNC -> FMC_A4
- U2 pad 24: LTDC_CLK -> FMC_A5
- U2 pad 26: MCU_VDD -> 3V3_MCU
- U2 pad 27: FMC_A3 -> W25q_FLASH_QUADSPI_IO3
- U2 pad 28: FMC_A4 -> W25q_FLASH_QUADSPI_IO2
- U2 pad 29: FMC_A5 -> W25q_FLASH_QUADSPI_IO1
- U2 pad 3: LTDC_B0 -> BTN1
- U2 pad 30: unconnected-(U1-PF9-Pad30) -> W25q_FLASH_QUADSPI_IO0
- U2 pad 31: LTDC_DE -> W25q_FLASH_QUADSPI_SCK
- U2 pad 35: LTDC_R5 -> FMC_SDNWE
- U2 pad 36: ESP32_SPI2_MOSI -> Joystick2_V
- U2 pad 38: unconnected-(U1-PC3_C-Pad38) -> FMC_SDCKE0
- U2 pad 39: MCU_VDD -> 3V3_MCU
- U2 pad 4: LTDC_G0 -> BTN2
- U2 pad 42: MCU_VDD -> 3V3_MCU
- U2 pad 43: unconnected-(U1-PA0-Pad43) -> WATCHDOG_PWM
- U2 pad 46: LTDC_R0 -> Joystick2_H
- U2 pad 47: unconnected-(U1-PH3-Pad47) -> Joystick1_V
- U2 pad 48: LTDC_G5 -> LTDC_G4
- U2 pad 49: unconnected-(U1-PH5-Pad49) -> Joystick1_H
- U2 pad 5: LTDC_G1 -> unconnected-(U2-PE6-Pad5)
- U2 pad 52: MCU_VDD -> 3V3_MCU
- U2 pad 54: unconnected-(U1-PA5-Pad54) -> LTDC_R4
- U2 pad 55: unconnected-(U1-PA6-Pad55) -> MOTOR_W_SHUNT_ADC
- U2 pad 56: W25q_FLASH_SPI1_MOSI -> MOTOR_V_SHUNT_ADC
- U2 pad 57: unconnected-(U1-PC4-Pad57) -> MOTOR_U_SHUNT_ADC
- U2 pad 58: FMC_SDCKE0 -> Ext_Voltage
- U2 pad 59: MCU_VDD -> 3V3_MCU
- U2 pad 6: MCU_VDD -> 3V3_MCU
- U2 pad 61: LTDC_R3 -> unconnected-(U2-PB0-Pad61)
- U2 pad 62: unconnected-(U1-PB1-Pad62) -> ADC_TEMP
- U2 pad 65: unconnected-(U1-PJ0-Pad65) -> LTDC_R7
- U2 pad 66: unconnected-(U1-PJ1-Pad66) -> Joystick1_Sel
- U2 pad 67: unconnected-(U1-PJ2-Pad67) -> LTDC_R3
- U2 pad 68: LTDC_R4 -> Joystick2_Sel
- U2 pad 69: unconnected-(U1-PJ4-Pad69) -> LTDC_R5
- U2 pad 73: MCU_VDD -> 3V3_MCU
- U2 pad 83: MCU_VDD -> 3V3_MCU
- U2 pad 90: LTDC_G4 -> W25q_FLASH_QUADSPI_NSS
- U2 pad 91: unconnected-(U1-PB11-Pad91) -> LTDC_G5
- U2 pad 94: MCU_VDD -> 3V3_MCU
- U2 pad 95: unconnected-(U1-PJ5-Pad95) -> LTDC_R6
- U2 pad 96: unconnected-(U1-PH6-Pad96) -> BACK_LIGHT_PWM
- U4 pad 1: Net-(J1-Pin_1) -> 3V3_ESP32
- U4 pad 10: ESP32_SPI2_NSS -> ESP32_SPI1_NSS
- U4 pad 16: ESP32_SPI2_MISO -> ESP32_SPI1_MISO
- U4 pad 5: ESP32_SPI2_SCK -> ESP32_SPI1_SCK
- U4 pad 6: ESP32_SPI2_MOSI -> ESP32_SPI1_MOSI
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
Commit message: 중간 저장
Parts:
- removed the C67 at (298.0, 94.5)
- removed the C67 at (294.3, 69.3)
- removed D12, D13: NSR0240V2, PCM_Diode_SMD_AKL:D_SOD-523
- removed D13: SS54F-HF, SamacSys_Parts:SODFL4626X120N
- removed D14: SMBJ28CA-Q, SamacSys_Parts:DIONM5436X244N
- removed the D2 at (205.5, 39.6)
- removed the D2 at (287.5, 53.6)
- removed the IC4 at (236.3, 112.1)
- removed the IC4 at (244.4, 110.2)
- removed LED1, LED2: LED_0603_Blue, PCM_LED_SMD_AKL:LED_0603_1608Metric
- removed LED3: LED_0603_Green_PWR, PCM_LED_SMD_AKL:LED_0603_1608Metric
- removed LED4: LED_0603_Blue_BLE, PCM_LED_SMD_AKL:LED_0603_1608Metric
- removed LED5: LED_0603_Red, PCM_LED_SMD_AKL:LED_0603_1608Metric
- removed Q4: STL130N6F7, SamacSys_Parts:FERD20U50DJFTR
- removed the R100 at (291.4, 79.3)
- removed the R100 at (291.4, 65.4)
- removed the R112 at (294.5, 98.2)
- removed the R112 at (276.9, 100.2)
- removed the R113 at (294.5, 100.2)
- removed the R113 at (276.9, 102.2)
- removed the R114 at (294.5, 102.2)
- removed the R114 at (276.9, 104.2)
- removed the R99 at (288.5, 83.3)
- removed the R99 at (291.4, 77.3)
- removed X1: SMD3225-4, PCM_Crystal_AKL:Crystal_SMD_3225-4Pin_3.2x2.5mm
- added C67: 0.1uF/50V, Capacitor_SMD:C_0603_1608Metric, F.Cu at (308.2, 92.0)
- added D2: SS58c, Diode_SMD:D_SMC, F.Cu at (270.3, 40.8)
- added D3: SMBJ54CA-Q, SamacSys_Parts:DIONM5436X244N, F.Cu at (260.7, 40.8)
- added D4: B5819WS, SamacSys_Parts:SOD2613X100N, F.Cu at (305.2, 42.2)
- added IC4: UCC27712QDRQ1, SamacSys_Parts:SOIC127P600X175-8N, F.Cu at (248.1, 18.0)
- added IC5: UCC27712QDRQ1, SamacSys_Parts:SOIC127P600X175-8N, F.Cu at (248.1, 24.3)
- added IC6: UCC27712QDRQ1, SamacSys_Parts:SOIC127P600X175-8N, F.Cu at (248.1, 30.5)
- added IC7: SN74HCS266QDRQ1, SamacSys_Parts:SOIC127P600X175-14N, F.Cu at (261.0, 107.2)
- added IC8: SN74HC74PWRG4, SamacSys_Parts:SOP65P640X120-14N, F.Cu at (272.8, 111.0)
- added IC9: SN74LVC3G17DCURG4, SamacSys_Parts:SOP50P310X90-8N, F.Cu at (279.2, 97.2)
- added J1: 12V~48V BAT, Connector_AMASS:AMASS_XT60PW-M_1x02_P7.20mm_Horizontal, F.Cu at (286.1, 24.0)
- added Q11: STL130N6F7, SamacSys_Parts:FERD20U50DJFTR, F.Cu at (246.1, 13.3)
- added R100: 33R/0.063w, Resistor_SMD:R_0402_1005Metric, F.Cu at (300.7, 89.2)
- added R112: 22R/0.063w, Resistor_SMD:R_0402_1005Metric, F.Cu at (213.1, 106.9)
- added R113: 22R/0.063w, Resistor_SMD:R_0402_1005Metric, F.Cu at (213.1, 108.8)
- added R114: 22R/0.063w, Resistor_SMD:R_0402_1005Metric, F.Cu at (216.0, 98.9)
- added R99: 33R/0.063w, Resistor_SMD:R_0402_1005Metric, F.Cu at (297.8, 107.1)
- D8: value LL4148 -> B5819WS; footprint PCM_Diode_SMD_AKL:D_MiniMELF -> SamacSys_Parts:SOD2613X100N
- TP1, TP10, TP11, TP12, TP13, TP14, TP15, TP16, TP17, TP18, TP19, TP20, TP21, TP22, TP23, TP24, TP25, TP3, TP4, TP5, TP6, TP7, TP8, TP9: footprint TestPoint:TestPoint_Pad_D2.0mm -> TestPoint:TestPoint_Pad_D1.5mm
- TP2: value TestPoint -> TP_Ext_Volt; footprint TestPoint:TestPoint_Pad_D2.0mm -> TestPoint:TestPoint_Pad_D1.5mm
- moved TP18 121.9 mm to (270.3, 90.0)
- moved TP19 121.8 mm to (270.3, 93.5)
- moved TP20 121.4 mm to (273.9, 90.0)
- moved TP21 121.3 mm to (273.9, 93.5)
- moved TP22 120.9 mm to (277.4, 90.0)
- moved TP23 120.8 mm to (277.4, 93.5)
- moved TP24 120.4 mm to (281.0, 90.0)
- moved TP25 120.4 mm to (281.0, 93.5)
- moved C122 118.5 mm to (278.4, 108.8)
- moved C123 118.5 mm to (278.4, 110.8)
- moved C124 118.5 mm to (278.4, 112.8)
- moved C112 110.5 mm to (270.5, 96.6)
- moved C113 110.5 mm to (270.5, 99.1)
- moved C114 110.5 mm to (270.5, 101.6)
- moved C115 110.5 mm to (270.5, 104.1)
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Connections:
- Q10 pad 1: unconnected-(Q10-S_1-Pad1) -> MOTOR_W
- Q10 pad 2: unconnected-(Q10-S_2-Pad2) -> MOTOR_W
- Q10 pad 3: unconnected-(Q10-S_3-Pad3) -> MOTOR_W
- Q10 pad 4: unconnected-(Q10-G-Pad4) -> Net-(Q10-G)
- Q10 pad 5: unconnected-(Q10-D_1-Pad5) -> PWR_INPUT(12V~48V)
- Q10 pad 6: unconnected-(Q10-D_2-Pad6) -> PWR_INPUT(12V~48V)
- Q10 pad 7: unconnected-(Q10-D_3-Pad7) -> PWR_INPUT(12V~48V)
- Q10 pad 8: unconnected-(Q10-D_4-Pad8) -> PWR_INPUT(12V~48V)
- Q10 pad 9: unconnected-(Q10-D_5-Pad9) -> PWR_INPUT(12V~48V)
- Q8 pad 1: unconnected-(Q8-S_1-Pad1) -> MOTOR_V
- Q8 pad 2: unconnected-(Q8-S_2-Pad2) -> MOTOR_V
- Q8 pad 3: unconnected-(Q8-S_3-Pad3) -> MOTOR_V
- Q8 pad 4: unconnected-(Q8-G-Pad4) -> Net-(Q8-G)
- Q8 pad 5: unconnected-(Q8-D_1-Pad5) -> PWR_INPUT(12V~48V)
- Q8 pad 6: unconnected-(Q8-D_2-Pad6) -> PWR_INPUT(12V~48V)
- Q8 pad 7: unconnected-(Q8-D_3-Pad7) -> PWR_INPUT(12V~48V)
- Q8 pad 8: unconnected-(Q8-D_4-Pad8) -> PWR_INPUT(12V~48V)
- Q8 pad 9: unconnected-(Q8-D_5-Pad9) -> PWR_INPUT(12V~48V)
- Q9 pad 1: unconnected-(Q9-S_1-Pad1) -> Net-(Q9-S_1)
- Q9 pad 2: unconnected-(Q9-S_2-Pad2) -> Net-(Q9-S_1)
- Q9 pad 3: unconnected-(Q9-S_3-Pad3) -> Net-(Q9-S_1)
- Q9 pad 4: unconnected-(Q9-G-Pad4) -> Net-(Q9-G)
- Q9 pad 5: unconnected-(Q9-D_1-Pad5) -> MOTOR_V
- Q9 pad 6: unconnected-(Q9-D_2-Pad6) -> MOTOR_V
- Q9 pad 7: unconnected-(Q9-D_3-Pad7) -> MOTOR_V
- Q9 pad 8: unconnected-(Q9-D_4-Pad8) -> MOTOR_V
- Q9 pad 9: unconnected-(Q9-D_5-Pad9) -> MOTOR_V
Other:
- copper layers 2 -> 4

Commit message: 풋프린트 연결 완료
Parts:
- removed D8: B5819WS, SamacSys_Parts:SOD2613X100N
- removed IC2: STWD100NXWY3F, SamacSys_Parts:SOT95P280X145-5N
- removed R19: 10k/0.063w, Resistor_SMD:R_0402_1005Metric
- removed R20: 100/0.063w, Resistor_SMD:R_0402_1005Metric
- removed R21: 4.7k/0.063w, Resistor_SMD:R_0402_1005Metric
- removed R22: 0R/0.063w, Resistor_SMD:R_0402_1005Metric
- removed R28, R29, R30, R31, R32, R33, R34, R35: 2k/0.063w, Resistor_SMD:R_0402_1005Metric
- added C125: 0.1uF/50V, Capacitor_SMD:C_0603_1608Metric, F.Cu at (-132.0, 159.6)
- added D12: NSR0240V2, PCM_Diode_SMD_AKL:D_SOD-523, F.Cu at (-122.3, 179.8)
- added D13: NSR0240V2, PCM_Diode_SMD_AKL:D_SOD-523, F.Cu at (-122.3, 183.1)
- added D14: MURA160T3G, SamacSys_Parts_Project:DIOM5226X220N, F.Cu at (-136.6, 88.2)
- added D15: MURA160T3G, SamacSys_Parts_Project:DIOM5226X220N, F.Cu at (-136.6, 92.1)
- added D16: MURA160T3G, SamacSys_Parts_Project:DIOM5226X220N, F.Cu at (-136.6, 95.9)
- added D17: MBRM130LT1G, SamacSys_Parts_Project:MBRM130LT1G, F.Cu at (-130.8, 94.6)
- added D18: MBRM130LT1G, SamacSys_Parts_Project:MBRM130LT1G, F.Cu at (-130.8, 98.2)
- added D19: MBRM130LT1G, SamacSys_Parts_Project:MBRM130LT1G, F.Cu at (-130.8, 101.7)
- added D20: MBRM130LT1G, SamacSys_Parts_Project:MBRM130LT1G, F.Cu at (-130.8, 105.2)
- added D21: MBRM130LT1G, SamacSys_Parts_Project:MBRM130LT1G, F.Cu at (-130.8, 108.8)
- added D22: MBRM130LT1G, SamacSys_Parts_Project:MBRM130LT1G, F.Cu at (-130.8, 112.3)
- added IC1: LMR51610XDBVR, SamacSys_Parts_Project:SOT95P280X145-6N, F.Cu at (-39.9, 76.7)
- added IC3: IS42S32800J-6TLI, SamacSys_Parts_Project:SOP50P1176X120-86N, F.Cu at (-53.7, 169.4)
- added J10: I2C_CONN, Connector_PinSocket_2.54mm:PinSocket_1x04_P2.54mm_Vertical, F.Cu at (-98.3, 147.2)
- added J11: ESP_DBG_CONN, Connector_PinSocket_2.54mm:PinSocket_1x03_P2.54mm_Vertical, F.Cu at (-65.3, 147.2)
- added J12: FPC_LCD_40_CONN, Connector_FFC-FPC:Amphenol_F32Q-1A7x1-11040_1x40-1MP_P0.5mm_Horizontal, F.Cu at (-131.4, 174.8)
- added J14: 2061-603/998-404, ul_2061_603:CONN3_2061-603&slash_998-404_WAG, F.Cu at (-114.6, 74.7)
- added J15: CAN_CONN2, Connector_PinSocket_2.54mm:PinSocket_1x04_P2.54mm_Vertical, F.Cu at (-93.7, 147.2)
- added J16: 2060-452/998-404, ul_2060_452:CONN2_2060-452&slash_998-404_WAG, F.Cu at (-92.5, 93.6)
- added J17: 2060-453/998-404, ul_2060_453:CONN3_2060-453&slash_998-404_WAG, F.Cu at (-106.3, 93.6)
- added J3: DEBUG_CONN, Connector_PinSocket_2.54mm:PinSocket_1x07_P2.54mm_Vertical, F.Cu at (-111.3, 120.7)
- added J4: UART_CONN, Connector_PinSocket_2.54mm:PinSocket_1x04_P2.54mm_Vertical, F.Cu at (-102.9, 147.2)
- added J8: ESP_BOOT_CONN, Connector_PinHeader_2.54mm:PinHeader_1x02_P2.54mm_Vertical, F.Cu at (-64.9, 138.2)
- added J9: CAN_CONN, Connector_JST:JST_SH_SM06B-SRSS-TB_1x06-1MP_P1.00mm_Horizontal, F.Cu at (-70.3, 122.2)
- added L1: SMDRI127-330MT, SamacSys_Parts_Project:SMDRI127330MT, F.Cu at (-56.9, 100.8)
- added L11: SWPA4020S4R7MT, SamacSys_Parts_Project:INDPM4040X200N, F.Cu at (-127.3, 185.9)
- added L9: SWPA4020S4R7MT, SamacSys_Parts_Project:INDPM4040X200N, F.Cu at (-127.3, 180.7)
- added LED1: LED_0603_Blue, PCM_LED_SMD_AKL:LED_0603_1608Metric, F.Cu at (-111.0, 159.0)
- added LED2: LED_0603_Blue, PCM_LED_SMD_AKL:LED_0603_1608Metric, F.Cu at (-111.0, 162.3)
- added LED3: LED_0603_Green_PWR, PCM_LED_SMD_AKL:LED_0603_1608Metric, F.Cu at (-73.6, 127.6)
- added LED4: LED_0603_Blue_BLE, PCM_LED_SMD_AKL:LED_0603_1608Metric, F.Cu at (-73.6, 131.0)
- added LED5: LED_0603_Red, PCM_LED_SMD_AKL:LED_0603_1608Metric, F.Cu at (-73.6, 134.3)
- added PS4: TPS61169DCKR, SamacSys_Parts_Project:SOT65P210X110-5N, F.Cu at (-122.0, 186.4)
- added PS5: TPS61169DCKR, SamacSys_Parts_Project:SOT65P210X110-5N, F.Cu at (-122.0, 189.5)
- added RT1: NCP18XH103F03RB, SamacSys_Parts_Project:THRMC1608X95N, F.Cu at (-45.5, 142.5)
- added S1: TSB008A2518A, SamacSys_Parts_Project:TSB008A2518A, F.Cu at (-121.2, 153.1)
- added S2: TSB008A2518A, SamacSys_Parts_Project:TSB008A2518A, F.Cu at (-121.2, 157.8)
- added S3: TSB008A2518A, SamacSys_Parts_Project:TSB008A2518A, F.Cu at (-73.5, 157.7)
- added S4: TSB008A2518A, SamacSys_Parts_Project:TSB008A2518A, F.Cu at (-121.2, 162.5)
- added S5: SS-12M11G4, SamacSys_Parts_Project:SS12M11G4, F.Cu at (-46.3, 99.1)
- added U1: TL431AIDBZR, SamacSys_Parts_Project:SOT95P237X112-3N, F.Cu at (-111.3, 145.0)
- added U10: TLV9064, Package_SO:TSSOP-14_4.4x5mm_P0.65mm, F.Cu at (-100.9, 186.5)
- added U11: TXS0104EPW, Package_SO:TSSOP-14_4.4x5mm_P0.65mm, F.Cu at (-111.6, 154.1)
- added U7: Hall_Analog_Joystick, Library:Hall_Analog_Joystick, F.Cu at (-50.3, 130.7)
- added U8: Hall_Analog_Joystick, Library:Hall_Analog_Joystick, F.Cu at (-31.2, 130.7)
- added U9: TLV9064, Package_SO:TSSOP-14_4.4x5mm_P0.65mm, F.Cu at (-100.9, 180.0)
- added X1: SMD3225-4, PCM_Crystal_AKL:Crystal_SMD_3225-4Pin_3.2x2.5mm, F.Cu at (-110.9, 140.6)
- added Y1: X1A0000610002, Crystal:Crystal_SMD_2012-2Pin_2.0x1.2mm, F.Cu at (-111.6, 148.7)
- D3: footprint SamacSys_Parts:DIONM5436X244N -> SamacSys_Parts_Project:DIOM5436X244N
- D4, D5, D6, D7: footprint SamacSys_Parts:SOD2613X100N -> SamacSys_Parts_Project:SOD2613X100N
- IC4, IC5, IC6: footprint SamacSys_Parts:SOIC127P600X175-8N -> SamacSys_Parts_Project:SOIC127P600X175-8N
- IC7: footprint SamacSys_Parts:SOIC127P600X175-14N -> SamacSys_Parts_Project:SOIC127P600X175-14N
- IC8: footprint SamacSys_Parts:SOP65P640X120-14N -> SamacSys_Parts_Project:SOP65P640X120-14N
- IC9: footprint SamacSys_Parts:SOP50P310X90-8N -> SamacSys_Parts_Project:SOP50P310X90-8N
- J1: value 12V~48V BAT -> 12V~48V BAT_XT60_MALE
- L6, L7, L8: footprint SamacSys_Parts:INDC2116X100N -> SamacSys_Parts_Project:INDC2116X100N
- PS1, PS2, PS3: footprint SamacSys_Parts:SOT95P280X110-6N -> SamacSys_Parts_Project:SOT95P280X110-6N
- Q10, Q11, Q6, Q7, Q8, Q9: footprint SamacSys_Parts:FERD20U50DJFTR -> SamacSys_Parts_Project:FERD20U50DJFTR
- R147, R148, R149: value 2.2/0.125w -> 2.2/0.25w
- R44, R45: value 0R/0.063w -> NC_0R/0.063w
- moved R18 446.6 mm to (-132.0, 162.1)
- moved C29 446.0 mm to (-144.0, 152.0)
- moved C32 446.0 mm to (-144.0, 154.6)
- moved C35 446.0 mm to (-144.0, 157.1)
- moved C36 446.0 mm to (-144.0, 159.6)
- moved C37 446.0 mm to (-144.0, 162.1)
- moved C38 446.0 mm to (-144.0, 164.6)
- moved C39 446.0 mm to (-144.0, 167.1)
- moved C54 446.0 mm to (-132.0, 152.0)
- moved C55 446.0 mm to (-132.0, 154.6)
- moved C56 446.0 mm to (-132.0, 157.1)
- moved C40 446.0 mm to (-140.0, 152.0)
- moved C41 446.0 mm to (-140.0, 154.6)
- moved C42 446.0 mm to (-140.0, 157.1)
- moved C43 446.0 mm to (-140.0, 159.6)
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Connections:
- net WATCHDOG_OUT renamed Net-(S4-NO)
- R44 pad 1: Net-(J6-Pin_2) -> USB_DM
- R45 pad 1: Net-(J7-Pin_1) -> USB_DP
- U2 pad 119: unconnected-(U2-PJ7-Pad119) -> OE_PIN
- U2 pad 43: WATCHDOG_PWM -> unconnected-(U2-PA0-Pad43)
Other:
- board size 150 x 150 mm -> 150 x 100 mm
