File: 1.hardware/bldc_motor_controller.kicad_pcb (KiCad board)
At the start: 4 copper layers, 150 x 100 mm, 426 parts, among them IC1 LMR51610XDBVR, IC3 IS42S32800J-6TLI, IC4 UCC27712QDRQ1, IC5 UCC27712QDRQ1, IC6 UCC27712QDRQ1, IC7 SN74HCS266QDRQ1, IC8 SN74HC74PWRG4, IC9 SN74LVC3G17DCURG4, J1 12V~48V BAT_XT60_MALE, J10 I2C_CONN, J11 ESP_DBG_CONN, J12 FPC_LCD_40_CONN, J14 2061-603/998-404, J15 CAN_CONN2, J16 2060-452/998-404, J17 2060-453/998-404, J2 12V-48V Jack, J3 DEBUG_CONN, J4 UART_CONN, J5 USB_C, J8 ESP_BOOT_CONN, J9 CAN_CONN, Q10 STL130N6F7, Q11 STL130N6F7, Q6 STL130N6F7, Q7 STL130N6F7, Q8 STL130N6F7, Q9 STL130N6F7, U1 TL431AIDBZR, U10 TLV9064, U11 TXS0104EPW, U2 STM32H743BITx, U3 SN65HVD230, U4 ESP32-C3-WROOM-02, U5 W25Q128JVS, U7 Hall_Analog_Joystick, U8 Hall_Analog_Joystick, U9 TLV9064, X1 SMD3225-4, Y1 X1A0000610002

Commit message: 중간 저장
Parts:
- removed C125: 0.1uF/50V, Capacitor_SMD:C_0603_1608Metric
- removed D22: MBRM130LT1G, SamacSys_Parts_Project:MBRM130LT1G
- removed IC9: SN74LVC3G17DCURG4, SamacSys_Parts_Project:SOP50P310X90-8N
- removed the J8 at (-64.9, 138.2)
- removed L11: SWPA4020S4R7MT, SamacSys_Parts_Project:INDPM4040X200N
- removed Q10, Q11, Q7, Q8, Q9: STL130N6F7, SamacSys_Parts_Project:FERD20U50DJFTR
- removed R182, R183, R184: 100k/0.063w, Resistor_SMD:R_0402_1005Metric
- removed R185, R186, R187: 47k/0.125w, Resistor_SMD:R_0402_1005Metric
- removed R188, R189, R190: 5k/0.063w, Resistor_SMD:R_0402_1005Metric
- removed R191, R192, R193: 100/0.1w, Resistor_SMD:R_0402_1005Metric
- removed R194, R195, R196: 22/0.063w, Resistor_SMD:R_0402_1005Metric
- removed the S1 at (-121.2, 153.1)
- removed TP24: TP_ZC_UW_2, TestPoint:TestPoint_Pad_D1.5mm
- removed TP25: TP_ZC_VW_3, TestPoint:TestPoint_Pad_D1.5mm
- removed U11: TXS0104EPW, Package_SO:TSSOP-14_4.4x5mm_P0.65mm
- removed the U5 at (-55.5, 184.5)
- removed the U8 at (-31.2, 130.7)
- added D8: PRTR5V0U2X, Package_TO_SOT_SMD:SOT-143, F.Cu at (-12.5, 131.5)
- added IC2: IS42S32800J-6TLI, SamacSys_Parts_Project:SOP50P1176X120-86N, F.Cu at (-87.2, 94.2)
- added J6: ESP_BOOT_CONN, Connector_PinHeader_2.54mm:PinHeader_1x02_P2.54mm_Vertical, F.Cu at (-9.90, 123.8)
- added J7: CAN_CONN, Connector_JST:JST_SH_SM06B-SRSS-TB_1x06-1MP_P1.00mm_Horizontal, F.Cu at (-17.6, 125.3)
- added L10: SWPA4020S4R7MT, SamacSys_Parts_Project:INDPM4040X200N, F.Cu at (-42.1, 122.3)
- added Q1: STL130N6F7, SamacSys_Parts_Project:FERD20U50DJFTR, F.Cu at (-70.5, 38.7)
- added Q2: STL130N6F7, SamacSys_Parts_Project:FERD20U50DJFTR, F.Cu at (-64.9, 38.7)
- added Q3: STL130N6F7, SamacSys_Parts_Project:FERD20U50DJFTR, F.Cu at (-59.3, 38.7)
- added Q4: STL130N6F7, SamacSys_Parts_Project:FERD20U50DJFTR, F.Cu at (-53.7, 38.7)
- added Q5: STL130N6F7, SamacSys_Parts_Project:FERD20U50DJFTR, F.Cu at (-48.1, 38.7)
- added R19: 4.7k/0.063w, Resistor_SMD:R_0402_1005Metric, F.Cu at (-43.4, 91.4)
- added R20: 120/0.1w, Resistor_SMD:R_0603_1608Metric, F.Cu at (-46.8, 93.8)
- added R21: 10K/0.063w, Resistor_SMD:R_0402_1005Metric, F.Cu at (-43.4, 93.4)
- added R22: 0R/0.063w, Resistor_SMD:R_0402_1005Metric, F.Cu at (-43.4, 95.4)
- added R28: 4.7k/0.063w, Resistor_SMD:R_0402_1005Metric, F.Cu at (-17.5, 120.5)
- added R29: 4.7k/0.063w, Resistor_SMD:R_0402_1005Metric, F.Cu at (-14.6, 112.5)
- added R30: NC_4.7k/0.1w, Resistor_SMD:R_0402_1005Metric, F.Cu at (-14.6, 114.5)
- added R31: 4.7k/0.1w, Resistor_SMD:R_0402_1005Metric, F.Cu at (-14.6, 116.5)
- added R32: NC_0R/0.063w, Resistor_SMD:R_0402_1005Metric, F.Cu at (-14.6, 118.5)
- added R33: NC_0R/0.063w, Resistor_SMD:R_0402_1005Metric, F.Cu at (-14.6, 120.5)
- added R34: 120/0.125w, Resistor_SMD:R_0805_2012Metric, F.Cu at (-8.14, 134.1)
- added R35: 4.7k/0.063w, Resistor_SMD:R_0402_1005Metric, F.Cu at (-11.7, 112.5)
- added S3: TSB008A2518A, SamacSys_Parts_Project:TSB008A2518A, F.Cu at (-39.0, 105.4)
- added U4: SN65HVD230, Package_SO:SOIC-8_3.9x4.9mm_P1.27mm, F.Cu at (-18.8, 132.5)
- added U6: W25Q128JVS, Package_SO:SOIC-8_5.3x5.3mm_P1.27mm, F.Cu at (-89.0, 109.3)
- C10: value 0.01uF/100V -> 0.1uF/100V
- C11: value 22uF/10V -> 0.01uF/100V; footprint Capacitor_SMD:C_0603_1608Metric -> Capacitor_SMD:C_0402_1005Metric
- C12, C14, C16, C18, C20, C22: value 10uF/25V -> 22uF/10V
- C13, C15, C17, C19, C21: value 22uF/10V -> 10uF/25V
- C23: value 0.1uF/50V -> 10uF/25V
- C29: value 4.7uF/10V -> 0.1uF/50V
- C3: value 30pF/50V -> 22uF/25V; footprint Capacitor_SMD:C_0603_1608Metric -> Capacitor_SMD:C_Elec_5x5.8
- C30: value 20pF/50V -> 4.7uF/10V; footprint Capacitor_SMD:C_0402_1005Metric -> Capacitor_SMD:C_0603_1608Metric
- C31: value 12pF/50V -> 20pF/50V
- C32: value 0.1uF/50V -> 12pF/50V; footprint Capacitor_SMD:C_0603_1608Metric -> Capacitor_SMD:C_0402_1005Metric
- C33: value 12pF/50V -> 0.1uF/50V; footprint Capacitor_SMD:C_0402_1005Metric -> Capacitor_SMD:C_0603_1608Metric
- C34: value 20pF/50V -> 12pF/50V
- C35: value 0.1uF/50V -> 20pF/50V; footprint Capacitor_SMD:C_0603_1608Metric -> Capacitor_SMD:C_0402_1005Metric
- C39: value 1uF/16V -> 0.1uF/50V
- C4: value 0.22uF/100V -> 30pF/50V
- C41: value 0.1uF/50V -> 1uF/16V
- C6: value 22uF/25V -> 0.22uF/100V; footprint Capacitor_SMD:C_Elec_5x5.8 -> Capacitor_SMD:C_0603_1608Metric
- C60, C65, C72: value 2.2uF/6.3V -> 0.1uF/50V
- C62, C67: value 0.1uF/50V -> 2.2uF/6.3V
- C7: value 100uF/100V -> 10uF/25V; footprint Capacitor_THT:CP_Radial_Tantal_D8.0mm_P5.00mm -> Capacitor_SMD:C_Elec_4x5.4
- C74: value 4.7uF/10V -> 2.2uF/6.3V
- C75: value 1uF/50V -> 0.1uF/50V
- C76: value 1uF/50V -> 4.7uF/10V
- C77: value 0.1uF/50V -> 1uF/50V
- C78: value 1uF/10V -> 1uF/50V
- C8: value 10uF/25V -> 47uF/100V; footprint Capacitor_SMD:C_Elec_4x5.4 -> Capacitor_SMD:C_Elec_10x10.2
- C80: value 39nF/50V -> 1uF/10V; footprint Capacitor_SMD:C_0402_1005Metric -> Capacitor_SMD:C_0603_1608Metric
- C81: value 39nF/50V -> 0.1uF/50V; footprint Capacitor_SMD:C_0402_1005Metric -> Capacitor_SMD:C_0603_1608Metric
- C9: value 0.1uF/100V -> 47uF/100V; footprint Capacitor_SMD:C_0402_1005Metric -> Capacitor_SMD:C_Elec_10x10.2
- D11: value WS2812B -> NSR0240V2; footprint LED_SMD:LED_WS2812B_PLCC4_5.0x5.0mm_P3.2mm -> PCM_Diode_SMD_AKL:D_SOD-523
- D13: value NSR0240V2 -> MURA160T3G; footprint PCM_Diode_SMD_AKL:D_SOD-523 -> SamacSys_Parts_Project:DIOM5226X220N
- D16: value MURA160T3G -> MBRM130LT1G; footprint SamacSys_Parts_Project:DIOM5226X220N -> SamacSys_Parts_Project:MBRM130LT1G
- D9: value PRTR5V0U2X -> WS2812B; footprint Package_TO_SOT_SMD:SOT-143 -> LED_SMD:LED_WS2812B_PLCC4_5.0x5.0mm_P3.2mm
- IC3: value IS42S32800J-6TLI -> UCC27712QDRQ1; footprint SamacSys_Parts_Project:SOP50P1176X120-86N -> SamacSys_Parts_Project:SOIC127P600X175-8N
- IC6: value UCC27712QDRQ1 -> SN74HCS266QDRQ1; footprint SamacSys_Parts_Project:SOIC127P600X175-8N -> SamacSys_Parts_Project:SOIC127P600X175-14N
- IC7: value SN74HCS266QDRQ1 -> SN74HC74PWRG4; footprint SamacSys_Parts_Project:SOIC127P600X175-14N -> SamacSys_Parts_Project:SOP65P640X120-14N
- IC8: value SN74HC74PWRG4 -> SN74LVC3G17DCURG4; footprint SamacSys_Parts_Project:SOP65P640X120-14N -> SamacSys_Parts_Project:SOP50P310X90-8N
- J11: value ESP_DBG_CONN -> EXTRA_SPI3_CONN; footprint Connector_PinSocket_2.54mm:PinSocket_1x03_P2.54mm_Vertical -> Connector_PinSocket_2.54mm:PinSocket_1x06_P2.54mm_Vertical
- J9: value CAN_CONN -> ESP_DBG_CONN; footprint Connector_JST:JST_SH_SM06B-SRSS-TB_1x06-1MP_P1.00mm_Horizontal -> Connector_PinSocket_2.54mm:PinSocket_1x03_P2.54mm_Vertical
- R100, R101, R102, R103, R104, R105, R97, R98, R99: value 33R/0.063w -> 22R/0.063w
- R106, R107: value 10.2R/0.125w -> 22R/0.063w; footprint Resistor_SMD:R_0805_2012Metric -> Resistor_SMD:R_0402_1005Metric
- R108: value 10k/0.063w -> 22R/0.063w
- R119: value 22R/0.063w -> 10k/0.063w
- R120, R122: value 22R/0.063w -> 100/0.1w; footprint Resistor_SMD:R_0402_1005Metric -> Resistor_SMD:R_0603_1608Metric
- R121: value 22R/0.063w -> 4.7k/0.063w
- R123, R124, R125: value 22R/0.063w -> 2.2/0.25w; footprint Resistor_SMD:R_0402_1005Metric -> Resistor_SMD:R_1206_3216Metric
- R126, R127, R128, R129, R130: value 22R/0.063w -> 49.9/0.1w; footprint Resistor_SMD:R_0402_1005Metric -> Resistor_SMD:R_0603_1608Metric
- R131: value 10k/0.063w -> 49.9/0.1w; footprint Resistor_SMD:R_0402_1005Metric -> Resistor_SMD:R_0603_1608Metric
- R132, R133: value 100/0.1w -> 2.2/0.25w; footprint Resistor_SMD:R_0603_1608Metric -> Resistor_SMD:R_0805_2012Metric
- R134: value 4.7k/0.063w -> 2.2/0.25w; footprint Resistor_SMD:R_0402_1005Metric -> Resistor_SMD:R_0805_2012Metric
- R135: value 4.7k/0.063w -> 2.2/0.25w; footprint Resistor_SMD:R_0402_1005Metric -> Resistor_SMD:R_1206_3216Metric
- R136: value 100/0.1w -> 2.2/0.125w; footprint Resistor_SMD:R_0603_1608Metric -> Resistor_SMD:R_0805_2012Metric
- R137: value 100/0.1w -> 2.2/0.25w; footprint Resistor_SMD:R_0603_1608Metric -> Resistor_SMD:R_1206_3216Metric
- R138, R140: value 2.2/0.25w -> 2.2/0.125w; footprint Resistor_SMD:R_1206_3216Metric -> Resistor_SMD:R_0805_2012Metric
- R141, R142, R143, R144, R145, R146: value 49.9/0.1w -> 3.3/0.125w; footprint Resistor_SMD:R_0603_1608Metric -> Resistor_SMD:R_0805_2012Metric
- R147, R148, R149: value 2.2/0.25w -> 5.1k/0.1w; footprint Resistor_SMD:R_0805_2012Metric -> Resistor_SMD:R_0603_1608Metric
- R15: value 4.7k/0.063w -> 10k/0.063w
- R150, R152: value 2.2/0.25w -> 5.1k/0.1w; footprint Resistor_SMD:R_1206_3216Metric -> Resistor_SMD:R_0603_1608Metric
- R151: value 2.2/0.125w -> 5.1k/0.1w; footprint Resistor_SMD:R_0805_2012Metric -> Resistor_SMD:R_0603_1608Metric
- R153, R155: value 2.2/0.125w -> 0.01R; footprint Resistor_SMD:R_0805_2012Metric -> Resistor_SMD:R_2512_6332Metric
- R154: value 2.2/0.25w -> 0.01R; footprint Resistor_SMD:R_1206_3216Metric -> Resistor_SMD:R_2512_6332Metric
- R156, R157, R158, R160, R161: value 3.3/0.125w -> 10k/0.063w; footprint Resistor_SMD:R_0805_2012Metric -> Resistor_SMD:R_0402_1005Metric
- R159: value 3.3/0.125w -> 100k/0.063w; footprint Resistor_SMD:R_0805_2012Metric -> Resistor_SMD:R_0402_1005Metric
- R16: value 10k/0.063w -> 4.7k/0.063w
- R162, R163, R164, R165, R166: value 5.1k/0.1w -> 10k/0.063w; footprint Resistor_SMD:R_0603_1608Metric -> Resistor_SMD:R_0402_1005Metric
- R167: value 5.1k/0.1w -> 100k/0.063w; footprint Resistor_SMD:R_0603_1608Metric -> Resistor_SMD:R_0402_1005Metric
- R168, R169: value 0.01R -> 100k/0.063w; footprint Resistor_SMD:R_2512_6332Metric -> Resistor_SMD:R_0402_1005Metric
- R170: value 0.01R -> 47k/0.125w; footprint Resistor_SMD:R_2512_6332Metric -> Resistor_SMD:R_0402_1005Metric
- R171, R172: value 10k/0.063w -> 47k/0.125w
- R173, R175: value 10k/0.063w -> 5k/0.063w
- R174: value 100k/0.063w -> 5k/0.063w
- R176, R177, R178: value 10k/0.063w -> 100/0.1w
- R179, R180, R181: value 10k/0.063w -> 22/0.063w
- R18: value 120/0.1w -> 4.7k/0.063w; footprint Resistor_SMD:R_0603_1608Metric -> Resistor_SMD:R_0402_1005Metric
- R23: value 4.7k/0.063w -> 0R/0.063w
- R25: value 10K/0.063w -> 4.7k/0.063w
- R26: value 0R/0.063w -> 4.7k/0.063w
- R27: value 0R/0.063w -> 10k/0.063w
- R37: value 4.7k/0.063w -> 1k/0.063w
- R38, R40, R41, R47, R48: value 4.7k/0.063w -> 33R/0.063w
- R39: value 10k/0.063w -> 33R/0.063w
- R42: value NC_4.7k/0.1w -> 33R/0.063w
- R43: value 4.7k/0.1w -> 33R/0.063w
- R44, R45: value NC_0R/0.063w -> 33R/0.063w
- R46: value 120/0.125w -> 33R/0.063w; footprint Resistor_SMD:R_0805_2012Metric -> Resistor_SMD:R_0402_1005Metric
- R49: value 1k/0.063w -> 33R/0.063w
- R94, R95: value 33R/0.063w -> 10.2R/0.125w; footprint Resistor_SMD:R_0402_1005Metric -> Resistor_SMD:R_0805_2012Metric
- R96: value 33R/0.063w -> 10k/0.063w
- TP10: value TP_JV1 -> TP_MOTOR_U
- TP11: value TP_JV2 -> TP_HALL_A
- TP12: value TP_MOTOR_U -> TP_MOTOR_V
- TP13: value TP_HALL_A -> TP_HALL_B
- TP14: value TP_MOTOR_V -> TP_MOTOR_W
- TP15: value TP_HALL_B -> TP_HALL_C
- TP16: value TP_MOTOR_W -> TP_HALL_3x_Sig
- TP17: value TP_HALL_C -> TP_MOTOR1_DIR
- TP18: value TP_HALL_3x_Sig -> TP_MOTOR_U_SHUNT_ADC
- TP19: value TP_MOTOR1_DIR -> TP_MOTOR_V_SHUNT_ADC
- TP2: value TP_Ext_Volt -> TP_12V
- TP20: value TP_MOTOR_U_SHUNT_ADC -> TP_MOTOR_W_SHUNT_ADC
- TP21: value TP_MOTOR_V_SHUNT_ADC -> TP_ZC_UV_1
- TP22: value TP_MOTOR_W_SHUNT_ADC -> TP_ZC_UW_2
- TP23: value TP_ZC_UV_1 -> TP_ZC_VW_3
- TP3: value TP_12V -> TP_Ext_Volt
- TP8: value TP_JH2 -> TP_JH1
- TP9: value TP_JH1 -> TP_JV1
- U3: value SN65HVD230 -> TXS0104EPW; footprint Package_SO:SOIC-8_3.9x4.9mm_P1.27mm -> Package_SO:TSSOP-14_4.4x5mm_P0.65mm
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- renumbered J15 to J10, J14 to J13, J16 to J14, J17 to J15, J10 to J8, S5 to S1, S3 to S5, U4 to U5, U7 to U8
Connections:
- C100 pad 1: Net-(IC4-LI) -> Net-(IC3-LI)
- C101 pad 1: Net-(IC5-LI) -> Net-(IC4-LI)
- C102 pad 1: Net-(IC6-LI) -> Net-(IC5-LI)
- C103 pad 1: Net-(IC4-HB) -> Net-(IC3-HB)
- C104 pad 1: Net-(IC5-HB) -> Net-(IC4-HB)
- C105 pad 1: Net-(IC6-HB) -> Net-(IC5-HB)
- C106 pad 1: Net-(IC4-HB) -> Net-(IC3-HB)
- C107 pad 1: Net-(IC5-HB) -> Net-(IC4-HB)
- C108 pad 1: Net-(IC6-HB) -> Net-(IC5-HB)
- C11 pad 1: 1V8 -> PWR_INPUT(12V~48V)
- C11 pad 2: GND -> GNDPWR
- C112 pad 1: Net-(IC8-~{1CLR}) -> Net-(IC7-~{1CLR})
- C113 pad 1: Net-(IC9-1A) -> Net-(IC8-1A)
- C12 pad 1: Net-(PS1-VIN) -> 1V8
- C13 pad 1: 3V3 -> Net-(PS1-VIN)
- C14 pad 1: Net-(PS2-VIN) -> 3V3
- C15 pad 1: 5V -> Net-(PS2-VIN)
- C16 pad 1: Net-(PS3-VIN) -> 5V
- C17 pad 1: 1V8 -> Net-(PS3-VIN)
- C18 pad 1: Net-(PS1-VIN) -> 1V8
- C19 pad 1: 3V3 -> Net-(PS1-VIN)
- C20 pad 1: Net-(PS2-VIN) -> 3V3
- C21 pad 1: 5V -> Net-(PS2-VIN)
- C22 pad 1: Net-(PS3-VIN) -> 5V
- C23 pad 1: Net-(PS1-VIN) -> Net-(PS3-VIN)
- C24 pad 1: Net-(PS2-VIN) -> Net-(PS1-VIN)
- C25 pad 1: Net-(PS3-VIN) -> Net-(PS2-VIN)
- C26 pad 1: Net-(PS1-SW) -> Net-(PS3-VIN)
- C26 pad 2: Net-(PS1-VBST) -> GND
- C27 pad 1: Net-(PS2-SW) -> Net-(PS1-SW)
- C27 pad 2: Net-(PS2-VBST) -> Net-(PS1-VBST)
- C28 pad 1: Net-(PS3-SW) -> Net-(PS2-SW)
- C28 pad 2: Net-(PS3-VBST) -> Net-(PS2-VBST)
- C29 pad 1: 3V3_MCU -> Net-(PS3-SW)
- C29 pad 2: GND -> Net-(PS3-VBST)
- C3 pad 1: Net-(C3-Pad1) -> 12V
- C3 pad 2: GNDPWR -> GND
- C30 pad 1: RCC_IN -> 3V3_MCU
- C31 pad 1: OSC_32_IN -> RCC_IN
- C32 pad 1: 3V3_MCU -> OSC_32_IN
- C33 pad 1: OSC_32_OUT -> 3V3_MCU
- C34 pad 1: RCC_OUT -> OSC_32_OUT
- C35 pad 1: 3V3_MCU -> RCC_OUT
- C37 pad 1: ADC_VREF_2V5 -> 3V3_MCU
- C39 pad 1: ADC_VREF_2V5 -> 3V3_MCU
- C40 pad 1: 3V3_MCU -> ADC_VREF_2V5
- C41 pad 1: Net-(S4-NO) -> ADC_VREF_2V5
- C48 pad 1: 3V3_MCU -> Net-(S4-NO)
- C57 pad 1: 3V3_ESP32 -> 3V3_MCU
- C58 pad 1: 3V3_ESP32 -> 5V
- C59 pad 1: 5V -> 3V3_ESP32
- C6 pad 1: 12V -> Net-(C6-Pad1)
- C6 pad 2: GND -> GNDPWR
- C62 pad 1: 3V3_MCU -> 3V3_ESP32
- C63 pad 1: 3V3_MCU -> 5V
- C7 pad 1: PWR_INPUT(12V~48V) -> 12V
- C7 pad 2: GNDPWR -> GND
- C74 pad 1: 3V3 -> 3V3_MCU
- C75 pad 1: LEDA -> 3V3_MCU
- C76 pad 1: LEDA -> 3V3
- C77 pad 1: 3V3 -> LEDA
- C78 pad 1: 3V3 -> LEDA
- C79 pad 1: ADC_TEMP -> 3V3
- C8 pad 1: 12V -> PWR_INPUT(12V~48V)
- C8 pad 2: GND -> GNDPWR
- C80 pad 1: Joystick2_H -> 3V3
- C81 pad 1: Joystick1_H -> ADC_TEMP
- C82 pad 1: Joystick1_V -> Joystick_H
- C83 pad 1: Joystick2_V -> Joystick_V
- C85 pad 1: Net-(IC4-VDD) -> Net-(IC3-VDD)
- C86 pad 1: Net-(IC5-VDD) -> Net-(IC4-VDD)
- C87 pad 1: Net-(IC6-VDD) -> Net-(IC5-VDD)
- C88 pad 1: Net-(IC4-VDD) -> Net-(IC3-VDD)
- C89 pad 1: Net-(IC5-VDD) -> Net-(IC4-VDD)
- C90 pad 1: Net-(IC6-VDD) -> Net-(IC5-VDD)
- C91 pad 1: Net-(IC4-VDD) -> Net-(IC3-VDD)
- C92 pad 1: Net-(IC5-VDD) -> Net-(IC4-VDD)
- C93 pad 1: Net-(IC6-VDD) -> Net-(IC5-VDD)
- C94 pad 1: Net-(IC4-HI) -> Net-(IC3-HI)
- C95 pad 1: Net-(IC5-HI) -> Net-(IC4-HI)
- C96 pad 1: Net-(IC6-HI) -> Net-(IC5-HI)
- C97 pad 1: Net-(IC4-VDD) -> Net-(IC3-VDD)
- C98 pad 1: Net-(IC5-VDD) -> Net-(IC4-VDD)
- C99 pad 1: Net-(IC6-VDD) -> Net-(IC5-VDD)
- D10 pad 2: Net-(D10-DOUT) -> unconnected-(D10-DOUT-Pad2)
- D10 pad 4: WS2812_PWM -> Net-(D10-DIN)
- D11 pad 1: 5V -> LEDA
- D11 pad 2: unconnected-(D11-DOUT-Pad2) -> Net-(D11-A)
- D13 pad 1: LEDA -> Net-(IC3-HB)
- D13 pad 2: Net-(D13-A) -> Net-(D13-Pad2)
- D16 pad 1: Net-(IC6-HB) -> Net-(D16-Pad1)
- D16 pad 2: Net-(D16-Pad2) -> Net-(Q1-G)
- D17 pad 2: Net-(Q6-G) -> Net-(Q2-G)
- D18 pad 2: Net-(Q7-G) -> Net-(Q3-G)
- D19 pad 2: Net-(Q8-G) -> Net-(Q4-G)
- D20 pad 2: Net-(Q9-G) -> Net-(Q5-G)
- D21 pad 2: Net-(Q10-G) -> Net-(Q6-G)
- D3 pad 1: Net-(C4-Pad1) -> Net-(C6-Pad1)
- D4 pad 2: Net-(C3-Pad1) -> Net-(C4-Pad1)
- D9 pad 1: GND -> 5V
- D9 pad 2: USB_DP -> Net-(D10-DIN)
- D9 pad 3: USB_DM -> GND
- D9 pad 4: USB_VBUS -> WS2812_PWM
- IC3 pad 1: 3V3_MCU -> Net-(IC3-LI)
- IC3 pad 2: SDRAM_DQ0 -> Net-(IC3-HI)
- IC3 pad 3: 3V3_MCU -> Net-(IC3-VDD)
- IC3 pad 4: SDRAM_DQ1 -> GNDPWR
- IC3 pad 5: SDRAM_DQ2 -> Net-(IC3-LO)
- IC3 pad 6: GND -> MOTOR_U
- IC3 pad 7: SDRAM_DQ3 -> Net-(IC3-HO)
- IC3 pad 8: SDRAM_DQ4 -> Net-(IC3-HB)
- IC4 pad 6: MOTOR_U -> MOTOR_V
- IC5 pad 6: MOTOR_V -> MOTOR_W
- IC6 pad 1: Net-(IC6-LI) -> HALL_A
- IC6 pad 2: Net-(IC6-HI) -> HALL_B
- IC6 pad 3: Net-(IC6-VDD) -> Net-(IC6-1Y)
- IC6 pad 4: GNDPWR -> HALL_3x_Sig
- IC6 pad 5: Net-(IC6-LO) -> Net-(IC6-1Y)
- IC6 pad 6: MOTOR_W -> HALL_C
- IC6 pad 7: Net-(IC6-HO) -> GND
- IC6 pad 8: Net-(IC6-HB) -> HALL_3x_Sig
- IC7 pad 1: HALL_A -> Net-(IC7-~{1CLR})
- IC7 pad 10: HALL_6x_Pulse_Sig -> unconnected-(IC7-2~{PRE}-Pad10)
- IC7 pad 2: HALL_B -> HALL_A
- IC7 pad 3: Net-(IC7-1Y) -> HALL_B
- IC7 pad 4: HALL_3x_Sig -> 5V
- IC7 pad 5: Net-(IC7-1Y) -> MOTOR_DIR
- IC7 pad 6: HALL_C -> unconnected-(IC7-1~{Q}-Pad6)
- IC7 pad 8: HALL_3x_Sig -> unconnected-(IC7-2~{Q}-Pad8)
- IC7 pad 9: HALL_3x_Late_Sig -> unconnected-(IC7-2Q-Pad9)
- IC8 pad 1: Net-(IC8-~{1CLR}) -> Net-(IC8-1A)
- IC8 pad 2: HALL_A -> unconnected-(IC8-3Y-Pad2)
- IC8 pad 3: HALL_B -> unconnected-(IC8-2A-Pad3)
- IC8 pad 4: 5V -> GND
- IC8 pad 5: MOTOR_DIR -> unconnected-(IC8-2Y-Pad5)
- IC8 pad 7: GND -> HALL_3x_Late_Sig
- IC8 pad 8: unconnected-(IC8-2~{Q}-Pad8) -> 5V
- J11 pad 1: Net-(J11-Pin_1) -> 3V3
- J11 pad 2: Net-(J11-Pin_2) -> EXTRA_SPI3_SCK
- J11 pad 3: GND -> EXTRA_SPI3_MISO
- J13 pad 1: MOTOR_U -> MOTOR_W
- J13 pad 2: MOTOR_U -> MOTOR_W
- J13 pad 5: MOTOR_W -> MOTOR_U
- J13 pad 6: MOTOR_W -> MOTOR_U
- J14 pad 1: 5V -> GND
- J14 pad 2: 5V -> GND
- J14 pad 3: GND -> 5V
- J14 pad 4: GND -> 5V
- J15 pad 1: HALL_A -> HALL_C
- J15 pad 2: HALL_A -> HALL_C
- J15 pad 5: HALL_C -> HALL_A
- J15 pad 6: HALL_C -> HALL_A
- J8 pad 1: +3.3V -> 3V3
- J9 pad 1: PWR_INPUT(5V~24V) -> Net-(J9-Pin_1)
- J9 pad 2: PWR_INPUT(5V~24V) -> Net-(J9-Pin_2)
- J9 pad 3: CANH -> GND
- L2 pad 1: Net-(C4-Pad1) -> Net-(C6-Pad1)
- L9 pad 2: Net-(D13-A) -> Net-(D11-A)
- PS4 pad 1: Net-(D12-A) -> Net-(D11-A)
- PS5 pad 1: Net-(D13-A) -> Net-(D12-A)
- Q6 pad 1: MOTOR_U -> Net-(Q6-S_1)
- Q6 pad 2: MOTOR_U -> Net-(Q6-S_1)
- Q6 pad 3: MOTOR_U -> Net-(Q6-S_1)
- Q6 pad 5: PWR_INPUT(12V~48V) -> MOTOR_W
- Q6 pad 6: PWR_INPUT(12V~48V) -> MOTOR_W
- Q6 pad 7: PWR_INPUT(12V~48V) -> MOTOR_W
- Q6 pad 8: PWR_INPUT(12V~48V) -> MOTOR_W
- Q6 pad 9: PWR_INPUT(12V~48V) -> MOTOR_W
- R100 pad 1: FMC_D26 -> LTDC_HSYNC
- R100 pad 2: SDRAM_DQ26 -> LCD_HS
- R101 pad 1: FMC_D27 -> LTDC_B2
- R101 pad 2: SDRAM_DQ27 -> LCD_B0
- R102 pad 1: FMC_D28 -> LTDC_B3
- R102 pad 2: SDRAM_DQ28 -> LCD_B1
- R103 pad 1: FMC_D29 -> LTDC_B4
- R103 pad 2: SDRAM_DQ29 -> LCD_B2
- R104 pad 1: FMC_D30 -> LTDC_B5
- R104 pad 2: SDRAM_DQ30 -> LCD_B3
- R105 pad 1: FMC_D31 -> LTDC_B6
- R105 pad 2: SDRAM_DQ31 -> LCD_B4
- R106 pad 1: LEDK1 -> LTDC_B7
- R106 pad 2: GND -> LCD_B5
- R107 pad 1: LEDK2 -> LTDC_G2
- R107 pad 2: GND -> LCD_G0
- R108 pad 1: 3V3 -> LTDC_G3
- R108 pad 2: LCD_DISP -> LCD_G1
- R109 pad 1: LTDC_DE -> LTDC_G4
- R109 pad 2: LCD_DE -> LCD_G2
- R110 pad 1: LTDC_CLK -> LTDC_G5
- R110 pad 2: LCD_PCLK -> LCD_G3
- R111 pad 1: LTDC_VSYNC -> LTDC_G6
- R111 pad 2: LCD_VS -> LCD_G4
- R112 pad 1: LTDC_HSYNC -> LTDC_G7
- R112 pad 2: LCD_HS -> LCD_G5
- R113 pad 1: LTDC_B2 -> LTDC_R2
- R113 pad 2: LCD_B0 -> LCD_R0
- R114 pad 1: LTDC_B3 -> LTDC_R3
- R114 pad 2: LCD_B1 -> LCD_R1
- R115 pad 1: LTDC_B4 -> LTDC_R4
- R115 pad 2: LCD_B2 -> LCD_R2
- R116 pad 1: LTDC_B5 -> LTDC_R5
- R116 pad 2: LCD_B3 -> LCD_R3
- R117 pad 1: LTDC_B6 -> LTDC_R6
- R117 pad 2: LCD_B4 -> LCD_R4
- R118 pad 1: LTDC_B7 -> LTDC_R7
- R118 pad 2: LCD_B5 -> LCD_R5
- R119 pad 1: LTDC_G2 -> GND
- R119 pad 2: LCD_G0 -> ADC_TEMP
- R120 pad 1: LTDC_G3 -> Joystick_H
- R120 pad 2: LCD_G1 -> Net-(U8-H)
- R121 pad 1: LTDC_G4 -> +3.3V
- R121 pad 2: LCD_G2 -> Joystick_Sel
- R122 pad 1: LTDC_G5 -> Net-(U8-V)
- R122 pad 2: LCD_G3 -> Joystick_V
- R123 pad 1: LTDC_G6 -> Net-(IC3-VDD)
- R123 pad 2: LCD_G4 -> 12V
- R124 pad 1: LTDC_G7 -> Net-(IC4-VDD)
- R124 pad 2: LCD_G5 -> 12V
- R125 pad 1: LTDC_R2 -> Net-(IC5-VDD)
- R125 pad 2: LCD_R0 -> 12V
- R126 pad 1: LTDC_R3 -> Net-(IC3-LI)
- R126 pad 2: LCD_R1 -> MOTOR_U_LI
- R127 pad 1: LTDC_R4 -> Net-(IC3-HI)
- R127 pad 2: LCD_R2 -> MOTOR_U_HI
- R128 pad 1: LTDC_R5 -> Net-(IC4-LI)
- R128 pad 2: LCD_R3 -> MOTOR_V_LI
- R129 pad 1: LTDC_R6 -> Net-(IC4-HI)
- R129 pad 2: LCD_R4 -> MOTOR_V_HI
- R130 pad 1: LTDC_R7 -> Net-(IC5-LI)
- R130 pad 2: LCD_R5 -> MOTOR_W_LI
- R131 pad 1: GND -> Net-(IC5-HI)
- R131 pad 2: ADC_TEMP -> MOTOR_W_HI
- R132 pad 1: Joystick2_H -> Net-(D13-Pad2)
- R132 pad 2: Net-(U8-H) -> Net-(IC3-VDD)
- R133 pad 1: Joystick1_H -> Net-(D14-Pad2)
- R133 pad 2: Net-(U7-H) -> Net-(IC4-VDD)
- R134 pad 1: +3.3V -> Net-(D15-Pad2)
- R134 pad 2: Joystick1_Sel -> Net-(IC5-VDD)
- R135 pad 1: +3.3V -> Net-(D16-Pad1)
- R135 pad 2: Joystick2_Sel -> Net-(IC3-HO)
- R136 pad 1: Net-(U7-V) -> Net-(D17-Pad1)
- R136 pad 2: Joystick1_V -> Net-(IC3-LO)
- R137 pad 1: Net-(U8-V) -> Net-(D18-Pad1)
- R137 pad 2: Joystick2_V -> Net-(IC4-HO)
- R138 pad 1: Net-(IC4-VDD) -> Net-(D19-Pad1)
- R138 pad 2: 12V -> Net-(IC4-LO)
- R139 pad 1: Net-(IC5-VDD) -> Net-(D20-Pad1)
- R139 pad 2: 12V -> Net-(IC5-HO)
- R140 pad 1: Net-(IC6-VDD) -> Net-(D21-Pad1)
- R140 pad 2: 12V -> Net-(IC5-LO)
- R141 pad 1: Net-(IC4-LI) -> Net-(Q1-G)
- R141 pad 2: MOTOR_U_LI -> Net-(IC3-HO)
- R142 pad 1: Net-(IC4-HI) -> Net-(Q2-G)
- R142 pad 2: MOTOR_U_HI -> Net-(IC3-LO)
- R143 pad 1: Net-(IC5-LI) -> Net-(Q3-G)
- R143 pad 2: MOTOR_V_LI -> Net-(IC4-HO)
- R144 pad 1: Net-(IC5-HI) -> Net-(Q4-G)
- R144 pad 2: MOTOR_V_HI -> Net-(IC4-LO)
- R145 pad 1: Net-(IC6-LI) -> Net-(Q5-G)
- R145 pad 2: MOTOR_W_LI -> Net-(IC5-HO)
- R146 pad 1: Net-(IC6-HI) -> Net-(Q6-G)
- R146 pad 2: MOTOR_W_HI -> Net-(IC5-LO)
- R147 pad 1: Net-(D14-Pad2) -> Net-(Q1-G)
- R147 pad 2: Net-(IC4-VDD) -> MOTOR_U
- R148 pad 1: Net-(D15-Pad2) -> Net-(Q2-G)
- R148 pad 2: Net-(IC5-VDD) -> GNDPWR
- R149 pad 1: Net-(D16-Pad2) -> Net-(Q3-G)
- R149 pad 2: Net-(IC6-VDD) -> MOTOR_V
- R15 pad 1: DEBUG_3V3 -> BTN1
- R15 pad 2: GND -> 3V3_MCU
- R150 pad 1: Net-(D17-Pad1) -> Net-(Q4-G)
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
Commit message: 중간 저장
Parts:
- removed C12, C18: 22uF/10V, Capacitor_SMD:C_0603_1608Metric
- removed C13, C19: 10uF/25V, Capacitor_SMD:C_0603_1608Metric
- removed C24, C27: 0.1uF/50V, Capacitor_SMD:C_0603_1608Metric
- removed D5: B5819WS, SamacSys_Parts_Project:SOD2613X100N
- removed L6: MPL2016S2R2MHT, SamacSys_Parts_Project:INDC2116X100N
- removed LED3: LED_0603_Green_PWR, PCM_LED_SMD_AKL:LED_0603_1608Metric
- removed PS1: TPS563201DDCT, SamacSys_Parts_Project:SOT95P280X110-6N
- removed R153, R154, R155: 0.01R, Resistor_SMD:R_2512_6332Metric
- removed R24: 4.7k/0.063w, Resistor_SMD:R_0402_1005Metric
- removed TP4: TP_1V8, TestPoint:TestPoint_Pad_D1.5mm
- added C125: 0.1uF/50V, Capacitor_SMD:C_0603_1608Metric, F.Cu at (38.2, 97.0)
- added C126: 1uF/16V, Capacitor_SMD:C_0603_1608Metric, F.Cu at (-26.6, 145.4)
- added C128: 1uF/16V, Capacitor_SMD:C_0603_1608Metric, F.Cu at (-20.6, 145.4)
- added IC11: TLV74018PDBVR, SamacSys_Parts_Project:SOT95P280X145-5N, F.Cu at (-23.6, 145.5)
- added IC9: SN74LVC3G17DCURG4, SamacSys_Parts_Project:SOP50P310X90-8N, F.Cu at (38.8, 94.1)
- L7: value MPL2016S2R2MHT -> MPL2520S2R2MHT; footprint SamacSys_Parts_Project:INDC2116X100N -> Inductor_SMD:L_1008_2520Metric
- L8: value MPL2016S3R3MHT -> MPL2520S2R2MHT; footprint SamacSys_Parts_Project:INDC2116X100N -> Inductor_SMD:L_1008_2520Metric
- R10: value 10k/0.1w -> 0.01R; footprint Resistor_SMD:R_0603_1608Metric -> Resistor_SMD:R_2512_6332Metric
- R135, R137, R139: value 2.2/0.25w -> 2.2/0.125w; footprint Resistor_SMD:R_1206_3216Metric -> Resistor_SMD:R_0805_2012Metric
- R4: value 30k/0.1w -> 20k/0.1w
- R6: value 10k/0.063w -> 0.01R; footprint Resistor_SMD:R_0402_1005Metric -> Resistor_SMD:R_2512_6332Metric
- R9: value 13.7k/0.1w -> 0.01R; footprint Resistor_SMD:R_0603_1608Metric -> Resistor_SMD:R_2512_6332Metric
- moved C110 285.0 mm to (193.9, 91.4), turned to 90 degrees
- moved C109 282.1 mm to (193.9, 56.4), turned to 90 degrees
- moved C111 282.1 mm to (194.0, 73.8), turned to 90 degrees
- moved R36 279.7 mm to (265.1, 154.8)
- moved Q1 276.9 mm to (205.7, 58.5), turned to 90 degrees
- moved C59 271.9 mm to (241.2, 154.5)
- moved C60 271.9 mm to (241.2, 157.0)
- moved C62 271.9 mm to (241.2, 162.0)
- moved R35 271.9 mm to (258.7, 141.0)
- moved R136 267.6 mm to (175.6, 74.7), turned to 180 degrees
- moved Q3 267.6 mm to (205.7, 76.0), turned to 90 degrees
- moved Q2 266.7 mm to (200.5, 65.4), turned to -90 degrees
- moved R141 263.2 mm to (175.6, 67.0), turned to 180 degrees
- moved R142 263.2 mm to (175.6, 72.7), turned to 180 degrees
- moved Q5 259.6 mm to (205.7, 93.4), turned to 90 degrees
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Connections:
- C10 pad 2: GNDPWR -> MOTOR_U_SHUNT_M
- C109 pad 2: GNDPWR -> MOTOR_U_SHUNT_M
- C11 pad 2: GNDPWR -> MOTOR_U_SHUNT_M
- C110 pad 2: GNDPWR -> MOTOR_U_SHUNT_M
- C111 pad 2: GNDPWR -> MOTOR_U_SHUNT_M
- C4 pad 2: GNDPWR -> MOTOR_U_SHUNT_M
- C48 pad 1: Net-(S4-NO) -> Net-(S4-COM)
- C6 pad 2: GNDPWR -> MOTOR_U_SHUNT_M
- C8 pad 2: GNDPWR -> MOTOR_U_SHUNT_M
- C9 pad 2: GNDPWR -> MOTOR_U_SHUNT_M
- D3 pad 2: GNDPWR -> MOTOR_U_SHUNT_M
- IC3 pad 4: GNDPWR -> MOTOR_U_SHUNT_M
- IC4 pad 4: GNDPWR -> MOTOR_U_SHUNT_M
- IC5 pad 4: GNDPWR -> MOTOR_U_SHUNT_M
- J1 pad 1: Net-(D2-A) -> MOTOR_U_SHUNT_M
- J1 pad 2: GNDPWR -> Net-(D2-A)
- J10 pad 4: GNDPWR -> MOTOR_U_SHUNT_M
- J2 pad 2: GNDPWR -> MOTOR_U_SHUNT_M
- J2 pad 3: GNDPWR -> MOTOR_U_SHUNT_M
- J7 pad 5: GNDPWR -> MOTOR_U_SHUNT_M
- J7 pad 6: GNDPWR -> MOTOR_U_SHUNT_M
- L5 pad 1: GNDPWR -> MOTOR_U_SHUNT_M
- Q2 pad 1: Net-(Q2-S_1) -> MOTOR_U_SHUNT_P
- Q2 pad 2: Net-(Q2-S_1) -> MOTOR_U_SHUNT_P
- Q2 pad 3: Net-(Q2-S_1) -> MOTOR_U_SHUNT_P
- Q4 pad 1: Net-(Q4-S_1) -> MOTOR_V_SHUNT_P
- Q4 pad 2: Net-(Q4-S_1) -> MOTOR_V_SHUNT_P
- Q4 pad 3: Net-(Q4-S_1) -> MOTOR_V_SHUNT_P
- Q6 pad 1: Net-(Q6-S_1) -> MOTOR_W_SHUNT_P
- Q6 pad 2: Net-(Q6-S_1) -> MOTOR_W_SHUNT_P
- Q6 pad 3: Net-(Q6-S_1) -> MOTOR_W_SHUNT_P
- R10 pad 1: GND -> MOTOR_W_SHUNT_P
- R10 pad 2: Net-(PS1-VFB) -> MOTOR_U_SHUNT_M
- R148 pad 2: GNDPWR -> MOTOR_U_SHUNT_M
- R150 pad 2: GNDPWR -> MOTOR_U_SHUNT_M
- R152 pad 2: GNDPWR -> MOTOR_U_SHUNT_M
- R164 pad 1: MOTOR_V_SHUNT_M -> MOTOR_U_SHUNT_M
- R166 pad 1: MOTOR_W_SHUNT_M -> MOTOR_U_SHUNT_M
- R4 pad 1: GNDPWR -> MOTOR_U_SHUNT_M
- R5 pad 1: GNDPWR -> MOTOR_U_SHUNT_M
- R6 pad 1: Net-(PS1-EN) -> MOTOR_U_SHUNT_P
- R6 pad 2: Net-(PS1-VIN) -> MOTOR_U_SHUNT_M
- R9 pad 1: Net-(PS1-VFB) -> MOTOR_V_SHUNT_P
- R9 pad 2: Net-(PS1-SW) -> MOTOR_U_SHUNT_M
- S4 pad 1: GND -> Net-(S4-COM)
- S4 pad 2: Net-(S4-NO) -> GND
- U2 pad 34: Net-(S4-NO) -> Net-(S4-COM)
Routing:
- net USB_DM: track 0.00 -> 77.0 mm
- net USB_DP: track 0.00 -> 76.4 mm
- net Net-(LED4-K): track 0.00 -> 36.7 mm, vias 0 -> 2
- net Net-(U2-PA12): track 0.00 -> 35.9 mm
- net Net-(U2-PA11): track 0.00 -> 34.7 mm
- net Net-(LED5-K): track 0.00 -> 32.6 mm, vias 0 -> 2
- net Net-(D1-K): track 0.00 -> 29.1 mm
- net Net-(U5-IO19): track 0.00 -> 26.2 mm
- net Net-(U5-IO18): track 0.00 -> 24.6 mm
- net ESP_BOOT: track 0.00 -> 24.6 mm, vias 0 -> 1
- net Net-(J5-CC1): track 0.00 -> 19.4 mm, vias 0 -> 2
- net W25q_FLASH_QUADSPI_IO1: track 0.00 -> 17.0 mm, vias 0 -> 2
- net Net-(IC1-SW): track 0.00 -> 15.9 mm
- net W25q_FLASH_QUADSPI_IO3: track 0.00 -> 15.7 mm
- net W25q_FLASH_QUADSPI_IO2: track 0.00 -> 15.6 mm, vias 0 -> 2
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Other:
- board size 150 x 100 mm -> 180 x 100 mm

Commit message: 중간 저장
Parts:
- removed C109, C110, C111: 22uF/100V, Capacitor_SMD:C_Elec_8x10.2
- removed C2: 2.2uF/100V, Capacitor_SMD:C_Elec_6.3x5.4
- removed C20, C22: 22uF/10V, Capacitor_SMD:C_0603_1608Metric
- removed C86, C87: 47uF/50V, Capacitor_SMD:C_Elec_6.3x7.7
- removed R135, R136, R137, R138, R139, R140: 2.2/0.125w, Resistor_SMD:R_0805_2012Metric
- added C12: 10uF/50V, Capacitor_SMD:C_1206_3216Metric, F.Cu at (87.3, 69.4)
- added C13: 22uF/25V, Capacitor_SMD:C_1206_3216Metric, F.Cu at (104.1, 88.9)
- added C18: 2.2uF/100V, Capacitor_SMD:C_1210_3225Metric, F.Cu at (49.2, 31.6)
- added H5: MountingHole, MountingHole:MountingHole_2.5mm, F.Cu at (155.0, 54.0)
- added H6: MountingHole, MountingHole:MountingHole_2.5mm, F.Cu at (155.0, 130.0)
- added H7: MountingHole, MountingHole:MountingHole_2.5mm, F.Cu at (79.0, 130.0)
- C14, C16: value 22uF/10V -> 22uF/25V; footprint Capacitor_SMD:C_0603_1608Metric -> Capacitor_SMD:C_1206_3216Metric
- C15, C17, C21, C23: value 10uF/25V -> 10uF/50V; footprint Capacitor_SMD:C_0603_1608Metric -> Capacitor_SMD:C_1206_3216Metric
- C3, C5: footprint Capacitor_SMD:C_Elec_5x5.8 -> Capacitor_SMD:C_1206_3216Metric
- C7: value 10uF/25V -> 22uF/25V; footprint Capacitor_SMD:C_Elec_4x5.4 -> Capacitor_SMD:C_1206_3216Metric
- C80: value 1uF/10V -> 1uF/50V
- C88, C89, C90, C91, C92, C93: value 10uF/25V -> 10uF/50V; footprint Capacitor_SMD:C_Elec_4x5.4 -> Capacitor_SMD:C_1206_3216Metric
- moved C93 239.7 mm to (162.5, 59.7)
- moved C89 223.3 mm to (145.9, 50.1)
- moved C90 223.2 mm to (145.9, 53.5)
- moved C92 223.1 mm to (145.9, 60.2)
- moved C16 60.3 mm to (122.1, 47.1), turned to 0 degrees
- moved C14 56.2 mm to (122.1, 43.8), turned to 0 degrees
- moved C5 26.6 mm to (104.1, 82.2), turned to 0 degrees
- moved C85 26.2 mm to (124.2, 73.0), turned to -90 degrees
- moved D7 22.5 mm to (82.5, 73.8), turned to 90 degrees
- moved C88 20.5 mm to (145.9, 46.8), turned to 0 degrees
- moved C17 20.3 mm to (80.9, 77.2), turned to 180 degrees
- moved C23 18.3 mm to (81.0, 79.5), turned to 180 degrees
- moved TP5 17.7 mm to (98.2, 87.5)
- moved C26 16.7 mm to (81.8, 81.5), turned to 180 degrees
- moved C91 16.4 mm to (145.9, 56.9), turned to 0 degrees
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Connections:
- C14 pad 1: 3V3 -> 5V
- C5 pad 1: 12V -> 3V3
- C85 pad 1: Net-(IC3-VDD) -> 12V
- D16 pad 1: Net-(D16-Pad1) -> Net-(IC3-HO)
- D17 pad 1: Net-(D17-Pad1) -> Net-(IC3-LO)
- D18 pad 1: Net-(D18-Pad1) -> Net-(IC4-HO)
- D19 pad 1: Net-(D19-Pad1) -> Net-(IC4-LO)
- D20 pad 1: Net-(D20-Pad1) -> Net-(IC5-HO)
- D21 pad 1: Net-(D21-Pad1) -> Net-(IC5-LO)
- U2 pad 137: unconnected-(U2-VDD33_USB-Pad137) -> 3V3_MCU

Commit message: 중간 저장
Parts:
- moved R133 270.8 mm to (175.1, 74.9), turned to 180 degrees
- moved R144 266.4 mm to (182.8, 80.9)
- moved R143 266.2 mm to (182.9, 72.7)
- moved C105 248.9 mm to (189.0, 6.27)
- moved D15 248.9 mm to (202.8, 14.5)
- moved R134 248.9 mm to (152.3, 33.7)
- moved R145 248.9 mm to (163.3, 33.7)
- moved R146 248.9 mm to (163.3, 36.6)
- moved R151 248.9 mm to (197.0, 11.3)
- moved R152 248.9 mm to (197.0, 13.8)
- moved C96 248.6 mm to (168.1, 94.9), turned to 180 degrees
- moved D21 248.0 mm to (185.6, 96.8)
- moved C102 247.9 mm to (168.1, 91.0), turned to 180 degrees
- moved C95 247.8 mm to (168.1, 80.8), turned to 180 degrees
- moved D20 247.7 mm to (185.6, 88.8)
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Connections:
- J10 pad 1: PWR_INPUT(5V~24V) -> PWR_INPUT(12V~48V)
- J7 pad 1: PWR_INPUT(5V~24V) -> PWR_INPUT(12V~48V)
- J7 pad 2: PWR_INPUT(5V~24V) -> PWR_INPUT(12V~48V)
Routing:
- net MOTOR_U: track 0.00 -> 48.9 mm, vias 0 -> 2
- net MOTOR_V: track 0.00 -> 48.3 mm, vias 0 -> 2
- net Net-(Q1-G): track 0.00 -> 32.0 mm
- net Net-(Q3-G): track 0.00 -> 31.2 mm
- net Net-(Q4-G): track 0.00 -> 23.2 mm
- net Net-(Q2-G): track 0.00 -> 22.8 mm
- net Net-(IC4-VDD): track 0.00 -> 16.1 mm, vias 0 -> 2
- net Net-(IC3-VDD): track 0.00 -> 15.9 mm, vias 0 -> 2
- net Net-(IC3-HO): track 0.00 -> 15.1 mm
- net Net-(IC4-LO): track 0.00 -> 14.9 mm
- net Net-(IC4-HO): track 0.00 -> 14.7 mm
- net Net-(IC3-LO): track 0.00 -> 14.6 mm
- net Net-(IC3-HB): track 0.00 -> 8.84 mm
- net Net-(IC4-HB): track 0.00 -> 8.73 mm
- net Net-(IC3-HI): track 0.00 -> 4.57 mm
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- added copper zone on F.Cu, net MOTOR_U
- added copper zone on F.Cu, net MOTOR_U_SHUNT_P
- added copper zone on F.Cu, net MOTOR_V
- added copper zone on F.Cu, net MOTOR_V_SHUNT_P
- added copper zone on F.Cu, net MOTOR_W
- added copper zone on F.Cu, net MOTOR_W_SHUNT_P
- added copper zone on B.Cu, net PWR_INPUT(12V~48V)
- added copper zone on F.Cu, net PWR_INPUT(12V~48V)

Commit message: 중간 저장
Parts:
- removed R38, R39, R40, R41, R42, R43, R44, R45, R46, R47, R48, R49, R50, R51, R52, R53, R54, R55, R56, R57, R58, R59, R60, R61, R62, R63, R64, R65, R66, R67, R68, R69, R70, R71, R72, R73, R74, R75, R76, R77, R78, R79, R80, R81, R82, R83, R84, R85, R86, R87, R88, R89: 33R/0.063w, Resistor_SMD:R_0402_1005Metric
- removed the R90 at (-127.6, 113.8)
- removed the R91 at (-127.6, 115.8)
- removed the R92 at (-127.6, 117.8)
- removed the R93 at (-127.6, 119.8)
- added C68: 0.1uF/50V, Capacitor_SMD:C_0603_1608Metric, F.Cu at (147.2, 106.2)
- added C69: 0.1uF/50V, Capacitor_SMD:C_0603_1608Metric, F.Cu at (147.2, 108.7)
- added C70: 0.1uF/50V, Capacitor_SMD:C_0603_1608Metric, F.Cu at (147.2, 111.2)
- added C71: 0.1uF/50V, Capacitor_SMD:C_0603_1608Metric, F.Cu at (147.2, 113.7)
- added U11: 4D02WGJ0330T, footprints:4D02_2X1_ROH, F.Cu at (154.1, 95.8)
- added U12: 4D02WGJ0330T, footprints:4D02_2X1_ROH, F.Cu at (147.0, 103.1)
- added U13: 4D02WGJ0330T, footprints:4D02_2X1_ROH, F.Cu at (157.7, 95.8)
- added U14: 4D02WGJ0330T, footprints:4D02_2X1_ROH, F.Cu at (150.6, 103.1)
- added U15: 4D02WGJ0330T, footprints:4D02_2X1_ROH, F.Cu at (161.2, 95.8)
- added U16: 4D02WGJ0330T, footprints:4D02_2X1_ROH, F.Cu at (154.1, 103.1)
- added U18: 4D02WGJ0330T, footprints:4D02_2X1_ROH, F.Cu at (147.0, 99.5)
- added U19: 4D02WGJ0330T, footprints:4D02_2X1_ROH, F.Cu at (157.7, 103.1)
- added U20: 4D02WGJ0330T, footprints:4D02_2X1_ROH, F.Cu at (150.6, 99.5)
- added U21: 4D02WGJ0330T, footprints:4D02_2X1_ROH, F.Cu at (154.1, 99.5)
- added U6: 4D02WGJ0330T, footprints:4D02_2X1_ROH, F.Cu at (157.7, 99.5)
- added U7: 4D02WGJ0330T, footprints:4D02_2X1_ROH, F.Cu at (147.0, 95.8)
- added U8: 4D02WGJ0330T, footprints:4D02_2X1_ROH, F.Cu at (161.2, 99.5)
- added U9: 4D02WGJ0330T, footprints:4D02_2X1_ROH, F.Cu at (150.6, 95.8)
- moved C66 283.9 mm to (143.8, 71.7), turned to 90 degrees
- moved C62 282.9 mm to (146.2, 88.2), turned to -90 degrees
- moved C60 272.8 mm to (132.1, 88.2), turned to -90 degrees
- moved C67 272.4 mm to (130.8, 71.7), turned to 90 degrees
- moved C64 270.5 mm to (129.2, 88.2), turned to -90 degrees
- moved C63 270.4 mm to (127.8, 65.8)
- moved C65 268.4 mm to (126.2, 88.2), turned to -90 degrees
- moved C61 264.9 mm to (122.8, 85.7), turned to 180 degrees
- moved IC3 255.5 mm to (135.8, 79.9), turned to 90 degrees
- moved R111 184.0 mm to (127.2, 137.3), turned to -90 degrees
- moved R92 182.5 mm to (126.2, 137.2), turned to -90 degrees
- moved R90 181.7 mm to (125.2, 137.2), turned to -90 degrees
- moved R93 180.3 mm to (124.2, 137.2), turned to -90 degrees
- moved R94 179.2 mm to (123.2, 137.2), turned to -90 degrees
- moved R95 178.0 mm to (122.2, 137.2), turned to -90 degrees
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- renumbered C6 to C1, C13 to C10, C90 to C100, C93 to C101, C99 to C102, C105 to C103, C108 to C104, C96 to C105, C102 to C106, C117 to C107, C114 to C108, C122 to C109, C28 to C11, C123 to C110, C125 to C111, C113 to C112, C115 to C113, C124 to C114, C119 to C115, C118 to C116, C120 to C117, C112 to C118, C116 to C119, C15 to C12, C121 to C120, C21 to C13, C25 to C14, C7 to C15, C3 to C16, C12 to C17, C1 to C18, C14 to C19, C8 to C2, C16 to C20, C29 to C21, C18 to C22, C17 to C23, C23 to C24, C26 to C25, C30 to C26, C33 to C27, C36 to C28, C37 to C29, C9 to C3, C38 to C30, C39 to C31, C42 to C32, C43 to C33, C44 to C34, C45 to C35, C46 to C36, C47 to C37, C49 to C38, C50 to C39, C10 to C4, C52 to C40, C54 to C41, C55 to C42, C56 to C43, C40 to C44, C41 to C45, C48 to C46, C57 to C47, C58 to C48, C31 to C49, C11 to C5, C35 to C50, C32 to C51, C34 to C52, C51 to C53, C53 to C54, C61 to C55, C63 to C56, C59 to C57, C60 to C58, C62 to C59, C126 to C6, C68 to C60, C70 to C61, C72 to C62, C74 to C63, C69 to C64, C71 to C65, C73 to C66, C75 to C67, C128 to C7, C64 to C72, C65 to C73, C66 to C74, C67 to C75, C79 to C76, C80 to C77, C76 to C78, C77 to C79, C4 to C8, C78 to C80, C82 to C81, C83 to C82, C81 to C83, C88 to C84, C91 to C85, C97 to C86, C85 to C87, C84 to C88, C103 to C89, C5 to C9, C106 to C90, C94 to C91, C100 to C92, C89 to C93, C92 to C94, C98 to C95, C104 to C96, C107 to C97, C95 to C98, C101 to C99, D11 to D10, D12 to D11, D13 to D12, D16 to D13, D17 to D14, D14 to D15, D18 to D16, D19 to D17, D15 to D18, D20 to D19, D3 to D2, D21 to D20, D2 to D3, D6 to D5, D7 to D6, D8 to D7, D9 to D8, D10 to D9, IC11 to IC1, IC7 to IC10, IC1 to IC2, IC2 to IC3, IC3 to IC4, IC4 to IC5, IC5 to IC6, IC6 to IC7, IC9 to IC8, IC8 to IC9, J2 to J1, J9 to J10, J6 to J11, J1 to J2, J7 to J4, J8 to J5, J10 to J6, J11 to J7, J5 to J8, J4 to J9, L2 to L1, L7 to L2, L1 to L3, L3 to L4, L8 to L5, L4 to L6, L5 to L7, L9 to L8, L10 to L9, LED4 to LED3, LED5 to LED4, PS2 to PS1, PS3 to PS2, PS4 to PS3, PS5 to PS4, R3 to R1, R14 to R10, R106 to R100, R107 to R101, R108 to R102, R95 to R103, R109 to R104, R110 to R105, R111 to R106, R112 to R107, R113 to R108, R114 to R109, R8 to R11, R115 to R110, R96 to R111, R116 to R112, R117 to R113, R118 to R114, R120 to R115, R122 to R116, R121 to R117, R119 to R118, R123 to R119, R20 to R12, R132 to R120, R141 to R121, R147 to R122, R126 to R123, R127 to R124, R142 to R125, R148 to R126, R6 to R127, R124 to R128, R133 to R129, R21 to R13, R143 to R130, R149 to R131, R128 to R132, R129 to R133, R144 to R134, R150 to R135, R9 to R136, R125 to R137, R134 to R138, R145 to R139, R16 to R14, R151 to R140, R130 to R141, R131 to R142, R146 to R143, R152 to R144, R10 to R145, R156 to R146, R158 to R147, R160 to R148, R161 to R149, R22 to R15, R176 to R150, R162 to R151, R170 to R152, R163 to R153, R177 to R154, R164 to R155, R171 to R156, R159 to R157, R165 to R158, R178 to R159, R23 to R16, R166 to R160, R172 to R161, R167 to R162, R179 to R163, R173 to R164, R157 to R165, R168 to R166, R180 to R167, R174 to R168, R18 to R17, R181 to R170, R175 to R171, R19 to R18, R15 to R19, R4 to R2, R17 to R20, R30 to R21, R31 to R22, R34 to R23, R37 to R24, R35 to R27, R36 to R28, R28 to R29, R5 to R3, R29 to R30, R32 to R31, R33 to R32, R27 to R33, R11 to R4, R12 to R5, R7 to R6, R1 to R7, R2 to R8, R13 to R9, R97 to R90, R94 to R91, R98 to R92, R99 to R93, R100 to R94, R101 to R95, R102 to R96, R103 to R97, R104 to R98, R105 to R99, S4 to S2, S2 to S3, S3 to S4, TP12 to TP10, TP14 to TP11, TP11 to TP12, TP15 to TP14, TP18 to TP15, TP19 to TP16, TP16 to TP17, TP20 to TP18, TP21 to TP19, TP3 to TP2, TP22 to TP20, TP17 to TP21, TP23 to TP22, TP5 to TP3, TP2 to TP4, TP6 to TP5, TP7 to TP6, TP8 to TP7, TP9 to TP8, TP10 to TP9, U6 to U10, U3 to U2, U8 to U22, U9 to U23, U10 to U24, U2 to U3
Connections:
- C1 pad 2: MOTOR_U_SHUNT_M -> GND_PWR
- C2 pad 2: MOTOR_U_SHUNT_M -> GND_PWR
- C3 pad 2: MOTOR_U_SHUNT_M -> GND_PWR
- C4 pad 2: MOTOR_U_SHUNT_M -> GND_PWR
- C5 pad 2: MOTOR_U_SHUNT_M -> GND_PWR
- C8 pad 2: MOTOR_U_SHUNT_M -> GND_PWR
- D2 pad 2: MOTOR_U_SHUNT_M -> GND_PWR
- IC4 pad 4: MOTOR_U_SHUNT_M -> GND_PWR
- IC5 pad 4: MOTOR_U_SHUNT_M -> GND_PWR
- IC6 pad 4: MOTOR_U_SHUNT_M -> GND_PWR
- J1 pad 2: MOTOR_U_SHUNT_M -> GND_PWR
- J1 pad 3: MOTOR_U_SHUNT_M -> GND_PWR
- J2 pad 1: MOTOR_U_SHUNT_M -> GND_PWR
- J4 pad 5: MOTOR_U_SHUNT_M -> GND_PWR
- J4 pad 6: MOTOR_U_SHUNT_M -> GND_PWR
- J6 pad 4: MOTOR_U_SHUNT_M -> GND_PWR
- L7 pad 1: MOTOR_U_SHUNT_M -> GND_PWR
- R126 pad 2: MOTOR_U_SHUNT_M -> GND_PWR
- R127 pad 2: MOTOR_U_SHUNT_M -> GND_PWR
- R135 pad 2: MOTOR_U_SHUNT_M -> GND_PWR
- R136 pad 2: MOTOR_U_SHUNT_M -> GND_PWR
- R144 pad 2: MOTOR_U_SHUNT_M -> GND_PWR
- R145 pad 2: MOTOR_U_SHUNT_M -> GND_PWR
- R151 pad 1: MOTOR_U_SHUNT_M -> GND_PWR
- R155 pad 1: MOTOR_U_SHUNT_M -> GND_PWR
- R160 pad 1: MOTOR_U_SHUNT_M -> GND_PWR
- R2 pad 1: MOTOR_U_SHUNT_M -> GND_PWR
- R3 pad 1: MOTOR_U_SHUNT_M -> GND
Routing:
- net LEDA: track 0.00 -> 77.4 mm, vias 0 -> 4
- net I2C1_SCL: track 0.00 -> 55.7 mm, vias 0 -> 2
- net LEDK1: track 0.00 -> 55.2 mm
- net TP_RES: track 0.00 -> 54.1 mm, vias 0 -> 2
- net LTDC_CLK: track 0.00 -> 49.4 mm, vias 0 -> 2
- net TP_INT: track 0.00 -> 48.5 mm, vias 0 -> 2
- net LTDC_DE: track 0.00 -> 48.5 mm, vias 0 -> 2
- net LTDC_VSYNC: track 0.00 -> 48.5 mm, vias 0 -> 2
- net LTDC_HSYNC: track 0.00 -> 48.2 mm, vias 0 -> 2
- net I2C1_SDA: track 0.00 -> 48.0 mm, vias 0 -> 2
- net LEDK2: track 0.00 -> 43.6 mm
- net 5V: track 0.00 -> 42.0 mm
- net LTDC_G7: track 0.00 -> 41.1 mm, vias 0 -> 2
- net LTDC_B6: track 0.00 -> 40.8 mm, vias 0 -> 2
- net LTDC_B7: track 0.00 -> 40.5 mm, vias 0 -> 2
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- added copper zone on F.Cu, net 12V
- added copper zone on B.Cu, net GND_PWR
