File: 1.hardware/bldc_motor_controller.kicad_pcb (KiCad board)
At the start: 4 copper layers, 180 x 100 mm, 364 parts, among them IC1 TLV74018PDBVR, IC10 SN74HC74PWRG4, IC2 LMR51610XDBVR, IC3 IS42S32800J-6TLI, IC4 UCC27712QDRQ1, IC5 UCC27712QDRQ1, IC6 UCC27712QDRQ1, IC7 SN74HCS266QDRQ1, IC8 SN74LVC3G17DCURG4, IC9 SN74LVC3G17DCURG4, J1 12V-48V Jack, J10 ESP_DBG_CONN, J11 ESP_BOOT_CONN, J12 FPC_LCD_40_CONN, J13 2061-603/998-404, J14 2060-452/998-404, J15 2060-453/998-404, J2 12V~48V BAT_XT60_MALE, J3 DEBUG_CONN, J4 CAN_CONN, J5 I2C_CONN, J6 CAN_CONN2, J7 EXTRA_SPI3_CONN, J8 USB_C, J9 UART_CONN, Q1 STL130N6F7, Q2 STL130N6F7, Q3 STL130N6F7, Q4 STL130N6F7, Q5 STL130N6F7, Q6 STL130N6F7, U1 TL431AIDBZR, U10 W25Q128JVS, U11 4D02WGJ0330T, U12 4D02WGJ0330T, U13 4D02WGJ0330T, U14 4D02WGJ0330T, U15 4D02WGJ0330T, U16 4D02WGJ0330T, U18 4D02WGJ0330T, U19 4D02WGJ0330T, U2 TXS0104EPW, U20 4D02WGJ0330T, U21 4D02WGJ0330T, U22 Hall_Analog_Joystick, U23 TLV9064, U24 TLV9064, U3 STM32H743BITx, U4 SN65HVD230, U5 ESP32-C3-WROOM-02, U6 4D02WGJ0330T, U7 4D02WGJ0330T, U8 4D02WGJ0330T, U9 4D02WGJ0330T, X1 SMD3225-4, Y1 X1A0000610002

Commit message: 중간 저장
Parts:
- added C121: 0.1uF/50V, Capacitor_SMD:C_0603_1608Metric, F.Cu at (139.2, 92.5)
- moved U8 42.9 mm to (130.0, 70.1), turned to -90 degrees
- moved C69 41.8 mm to (127.8, 71.7), turned to 90 degrees
- moved C68 38.3 mm to (141.1, 68.4), turned to 90 degrees
- moved U19 35.2 mm to (142.8, 71.2), turned to -90 degrees
- moved U16 35.0 mm to (139.6, 71.2), turned to -90 degrees
- moved U14 34.6 mm to (137.0, 71.2), turned to -90 degrees
- moved U12 34.3 mm to (134.4, 71.2), turned to -90 degrees
- moved C70 27.5 mm to (148.7, 83.8)
- moved C71 25.3 mm to (145.3, 88.5), turned to -90 degrees
- moved U15 24.2 mm to (138.1, 88.6), turned to 90 degrees
- moved U13 23.3 mm to (135.6, 88.6), turned to 90 degrees
- moved U11 22.3 mm to (133.0, 88.6), turned to 90 degrees
- moved U9 22.3 mm to (129.5, 88.5), turned to 90 degrees
- moved U7 21.3 mm to (126.9, 88.5), turned to 90 degrees
- moved U21 20.3 mm to (149.6, 79.7), turned to 180 degrees
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Connections:
- U12 pad 1: FMC_NBL1 -> FMC_A9
- U12 pad 2: FMC_SDCLK -> FMC_SDCKE0
- U12 pad 3: FMC_SDCKE0 -> FMC_SDCLK
- U12 pad 4: FMC_A9 -> FMC_NBL1
- U12 pad 5: SDRAM_A9 -> SDRAM_DQM1
- U12 pad 6: SDRAM_CKE -> SDRAM_CLK
- U12 pad 7: SDRAM_CLK -> SDRAM_CKE
- U12 pad 8: SDRAM_DQM1 -> SDRAM_A9
- U14 pad 1: FMC_A8 -> FMC_A5
- U14 pad 2: FMC_A7 -> FMC_A6
- U14 pad 3: FMC_A6 -> FMC_A7
- U14 pad 4: FMC_A5 -> FMC_A8
- U14 pad 5: SDRAM_A5 -> SDRAM_A8
- U14 pad 6: SDRAM_A6 -> SDRAM_A7
- U14 pad 7: SDRAM_A7 -> SDRAM_A6
- U14 pad 8: SDRAM_A8 -> SDRAM_A5
- U16 pad 1: FMC_A4 -> FMC_D31
- U16 pad 2: FMC_A3 -> FMC_NBL3
- U16 pad 3: FMC_NBL3 -> FMC_A3
- U16 pad 4: FMC_D31 -> FMC_A4
- U16 pad 5: SDRAM_DQ31 -> SDRAM_A4
- U16 pad 6: SDRAM_DQM3 -> SDRAM_A3
- U16 pad 7: SDRAM_A3 -> SDRAM_DQM3
- U16 pad 8: SDRAM_A4 -> SDRAM_DQ31
- U19 pad 1: FMC_D30 -> FMC_D27
- U19 pad 2: FMC_D29 -> FMC_D28
- U19 pad 3: FMC_D28 -> FMC_D29
- U19 pad 4: FMC_D27 -> FMC_D30
- U19 pad 5: SDRAM_DQ27 -> SDRAM_DQ30
- U19 pad 6: SDRAM_DQ28 -> SDRAM_DQ29
- U19 pad 7: SDRAM_DQ29 -> SDRAM_DQ28
- U19 pad 8: SDRAM_DQ30 -> SDRAM_DQ27
- U6 pad 1: FMC_D15 -> FMC_D12
- U6 pad 2: FMC_D14 -> FMC_D13
- U6 pad 3: FMC_D13 -> FMC_D14
- U6 pad 4: FMC_D12 -> FMC_D15
- U6 pad 5: SDRAM_DQ12 -> SDRAM_DQ15
- U6 pad 6: SDRAM_DQ13 -> SDRAM_DQ14
- U6 pad 7: SDRAM_DQ14 -> SDRAM_DQ13
- U6 pad 8: SDRAM_DQ15 -> SDRAM_DQ12
- U8 pad 1: FMC_D11 -> FMC_D8
- U8 pad 2: FMC_D10 -> FMC_D9
- U8 pad 3: FMC_D9 -> FMC_D10
- U8 pad 4: FMC_D8 -> FMC_D11
- U8 pad 5: SDRAM_DQ8 -> SDRAM_DQ11
- U8 pad 6: SDRAM_DQ9 -> SDRAM_DQ10
- U8 pad 7: SDRAM_DQ10 -> SDRAM_DQ9
- U8 pad 8: SDRAM_DQ11 -> SDRAM_DQ8
Routing:
- net 3V3_MCU: track 26.9 -> 61.1 mm, vias 0 -> 2
- net SDRAM_DQ26: track 0.00 -> 10.8 mm
- net SDRAM_DQ25: track 0.00 -> 10.2 mm
- net SDRAM_DQ24: track 0.00 -> 8.10 mm
- net SDRAM_DQ23: track 0.00 -> 7.88 mm, vias 0 -> 2
- net SDRAM_DQM2: track 0.00 -> 2.73 mm
- net SDRAM_DQM3: track 0.00 -> 2.71 mm
- net SDRAM_A3: track 0.00 -> 2.71 mm
- net SDRAM_A4: track 0.00 -> 2.71 mm
- net SDRAM_DQM1: track 0.00 -> 2.69 mm
- net SDRAM_DQ7: track 0.00 -> 2.64 mm
- net SDRAM_DQ29: track 0.00 -> 2.58 mm
- net SDRAM_DQ30: track 0.00 -> 2.58 mm
- net SDRAM_DQ21: track 0.00 -> 2.58 mm
- net SDRAM_DQ22: track 0.00 -> 2.58 mm
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
Commit message: 많이 간소화함 일부 핀이 비연결로 확인됨
Parts:
- removed L6: 60R_100Mhz, Inductor_SMD:L_0603_1608Metric
- moved R115 154.4 mm to (62.2, 116.8), turned to 180 degrees
- moved R117 152.9 mm to (66.6, 135.9), turned to 90 degrees
- moved C81 149.4 mm to (64.2, 116.6), turned to 90 degrees
- moved R116 144.6 mm to (52.4, 122.6), turned to 90 degrees
- moved TP7 144.0 mm to (55.6, 118.4)
- moved TP8 140.6 mm to (52.2, 118.4)
- moved C82 137.4 mm to (52.2, 120.6), turned to 180 degrees
- moved C12 47.0 mm to (53.1, 44.0)
- moved C13 47.0 mm to (53.1, 46.4)
- moved C14 47.0 mm to (53.9, 48.4)
- moved C23 47.0 mm to (47.7, 44.0)
- moved C24 47.0 mm to (47.8, 46.4)
- moved C25 47.0 mm to (48.6, 48.4)
- moved C62 38.1 mm to (108.8, 91.0), turned to 180 degrees
- moved C71 36.5 mm to (108.8, 89.5), turned to 180 degrees
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Connections:
- C57 pad 1: 3V3_ESP32 -> 3V3_MCU
- C58 pad 1: 3V3_ESP32 -> 3V3_MCU
- C59 pad 1: 3V3_ESP32 -> 3V3_MCU
- R27 pad 1: 3V3_ESP32 -> 3V3_MCU
- R28 pad 1: 3V3_ESP32 -> 3V3_MCU
- R29 pad 1: 3V3_ESP32 -> 3V3_MCU
- R30 pad 1: 3V3_ESP32 -> 3V3_MCU
- U5 pad 1: 3V3_ESP32 -> 3V3_MCU
Routing:
- net FMC_D7: track 0.00 -> 66.0 mm, vias 0 -> 2
- net FMC_D16: track 0.00 -> 64.2 mm, vias 0 -> 2
- net FMC_D20: track 0.00 -> 63.4 mm, vias 0 -> 2
- net FMC_D17: track 0.00 -> 63.3 mm, vias 0 -> 2
- net FMC_D18: track 0.00 -> 62.6 mm, vias 0 -> 2
- net FMC_D19: track 0.00 -> 62.4 mm, vias 0 -> 2
- net FMC_D6: track 0.00 -> 61.6 mm, vias 0 -> 2
- net FMC_D5: track 0.00 -> 61.0 mm, vias 0 -> 2
- net LTDC_B6: track 40.8 -> 99.6 mm
- net FMC_BA0: track 0.00 -> 58.2 mm, vias 0 -> 2
- net FMC_A11: track 0.00 -> 57.4 mm, vias 0 -> 2
- net FMC_BA1: track 0.00 -> 56.3 mm, vias 0 -> 2
- net LTDC_B7: track 40.5 -> 96.7 mm
- net FMC_SDNRAS: track 0.00 -> 55.0 mm, vias 0 -> 2
- net FMC_A10: track 0.00 -> 54.5 mm, vias 0 -> 2
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- removed copper zone on F.Cu, net 12V

Commit message: 중간 저장
Parts:
- moved TP12 293.0 mm to (198.3, 114.8)
- moved TP9 291.0 mm to (198.4, 65.6)
- moved TP13 290.0 mm to (198.3, 119.2)
- moved TP10 287.3 mm to (198.4, 71.5)
- moved TP14 287.2 mm to (198.4, 123.0)
- moved TP11 283.7 mm to (198.4, 77.6)
- moved J7 202.2 mm to (124.4, 160.8), turned to 90 degrees
- moved J4 150.5 mm to (126.3, 169.1)
- moved R28 99.3 mm to (166.8, 140.4)
- moved R27 91.9 mm to (166.8, 138.8)
- moved J5 67.1 mm to (80.5, 160.2)
- moved J6 67.1 mm to (87.5, 179.7)
- moved C83 56.7 mm to (-44.0, 145.9)
- moved RT1 56.7 mm to (-40.3, 152.7)
- moved R118 56.7 mm to (-37.0, 145.6)
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Routing:
- net 12V: track 0.00 -> 129.5 mm, vias 0 -> 3
- net DEBUG_RESET: track 0.00 -> 102.1 mm, vias 0 -> 4
- net DEBUG_JTDO_SWO: track 0.00 -> 95.5 mm, vias 0 -> 4
- net DEBUG_JTDI: track 0.00 -> 76.5 mm, vias 0 -> 2
- net Ext_Voltage: track 2.42 -> 76.0 mm, vias 0 -> 2
- net FMC_SDCKE0: track 0.00 -> 71.7 mm, vias 0 -> 2
- net FMC_D0: track 0.00 -> 71.1 mm, vias 0 -> 2
- net DEBUG_SWCLK: track 0.00 -> 69.8 mm, vias 0 -> 2
- net FMC_D1: track 0.00 -> 68.2 mm, vias 0 -> 2
- net FMC_A6: track 0.00 -> 66.5 mm, vias 0 -> 4
- net FMC_A7: track 0.00 -> 66.4 mm, vias 0 -> 4
- net FMC_D4: track 0.00 -> 62.6 mm, vias 0 -> 2
- net FMC_D15: track 0.00 -> 61.6 mm, vias 0 -> 2
- net FMC_A4: track 0.00 -> 61.2 mm, vias 0 -> 2
- net FMC_D14: track 0.00 -> 60.7 mm, vias 0 -> 2
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Other:
- board size 180 x 100 mm -> 150 x 100 mm

Commit message: 중간 저장
Parts:
- added C122: 0.1uF/50V, Capacitor_SMD:C_0603_1608Metric, F.Cu at (100.2, 88.5)
- moved U4 122.7 mm to (95.8, 88.5), turned to 180 degrees
- moved J4 101.9 mm to (54.1, 97.2), turned to -90 degrees
- moved JP1 80.9 mm to (66.8, 100.2), turned to 90 degrees
- moved R23 80.1 mm to (64.5, 100.2), turned to -90 degrees
- moved TP2 74.7 mm to (95.5, 70.2)
- moved J7 69.2 mm to (163.8, 103.9), turned to 0 degrees
- moved C88 42.9 mm to (-39.8, 78.5)
- moved R17 41.8 mm to (71.0, 132.7), turned to 90 degrees
- moved R18 40.9 mm to (73.3, 132.7), turned to 90 degrees
- moved C83 39.5 mm to (-46.1, 106.5)
- moved RT1 39.5 mm to (-42.3, 113.3)
- moved R118 39.5 mm to (-39.1, 106.2)
- moved LED1 38.4 mm to (71.0, 130.2), turned to -90 degrees
- moved LED2 37.4 mm to (73.3, 130.2), turned to -90 degrees
- moved C77 34.8 mm to (131.9, 144.4), turned to -90 degrees
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Connections:
- U4 pad 3: +3.3V -> 3V3_MCU
Routing:
- net PWR_INPUT(12V~48V): track 12.9 -> 76.9 mm, vias 88 -> 90
- net GND: track 0.00 -> 62.6 mm, vias 0 -> 29
- net CANH: track 0.00 -> 50.4 mm, vias 0 -> 3
- net CANL: track 0.00 -> 47.5 mm, vias 0 -> 3
- net 3V3_MCU: track 86.8 -> 134.0 mm, vias 0 -> 24
- net CAN_RXD: track 0.00 -> 22.3 mm, vias 0 -> 2
- net GND_PWR: track 0.00 -> 21.5 mm
- net CAN_TXD: track 0.00 -> 18.3 mm, vias 0 -> 2
- net 3V3: track 17.1 -> 35.1 mm
- net Ext_Voltage: track 76.0 -> 82.1 mm, vias 2 -> 3
- net Net-(C8-Pad1): track 5.29 -> 8.10 mm
- net Net-(JP1-A): track 0.00 -> 2.41 mm
- net DEBUG_JTDO_SWO: track 95.5 -> 96.1 mm
- net FMC_NBL1: track 46.4 -> 45.8 mm
- net TP_INT: track 84.1 -> 84.7 mm
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- added copper zone on In1.Cu, net 3V3_MCU

Commit message: 스펙 정함
4층 기판, 비아 0.3 / 0.5 사이즈, 외부 2온즈, Plugger Via, 77달러 정도 나옴
Parts:
- removed C56: 0.1uF/50V, Capacitor_SMD:C_0603_1608Metric
- removed D9: WS2812B, LED_SMD:LED_WS2812B_PLCC4_5.0x5.0mm_P3.2mm
- removed R24: 1k/0.063w, Resistor_SMD:R_0402_1005Metric
- moved R14 300.2 mm to (256.3, 102.8)
- moved R25 261.8 mm to (244.3, 113.7)
- moved R26 261.8 mm to (244.3, 115.6)
- moved R33 261.8 mm to (244.3, 117.6)
- moved C107 246.5 mm to (233.0, 83.7)
- moved C109 246.5 mm to (236.9, 103.1)
- moved C110 246.5 mm to (236.9, 105.1)
- moved C114 246.5 mm to (236.9, 107.0)
- moved C115 246.5 mm to (233.0, 88.7)
- moved C116 246.5 mm to (233.0, 86.2)
- moved C117 246.5 mm to (233.0, 91.2)
- moved C120 246.5 mm to (233.0, 93.8)
- moved R149 246.5 mm to (216.8, 93.4)
- moved R150 246.5 mm to (222.6, 95.4)
- moved R151 246.5 mm to (216.8, 95.4)
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Connections:
- C57 pad 1: 3V3_MCU -> 3V3
- C58 pad 1: 3V3_MCU -> 3V3
- C59 pad 1: 3V3_MCU -> 3V3
- D8 pad 2: Net-(D8-DOUT) -> unconnected-(D8-DOUT-Pad2)
- R17 pad 1: 3V3_MCU -> 3V3
- R18 pad 1: 3V3_MCU -> 3V3
- R19 pad 2: 3V3_MCU -> 3V3
- R20 pad 2: 3V3_MCU -> 3V3
- R27 pad 1: 3V3_MCU -> 3V3
- R28 pad 1: 3V3_MCU -> 3V3
- R29 pad 1: 3V3_MCU -> 3V3
- R30 pad 1: 3V3_MCU -> 3V3
- RT1 pad 2: ADC_VREF_2V5 -> 3V3
- U5 pad 1: 3V3_MCU -> 3V3
Routing:
- net 5V: track 46.1 -> 130.0 mm, vias 0 -> 2
- net GND: track 62.6 -> 133.4 mm, vias 29 -> 45
- net Joystick_V: track 1.29 -> 62.9 mm, vias 0 -> 2
- net FMC_A8: track 1.33 -> 61.8 mm, vias 1 -> 4
- net FMC_A9: track 1.12 -> 60.4 mm, vias 1 -> 4
- net Joystick_H: track 1.29 -> 55.4 mm, vias 0 -> 4
- net GND_PWR: track 21.5 -> 73.2 mm, vias 0 -> 10
- net HALL_6x_Pulse_Sig: track 0.00 -> 50.7 mm, vias 0 -> 2
- net 3V3_MCU: track 134.0 -> 180.4 mm, vias 24 -> 23
- net MOTOR_DIR: track 0.00 -> 45.8 mm
- net BTN2: track 2.33 -> 46.2 mm
- net BTN1: track 2.33 -> 44.9 mm
- net ADC_VREF_2V5: track 0.00 -> 37.5 mm, vias 0 -> 2
- net LED2: track 0.00 -> 37.0 mm
- net LED1: track 0.00 -> 36.2 mm
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- added copper zone on In1.Cu, net 3V3
- added copper zone on In2.Cu, net GND
- added copper zone on F.Cu, net GND_PWR
