File: 1.hardware/bldc_motor_controller.kicad_sch (KiCad schematic)
At the start: 0 parts

Commit message: 중간 수정
Other:
- sheet interface renamed 3.interface
- sheet lcd renamed 5.lcd
- sheet mcu renamed 2.mcu
- sheet memory renamed 4.memory
- sheet motor_control renamed 7.motor_control
- sheet power renamed 1.power
- sheet sensor renamed 6.sensor
Changed lines of the file:
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@@
 			(color 0 0 0 0.0000)
 		)
-		(property "Sheetname" "motor_control"
+		(property "Sheetname" "7.motor_control"
 			(at 31.75 78.0284 0)
 			(effects
@@
 			(project "bldc_motor_controller"
 				(path "/a25adab6-a8c3-4e0e-8ba9-baac00aaa394"
-					(page "7")
+					(page "8")
 				)
 			)
@@
 			(color 0 0 0 0.0000)
 		)
-		(property "Sheetname" "sensor"
+		(property "Sheetname" "6.sensor"
 			(at 134.62 78.0284 0)
 			(effects
@@
 			(project "bldc_motor_controller"
 				(path "/a25adab6-a8c3-4e0e-8ba9-baac00aaa394"
-					(page "5")
+					(page "7")
 				)
 			)
@@
 			(color 0 0 0 0.0000)
 		)
-		(property "Sheetname" "interface"
+		(property "Sheetname" "3.interface"
 			(at 33.02 127.5584 0)
 			(effects
@@
 			(project "bldc_motor_controller"
 				(path "/a25adab6-a8c3-4e0e-8ba9-baac00aaa394"
-					(page "8")
+					(page "4")
 				)
 			)
@@
 			(color 0 0 0 0.0000)
 		)
-		(property "Sheetname" "lcd"
+		(property "Sheetname" "5.lcd"
 			(at 83.82 78.0284 0)
 			(effects
@@
 			(color 0 0 0 0.0000)
 		)
-		(property "Sheetname" "memory"
+		(property "Sheetname" "4.memory"
 			(at 134.62 27.2284 0)
 			(effects
@@
 			(project "bldc_motor_controller"
 				(path "/a25adab6-a8c3-4e0e-8ba9-baac00aaa394"
-					(page "7")
-				)
-			)
-		)
-	)
-	(sheet
-		(at 31.75 27.94)
+					(page "5")
+				)
+			)
+		)
+	)
+	(sheet
+		(at 83.82 27.94)
 		(size 46.99 36.83)
 		(exclude_from_sim no)
@@
 			(color 0 0 0 0.0000)
 		)
-		(property "Sheetname" "mcu"
-			(at 31.75 27.2284 0)
+		(property "Sheetname" "2.mcu"
+			(at 83.82 27.2284 0)
 			(effects
 				(font
@@
 		)
 		(property "Sheetfile" "mcu.kicad_sch"
-			(at 31.75 65.3546 0)
+			(at 83.82 65.3546 0)
+			(effects
+				(font
+					(size 1.27 1.27)
+				)
+				(justify left top)
+			)
+		)
+		(instances
+			(project "bldc_motor_controller"
+				(path "/a25adab6-a8c3-4e0e-8ba9-baac00aaa394"
+					(page "3")
+				)
+			)
+		)
+	)
+	(sheet
+		(at 33.02 27.94)
+		(size 45.72 36.83)
+		(exclude_from_sim no)
+		(in_bom yes)
+		(on_board yes)
+		(dnp no)
+		(fields_autoplaced yes)
+		(stroke
+			(width 0.1524)
+			(type solid)
+		)
+		(fill
+			(color 0 0 0 0.0000)
+		)
+		(property "Sheetname" "1.power"
+			(at 33.02 27.2284 0)
+			(effects
+				(font
+					(size 1.27 1.27)
+				)
+				(justify left bottom)
+			)
+		)
+		(property "Sheetfile" "power.kicad_sch"
+			(at 33.02 65.3546 0)
 			(effects
 				(font
@@
 				)
 			)
-		)
-	)
-	(sheet
-		(at 83.82 27.94)
-		(size 45.72 36.83)
-		(exclude_from_sim no)
-		(in_bom yes)
-		(on_board yes)
-		(dnp no)
-		(fields_autoplaced yes)
-		(stroke
-			(width 0.1524)
-			(type solid)
-		)
-		(fill
-			(color 0 0 0 0.0000)
-		)
-		(property "Sheetname" "power"
-			(at 83.82 27.2284 0)
-			(effects
-				(font
-					(size 1.27 1.27)
-				)
-				(justify left bottom)
-			)
-		)
-		(property "Sheetfile" "power.kicad_sch"
-			(at 83.82 65.3546 0)
-			(effects
-				(font
-					(size 1.27 1.27)
-				)
-				(justify left top)
-			)
-		)
-		(instances
-			(project "bldc_motor_controller"
-				(path "/a25adab6-a8c3-4e0e-8ba9-baac00aaa394"
-					(page "3")
-				)
-			)

Commit message: 중간 저장
Other:
- added sheet 8.motor_sense (motor_sense.kicad_sch)
Changed lines of the file:
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@@
+	)
+	(sheet
+		(at 85.09 128.27)
+		(size 44.45 38.1)
+		(exclude_from_sim no)
+		(in_bom yes)
+		(on_board yes)
+		(dnp no)
+		(fields_autoplaced yes)
+		(stroke
+			(width 0.1524)
+			(type solid)
+		)
+		(fill
+			(color 0 0 0 0.0000)
+		)
+		(property "Sheetname" "8.motor_sense"
+			(at 85.09 127.5584 0)
+			(effects
+				(font
+					(size 1.27 1.27)
+				)
+				(justify left bottom)
+			)
+		)
+		(property "Sheetfile" "motor_sense.kicad_sch"
+			(at 85.09 166.9546 0)
+			(effects
+				(font
+					(size 1.27 1.27)
+				)
+				(justify left top)
+			)
+		)
+		(instances
+			(project "bldc_motor_controller"
+				(path "/a25adab6-a8c3-4e0e-8ba9-baac00aaa394"
+					(page "9")
+				)
+			)
+		)
 	)
 	(sheet

Commit message: 중간 저장
Other:
- sheet 7.motor_control renamed 7.motor_control1
- sheet 8.motor_sense renamed 9.motor_sense
- added sheet 8.motor_control2 (motor_control2.kicad_sch)
Changed lines of the file:
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@@
 	(paper "A4")
 	(sheet
-		(at 31.75 78.74)
+		(at 180.34 19.05)
+		(size 44.45 36.83)
+		(exclude_from_sim no)
+		(in_bom yes)
+		(on_board yes)
+		(dnp no)
+		(fields_autoplaced yes)
+		(stroke
+			(width 0.1524)
+			(type solid)
+		)
+		(fill
+			(color 0 0 0 0.0000)
+		)
+		(property "Sheetname" "7.motor_control1"
+			(at 180.34 18.3384 0)
+			(effects
+				(font
+					(size 1.27 1.27)
+				)
+				(justify left bottom)
+			)
+		)
+		(property "Sheetfile" "motor_control.kicad_sch"
+			(at 180.34 56.4646 0)
+			(effects
+				(font
+					(size 1.27 1.27)
+				)
+				(justify left top)
+			)
+		)
+		(instances
+			(project "bldc_motor_controller"
+				(path "/a25adab6-a8c3-4e0e-8ba9-baac00aaa394"
+					(page "8")
+				)
+			)
+		)
+	)
+	(sheet
+		(at 121.92 60.96)
+		(size 44.45 36.83)
+		(exclude_from_sim no)
+		(in_bom yes)
+		(on_board yes)
+		(dnp no)
+		(fields_autoplaced yes)
+		(stroke
+			(width 0.1524)
+			(type solid)
+		)
+		(fill
+			(color 0 0 0 0.0000)
+		)
+		(property "Sheetname" "6.sensor"
+			(at 121.92 60.2484 0)
+			(effects
+				(font
+					(size 1.27 1.27)
+				)
+				(justify left bottom)
+			)
+		)
+		(property "Sheetfile" "sensor.kicad_sch"
+			(at 121.92 98.3746 0)
+			(effects
+				(font
+					(size 1.27 1.27)
+				)
+				(justify left top)
+			)
+		)
+		(instances
+			(project "bldc_motor_controller"
+				(path "/a25adab6-a8c3-4e0e-8ba9-baac00aaa394"
+					(page "7")
+				)
+			)
+		)
+	)
+	(sheet
+		(at 121.92 19.05)
+		(size 44.45 36.83)
+		(exclude_from_sim no)
+		(in_bom yes)
+		(on_board yes)
+		(dnp no)
+		(fields_autoplaced yes)
+		(stroke
+			(width 0.1524)
+			(type solid)
+		)
+		(fill
+			(color 0 0 0 0.0000)
+		)
+		(property "Sheetname" "3.interface"
+			(at 121.92 18.3384 0)
+			(effects
+				(font
+					(size 1.27 1.27)
+				)
+				(justify left bottom)
+			)
+		)
+		(property "Sheetfile" "interface.kicad_sch"
+			(at 121.92 56.4646 0)
+			(effects
+				(font
+					(size 1.27 1.27)
+				)
+				(justify left top)
+			)
+		)
+		(instances
+			(project "bldc_motor_controller"
+				(path "/a25adab6-a8c3-4e0e-8ba9-baac00aaa394"
+					(page "4")
+				)
+			)
+		)
+	)
+	(sheet
+		(at 69.85 60.96)
 		(size 46.99 36.83)
 		(exclude_from_sim no)
@@
 			(color 0 0 0 0.0000)
 		)
-		(property "Sheetname" "7.motor_control"
-			(at 31.75 78.0284 0)
-			(effects
-				(font
-					(size 1.27 1.27)
-				)
-				(justify left bottom)
-			)
-		)
-		(property "Sheetfile" "motor_control.kicad_sch"
-			(at 31.75 116.1546 0)
-			(effects
-				(font
-					(size 1.27 1.27)
-				)
-				(justify left top)
-			)
-		)
-		(instances
-			(project "bldc_motor_controller"
-				(path "/a25adab6-a8c3-4e0e-8ba9-baac00aaa394"
-					(page "8")
-				)
-			)
-		)
-	)
-	(sheet
-		(at 134.62 78.74)
-		(size 44.45 36.83)
-		(exclude_from_sim no)
-		(in_bom yes)
-		(on_board yes)
-		(dnp no)
-		(fields_autoplaced yes)
-		(stroke
-			(width 0.1524)
-			(type solid)
-		)
-		(fill
-			(color 0 0 0 0.0000)
-		)
-		(property "Sheetname" "6.sensor"
-			(at 134.62 78.0284 0)
-			(effects
-				(font
-					(size 1.27 1.27)
-				)
-				(justify left bottom)
-			)
-		)
-		(property "Sheetfile" "sensor.kicad_sch"
-			(at 134.62 116.1546 0)
-			(effects
-				(font
-					(size 1.27 1.27)
-				)
-				(justify left top)
-			)
-		)
-		(instances
-			(project "bldc_motor_controller"
-				(path "/a25adab6-a8c3-4e0e-8ba9-baac00aaa394"
-					(page "7")
-				)
-			)
-		)
-	)
-	(sheet
-		(at 33.02 128.27)
-		(size 46.99 38.1)
-		(exclude_from_sim no)
-		(in_bom yes)
-		(on_board yes)
-		(dnp no)
-		(fields_autoplaced yes)
-		(stroke
-			(width 0.1524)
-			(type solid)
-		)
-		(fill
-			(color 0 0 0 0.0000)
-		)
-		(property "Sheetname" "3.interface"
-			(at 33.02 127.5584 0)
-			(effects
-				(font
-					(size 1.27 1.27)
-				)
-				(justify left bottom)
-			)
-		)
-		(property "Sheetfile" "interface.kicad_sch"
-			(at 33.02 166.9546 0)
-			(effects
-				(font
-					(size 1.27 1.27)
-				)
-				(justify left top)
-			)
-		)
-		(instances
-			(project "bldc_motor_controller"
-				(path "/a25adab6-a8c3-4e0e-8ba9-baac00aaa394"
-					(page "4")
-				)
-			)
-		)
-	)
-	(sheet
-		(at 83.82 78.74)
+		(property "Sheetname" "5.lcd"
+			(at 69.85 60.2484 0)
+			(effects
+				(font
+					(size 1.27 1.27)
+				)
+				(justify left bottom)
+			)
+		)
+		(property "Sheetfile" "lcd.kicad_sch"
+			(at 69.85 98.3746 0)
+			(effects
+				(font
+					(size 1.27 1.27)
+				)
+				(justify left top)
+			)
+		)
+		(instances
+			(project "bldc_motor_controller"
+				(path "/a25adab6-a8c3-4e0e-8ba9-baac00aaa394"
+					(page "6")
+				)
+			)
+		)
+	)
+	(sheet
+		(at 19.05 60.96)
 		(size 45.72 36.83)
 		(exclude_from_sim no)
@@
 			(color 0 0 0 0.0000)
 		)
-		(property "Sheetname" "5.lcd"
-			(at 83.82 78.0284 0)
-			(effects
-				(font
-					(size 1.27 1.27)
-				)
-				(justify left bottom)
-			)
-		)
-		(property "Sheetfile" "lcd.kicad_sch"
-			(at 83.82 116.1546 0)
-			(effects
-				(font
-					(size 1.27 1.27)
-				)
-				(justify left top)
-			)
-		)
-		(instances
-			(project "bldc_motor_controller"
-				(path "/a25adab6-a8c3-4e0e-8ba9-baac00aaa394"
-					(page "6")
-				)
-			)
-		)
-	)
-	(sheet
-		(at 134.62 27.94)
-		(size 44.45 36.83)
-		(exclude_from_sim no)
-		(in_bom yes)
-		(on_board yes)
-		(dnp no)
-		(fields_autoplaced yes)
-		(stroke
-			(width 0.1524)
-			(type solid)
-		)
-		(fill
-			(color 0 0 0 0.0000)
-		)
 		(property "Sheetname" "4.memory"
-			(at 134.62 27.2284 0)
+			(at 19.05 60.2484 0)
 			(effects
 				(font
@@
 		)
 		(property "Sheetfile" "memory.kicad_sch"
-			(at 134.62 65.3546 0)
+			(at 19.05 98.3746 0)
 			(effects
 				(font
@@
 	)
 	(sheet
-		(at 85.09 128.27)
+		(at 180.34 106.68)
 		(size 44.45 38.1)
 		(exclude_from_sim no)
@@
 			(color 0 0 0 0.0000)
 		)
-		(property "Sheetname" "8.motor_sense"
-			(at 85.09 127.5584 0)
+		(property "Sheetname" "9.motor_sense"
+			(at 180.34 105.9684 0)
 			(effects
 				(font
@@
 		)
 		(property "Sheetfile" "motor_sense.kicad_sch"
-			(at 85.09 166.9546 0)
+			(at 180.34 145.3646 0)
+			(effects
+				(font
+					(size 1.27 1.27)
+				)
+				(justify left top)
+			)
+		)
+		(instances
+			(project "bldc_motor_controller"
+				(path "/a25adab6-a8c3-4e0e-8ba9-baac00aaa394"
+					(page "10")
+				)
+			)
+		)
+	)
+	(sheet
+		(at 180.34 62.23)
+		(size 44.45 38.1)
+		(exclude_from_sim no)
+		(in_bom yes)
+		(on_board yes)
+		(dnp no)
+		(fields_autoplaced yes)
+		(stroke
+			(width 0.1524)
+			(type solid)
+		)
+		(fill
+			(color 0 0 0 0.0000)
+		)
+		(property "Sheetname" "8.motor_control2"
+			(at 180.34 61.5184 0)
+			(effects
+				(font
+					(size 1.27 1.27)
+				)
+				(justify left bottom)
+			)
+		)
+		(property "Sheetfile" "motor_control2.kicad_sch"
+			(at 180.34 100.9146 0)
 			(effects
 				(font
@@
 	)
 	(sheet
-		(at 83.82 27.94)
+		(at 69.85 19.05)
 		(size 46.99 36.83)
 		(exclude_from_sim no)
@@
 		)
 		(property "Sheetname" "2.mcu"
-			(at 83.82 27.2284 0)
+			(at 69.85 18.3384 0)
 			(effects
 				(font
@@
 		)
 		(property "Sheetfile" "mcu.kicad_sch"
-			(at 83.82 65.3546 0)
+			(at 69.85 56.4646 0)
 			(effects
 				(font
@@
 	)
 	(sheet
-		(at 33.02 27.94)
+		(at 19.05 19.05)
 		(size 45.72 36.83)
 		(exclude_from_sim no)
@@
 		)
 		(property "Sheetname" "1.power"
-			(at 33.02 27.2284 0)
+			(at 19.05 18.3384 0)
 			(effects
 				(font
@@
 		)
 		(property "Sheetfile" "power.kicad_sch"
-			(at 33.02 65.3546 0)
-			(effects
-				(font
+			(at 19.05 56.4646 0)
+			(effects
+				(font

Commit message: 중간 저장
Other:
- sheet 7.motor_control1 renamed 7.motor_control
- removed sheet 8.motor_control2
Changed lines of the file:
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@@
 			(color 0 0 0 0.0000)
 		)
-		(property "Sheetname" "7.motor_control1"
+		(property "Sheetname" "7.motor_control"
 			(at 180.34 18.3384 0)
 			(effects
@@
 			(effects
 				(font
-					(size 1.27 1.27)
-				)
-				(justify left top)
-			)
-		)
-		(instances
-			(project "bldc_motor_controller"
-				(path "/a25adab6-a8c3-4e0e-8ba9-baac00aaa394"
-					(page "10")
-				)
-			)
-		)
-	)
-	(sheet
-		(at 180.34 62.23)
-		(size 44.45 38.1)
-		(exclude_from_sim no)
-		(in_bom yes)
-		(on_board yes)
-		(dnp no)
-		(fields_autoplaced yes)
-		(stroke
-			(width 0.1524)
-			(type solid)
-		)
-		(fill
-			(color 0 0 0 0.0000)
-		)
-		(property "Sheetname" "8.motor_control2"
-			(at 180.34 61.5184 0)
-			(effects
-				(font
-					(size 1.27 1.27)
-				)
-				(justify left bottom)
-			)
-		)
-		(property "Sheetfile" "motor_control2.kicad_sch"
-			(at 180.34 100.9146 0)
-			(effects
-				(font

Commit message: 중간 저장
Changed lines of the file:
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@@
 	)
 	(sheet
-		(at 180.34 106.68)
+		(at 180.34 60.96)
 		(size 44.45 38.1)
 		(exclude_from_sim no)
@@
 		)
 		(property "Sheetname" "9.motor_sense"
-			(at 180.34 105.9684 0)
+			(at 180.34 60.2484 0)
 			(effects
 				(font
@@
 		)
 		(property "Sheetfile" "motor_sense.kicad_sch"
-			(at 180.34 145.3646 0)
+			(at 180.34 99.6446 0)
 			(effects
 				(font
