File: 1.hardware/memory.kicad_sch (KiCad schematic)
At the start: 2 parts, among them IC1 IS42S32800J-6TLI, U2 NC_IS42S16400J-xC

Commit message: 중간 저장
Other:
- moved on the sheet: IC1
Changed lines of the file:
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@@
 	(symbol
 		(lib_id "SamacSys_Parts:IS42S32800J-6TLI")
-		(at 259.08 73.66 0)
+		(at 233.68 72.39 0)
 		(unit 1)
 		(exclude_from_sim no)
@@
 		(fields_autoplaced yes)
 		(property "Reference" "IC1"
-			(at 275.59 66.04 0)
+			(at 250.19 64.77 0)
 			(effects
 				(font
@@
 		)
 		(property "Value" "IS42S32800J-6TLI"
-			(at 275.59 68.58 0)
+			(at 250.19 67.31 0)
 			(effects
 				(font
@@
 		)
 		(property "Footprint" "SOP50P1176X120-86N"
-			(at 288.29 71.12 0)
+			(at 262.89 69.85 0)
 			(effects
 				(font
@@
 		)
 		(property "Datasheet" "https://www.arrow.com/en/products/is42s32800j-6tli/integrated-silicon-solution-inc?region=nac"
-			(at 288.29 73.66 0)
+			(at 262.89 72.39 0)
 			(effects
 				(font
@@
 		)
 		(property "Description" "DRAM 256M, 3.3V, SDRAM, 8Mx32, 166Mhz, 86 pin TSOP II RoHS, IT"
-			(at 259.08 73.66 0)
+			(at 233.68 72.39 0)
 			(effects
 				(font
@@
 		)
 		(property "Description_1" "DRAM 256M, 3.3V, SDRAM, 8Mx32, 166Mhz, 86 pin TSOP II RoHS, IT"
-			(at 288.29 76.2 0)
+			(at 262.89 74.93 0)
 			(effects
 				(font
@@
 		)
 		(property "Height" "1.2"
-			(at 288.29 78.74 0)
+			(at 262.89 77.47 0)
 			(effects
 				(font
@@
 		)
 		(property "Manufacturer_Name" "Integrated Silicon Solution Inc."
-			(at 288.29 81.28 0)
+			(at 262.89 80.01 0)
 			(effects
 				(font
@@
 		)
 		(property "Manufacturer_Part_Number" "IS42S32800J-6TLI"
-			(at 288.29 83.82 0)
+			(at 262.89 82.55 0)
 			(effects
 				(font
@@
 		)
 		(property "Mouser Part Number" "N/A"
-			(at 288.29 86.36 0)
+			(at 262.89 85.09 0)
 			(effects
 				(font
@@
 		)
 		(property "Mouser Price/Stock" "https://www.mouser.com/Search/Refine.aspx?Keyword=N%2FA"
-			(at 288.29 88.9 0)
+			(at 262.89 87.63 0)
 			(effects
 				(font
@@
 		)
 		(property "Arrow Part Number" "IS42S32800J-6TLI"
-			(at 288.29 91.44 0)
+			(at 262.89 90.17 0)
 			(effects
 				(font
@@
 		)
 		(property "Arrow Price/Stock" "https://www.arrow.com/en/products/is42s32800j-6tli/integrated-silicon-solution-inc?utm_currency=USD&region=nac"
-			(at 288.29 93.98 0)
+			(at 262.89 92.71 0)
 			(effects
 				(font

Commit message: 중간 저장2
Parts:
- added C52, C53, C54, C56, C57, C58, C59: 0.1uF/16V, Capacitor_SMD:C_0402_1005Metric, symbol Device:C_Small_US
- added C55: 2.2uF/6.3V, Capacitor_SMD:C_0603_1608Metric, symbol Device:C_Small_US
- added R23, R24, R25, R26, R27, R28, R29, R30, R31, R32, R33, R34, R35, R36, R37, R38, R39, R40, R41, R42, R43, R44, R45, R46, R47, R48, R49, R50, R51, R52, R53, R54, R55, R56, R57, R58, R59, R60, R61, R62, R63, R64, R65, R66, R67, R68, R69, R70, R71, R72, R73, R74, R75, R76, R77, R78: 33R/0.063w, symbol Device:R_Small_US
- U2: now not fitted; now left out of the parts list
Connections:
- net FMC_A0: now also R55.1
- net FMC_A1: now also R56.1
- net FMC_A10: now also R65.1
- net FMC_A11: now also R66.1
- net FMC_A2: now also R57.1
- net FMC_A3: now also R58.1
- net FMC_A4: now also R59.1
- net FMC_A5: now also R60.1
- net FMC_A6: now also R61.1
- net FMC_A7: now also R62.1
- net FMC_A8: now also R63.1
- net FMC_A9: now also R64.1
- net FMC_BA0: now also R67.1
- net FMC_BA1: now also R68.1
- net FMC_D0: now also R23.1
- net FMC_D1: now also R24.1
- net FMC_D10: now also R33.1
- net FMC_D11: now also R34.1
- net FMC_D12: now also R35.1
- net FMC_D13: now also R36.1
- net FMC_D14: now also R37.1
- net FMC_D15: now also R38.1
- net FMC_D16: now also R39.1
- net FMC_D17: now also R40.1
- net FMC_D18: now also R41.1
- net FMC_D19: now also R42.1
- net FMC_D2: now also R25.1
- net FMC_D20: now also R43.1
- net FMC_D21: now also R44.1
- net FMC_D22: now also R45.1
- net FMC_D23: now also R46.1
- net FMC_D24: now also R47.1
- net FMC_D25: now also R48.1
- net FMC_D26: now also R49.1
- net FMC_D27: now also R50.1
- net FMC_D28: now also R51.1
- net FMC_D29: now also R52.1
- net FMC_D3: now also R26.1
- net FMC_D30: now also R53.1
- net FMC_D31: now also R54.1
- net FMC_D4: now also R27.1
- net FMC_D5: now also R28.1
- net FMC_D6: now also R29.1
- net FMC_D7: now also R30.1
- net FMC_D8: now also R31.1
- net FMC_D9: now also R32.1
- net FMC_NBL0: now also R75.1
- net FMC_NBL1: now also R76.1
- net FMC_NBL2: now also R77.1
- net FMC_NBL3: now also R78.1
- net FMC_SDCKE0: now also R70.1
- net FMC_SDCLK: now also R72.1
- net FMC_SDNCAS: now also R73.1
- net FMC_SDNE0: now also R69.1
- net FMC_SDNRAS: now also R71.1
- net 3V3_MCU: now reaches U2.1 (VDD), U2.14 (VDD), U2.27 (VDD)
- net 3V3_MCU: now also IC1.1 (VDD_1), IC1.15 (VDD_2), IC1.29 (VDD_3), IC1.3 (VDDQ_1), IC1.35 (VDDQ_3), IC1.41 (VDDQ_4), IC1.49 (VDDQ_5), IC1.55 (VDDQ_6), IC1.75 (VDDQ_7), IC1.81 (VDDQ_8), IC1.9 (VDDQ_2), U2.3 (VDDQ), U2.43 (VDDQ), U2.49 (VDDQ), U2.9 (VDDQ), C52.1, C53.1, C54.1, C55.1, C56.1, C57.1, C58.1, C59.1
- net SDRAM_DQ5: now reaches U2.10 (DQ5)
- net SDRAM_DQ5: now also IC1.10 (DQ5), R28.2
- net SDRAM_DQ6: now reaches U2.11 (DQ6)
- net SDRAM_DQ6: now also IC1.11 (DQ6), R29.2
- net GND: now reaches U2.12 (GNDQ), U2.46 (GNDQ), U2.52 (GNDQ), U2.6 (GNDQ)
- net GND: now also IC1.12 (VSSQ_2), IC1.32 (VSSQ_3), IC1.38 (VSSQ_4), IC1.44 (VSS_1), IC1.46 (VSSQ_5), IC1.52 (VSSQ_6), IC1.58 (VSS_2), IC1.6 (VSSQ_1), IC1.72 (VSS_3), IC1.78 (VSSQ_7), IC1.84 (VSSQ_8), IC1.86 (VSS_4), U2.28 (GND), U2.41 (GND), U2.54 (GND), C52.2, C53.2, C54.2, C55.2, C56.2, C57.2, C58.2, C59.2
- net SDRAM_DQ7: now reaches U2.13 (DQ7)
- net SDRAM_DQ7: now also IC1.13 (DQ7), R30.2
- net SDRAM_WE: now reaches U2.16 (~{WE})
- net SDRAM_WE: now also IC1.17 (~{WE}), R74.2
- net SDRAM_CAS: now reaches U2.17 (~{CAS})
- net SDRAM_CAS: now also IC1.18 (~{CAS}), R73.2
- net SDRAM_RAS: now reaches U2.18 (~{RAS})
- net SDRAM_RAS: now also IC1.19 (~{RAS}), R71.2
- net SDRAM_CS: now reaches U2.19 (~{CS})
- net SDRAM_CS: now also IC1.20 (~{CS}), R69.2
- net SDRAM_DQ0: now reaches U2.2 (DQ0)
- net SDRAM_DQ0: now also IC1.2 (DQ0), R23.2
- net SDRAM_BA0: now reaches U2.20 (BA0)
- net SDRAM_BA0: now also IC1.22 (BA0), R67.2
- net SDRAM_BA1: now reaches U2.21 (BA1)
- net SDRAM_BA1: now also IC1.23 (BA1), R68.2
- net SDRAM_A10: now reaches U2.22 (A10)
- net SDRAM_A10: now also IC1.24 (A10), R65.2
- net SDRAM_A0: now reaches U2.23 (A0)
- net SDRAM_A0: now also IC1.25 (A0), R55.2
- net SDRAM_A1: now reaches U2.24 (A1)
- net SDRAM_A1: now also IC1.26 (A1), R56.2
- net SDRAM_A2: now reaches U2.25 (A2)
- net SDRAM_A2: now also IC1.27 (A2), R57.2
- net SDRAM_A3: now reaches U2.26 (A3)
- net SDRAM_A3: now also IC1.60 (A3), R58.2
- net SDRAM_A4: now reaches U2.29 (A4)
- net SDRAM_A4: now also IC1.61 (A4), R59.2
- net SDRAM_A5: now reaches U2.30 (A5)
- net SDRAM_A5: now also IC1.62 (A5), R60.2
- net SDRAM_A6: now reaches U2.31 (A6)
- net SDRAM_A6: now also IC1.63 (A6), R61.2
- net SDRAM_A7: now reaches U2.32 (A7)
- net SDRAM_A7: now also IC1.64 (A7), R62.2
- net SDRAM_A8: now reaches U2.33 (A8)
- net SDRAM_A8: now also IC1.65 (A8), R63.2
- net SDRAM_A9: now reaches U2.34 (A9)
- net SDRAM_A9: now also IC1.66 (A9), R64.2
- net SDRAM_A11: now reaches U2.35 (A11)
- net SDRAM_A11: now also IC1.21 (A11), R66.2
- net SDRAM_CKE: now reaches U2.37 (CKE)
- net SDRAM_CKE: now also IC1.67 (CKE), R70.2
- net SDRAM_CLK: now reaches U2.38 (CLK)
- net SDRAM_CLK: now also IC1.68 (CLK), R72.2
- net SDRAM_DQ1: now reaches U2.4 (DQ1)
- net SDRAM_DQ1: now also IC1.4 (DQ1), R24.2
- net SDRAM_DQ8: now reaches U2.42 (DQ8)
- net SDRAM_DQ8: now also IC1.74 (DQ8), R31.2
- net SDRAM_DQ9: now reaches U2.44 (DQ9)
- net SDRAM_DQ9: now also IC1.76 (DQ9), R32.2
- net SDRAM_DQ10: now reaches U2.45 (DQ10)
- net SDRAM_DQ10: now also IC1.77 (DQ10), R33.2
- net SDRAM_DQ11: now reaches U2.47 (DQ11)
- net SDRAM_DQ11: now also IC1.79 (DQ11), R34.2
- net SDRAM_DQ12: now reaches U2.48 (DQ12)
- net SDRAM_DQ12: now also IC1.80 (DQ12), R35.2
- net SDRAM_DQ2: now reaches U2.5 (DQ2)
- net SDRAM_DQ2: now also IC1.5 (DQ2), R25.2
- net SDRAM_DQ13: now reaches U2.50 (DQ13)
- net SDRAM_DQ13: now also IC1.82 (DQ13), R36.2
- net SDRAM_DQ14: now reaches U2.51 (DQ14)
- net SDRAM_DQ14: now also IC1.83 (DQ14), R37.2
- net SDRAM_DQ15: now reaches U2.53 (DQ15)
- net SDRAM_DQ15: now also IC1.85 (DQ15), R38.2
- net SDRAM_DQ3: now reaches U2.7 (DQ3)
- net SDRAM_DQ3: now also IC1.7 (DQ3), R26.2
- net SDRAM_DQ4: now reaches U2.8 (DQ4)
- net SDRAM_DQ4: now also IC1.8 (DQ4), R27.2
- net SDRAM_DQM0: now reaches IC1.16 (DQM0)
- net SDRAM_DQM0: now also R75.2
- net SDRAM_DQM2: now reaches IC1.28 (DQM2)
- net SDRAM_DQM2: now also R77.2
- net SDRAM_DQ16: now reaches IC1.31 (DQ16)
- net SDRAM_DQ16: now also R39.2
- net SDRAM_DQ17: now reaches IC1.33 (DQ17)
- net SDRAM_DQ17: now also R40.2
- net SDRAM_DQ18: now reaches IC1.34 (DQ18)
- net SDRAM_DQ18: now also R41.2
- net SDRAM_DQ19: now reaches IC1.36 (DQ19)
- net SDRAM_DQ19: now also R42.2
- net SDRAM_DQ20: now reaches IC1.37 (DQ20)
- net SDRAM_DQ20: now also R43.2
- net SDRAM_DQ21: now reaches IC1.39 (DQ21)
- net SDRAM_DQ21: now also R44.2
- net SDRAM_DQ22: now reaches IC1.40 (DQ22)
- net SDRAM_DQ22: now also R45.2
- net SDRAM_DQ23: now reaches IC1.42 (DQ23)
- net SDRAM_DQ23: now also R46.2
- net SDRAM_DQ24: now reaches IC1.45 (DQ24)
- net SDRAM_DQ24: now also R47.2
- net SDRAM_DQ25: now reaches IC1.47 (DQ25)
- net SDRAM_DQ25: now also R48.2
- net SDRAM_DQ26: now reaches IC1.48 (DQ26)
- net SDRAM_DQ26: now also R49.2
- net SDRAM_DQ27: now reaches IC1.50 (DQ27)
- net SDRAM_DQ27: now also R50.2
- net SDRAM_DQ28: now reaches IC1.51 (DQ28)
- net SDRAM_DQ28: now also R51.2
- net SDRAM_DQ29: now reaches IC1.53 (DQ29)
- net SDRAM_DQ29: now also R52.2
- net SDRAM_DQ30: now reaches IC1.54 (DQ30)
- net SDRAM_DQ30: now also R53.2
- net SDRAM_DQ31: now reaches IC1.56 (DQ31)
- net SDRAM_DQ31: now also R54.2
- net SDRAM_DQM3: now reaches IC1.59 (DQM3)
- net SDRAM_DQM3: now also R78.2
- net SDRAM_DQM1: now reaches IC1.71 (DQM1)
- net SDRAM_DQM1: now also R76.2
- new net FMC_SDNWE: R74.1
- no-connect marks 0 -> 6
Other:
- moved on the sheet: IC1

Commit message: 중간 수정
Parts:
- added C24: 0.1uF/16V, Capacitor_SMD:C_0402_1005Metric, symbol Device:C_Small_US
- added U6: W25Q128JVS, Package_SO:SOIC-8_5.3x5.3mm_P1.27mm, symbol Memory_Flash:W25Q128JVS
Connections:
- net 3V3_MCU: now also C24.1, U6.8 (VCC)
- net GND: now also C24.2, U6.4 (GND)

Commit message: 중간 저장
Parts:
- added C57, C58: 0.1uF/16V, Capacitor_SMD:C_0402_1005Metric, symbol Device:C_Small_US
- added C59: 2.2uF/6.3V, Capacitor_SMD:C_0603_1608Metric, symbol Device:C_Small_US
- added R100, R99: 10k/0.063w, symbol Device:R_Small_US
- renumbered C24 to C41, C52 to C42, C56 to C43, C53 to C44, C57 to C45, C54 to C46, C58 to C47, C55 to C48, C59 to C49, IC1 to IC2, R55 to R34, R56 to R35, R57 to R36, R58 to R37, R59 to R38, R60 to R39, R61 to R40, R62 to R41, R63 to R42, R64 to R43, R65 to R44, R66 to R45, R67 to R46, R68 to R47, R69 to R48, R70 to R49, R71 to R50, R72 to R51, R73 to R52, R74 to R53, R75 to R54, R76 to R55, R77 to R56, R78 to R57, R23 to R58, R24 to R59, R25 to R60, R26 to R61, R27 to R62, R28 to R63, R29 to R64, R30 to R65, R31 to R66, R32 to R67, R33 to R68, R34 to R69, R35 to R70, R36 to R71, R37 to R72, R38 to R73, R39 to R74, R40 to R75, R41 to R76, R42 to R77, R43 to R78, R44 to R79, R45 to R80, R46 to R81, R47 to R82, R48 to R83, R49 to R84, R50 to R85, R51 to R86, R52 to R87, R53 to R88, R54 to R89, U6 to U3, U2 to U4
Connections:
- net 3V3_MCU: now also C57.1, C58.1, C59.1, R100.1, R99.1
- net GND: now also C57.2, C58.2, C59.2
- net W25q_FLASH_SPI1_NSS: now reaches U3.1 (~{CS})
- net W25q_FLASH_SPI1_MISO: now reaches U3.2 (DO/IO_{1})
- net at U3.3 (~{WP}/IO_{2}): now also R99.2
- net W25q_FLASH_SPI1_MOSI: now reaches U3.5 (DI/IO_{0})
- net W25q_FLASH_SPI1_SCK: now reaches U3.6 (CLK)
- net at U3.7 (~{HOLD}/~{RESET}/IO_{3}): now also R100.2
Other:
- moved on the sheet: C41, U3

Commit message: 중간 저장
Parts:
- IC2: footprint SOP50P1176X120-86N -> SamacSys_Parts:SOP50P1176X120-86N
- R100, R34, R35, R36, R37, R38, R39, R40, R41, R42, R43, R44, R45, R46, R47, R48, R49, R50, R51, R52, R53, R54, R55, R56, R57, R58, R59, R60, R61, R62, R63, R64, R65, R66, R67, R68, R69, R70, R71, R72, R73, R74, R75, R76, R77, R78, R79, R80, R81, R82, R83, R84, R85, R86, R87, R88, R89, R99: footprint (none) -> Resistor_SMD:R_0402_1005Metric
Changed lines of the file:
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@@
 			)
 		)
-		(property "Footprint" ""
+		(property "Footprint" "Resistor_SMD:R_0402_1005Metric"
 			(at 242.57 128.27 0)
 			(effects
@@
 			)
 		)
-		(property "Footprint" ""
+		(property "Footprint" "Resistor_SMD:R_0402_1005Metric"
 			(at 242.57 110.49 0)
 			(effects
@@
 			)
 		)
-		(property "Footprint" ""
+		(property "Footprint" "Resistor_SMD:R_0402_1005Metric"
 			(at 201.93 158.75 0)
 			(effects
@@
 			)
 		)
-		(property "Footprint" ""
+		(property "Footprint" "Resistor_SMD:R_0402_1005Metric"
 			(at 242.57 148.59 0)
 			(effects
@@
 			)
 		)
-		(property "Footprint" ""
+		(property "Footprint" "Resistor_SMD:R_0402_1005Metric"
 			(at 201.93 135.89 0)
 			(effects
@@
 			)
 		)
-		(property "Footprint" ""
+		(property "Footprint" "Resistor_SMD:R_0402_1005Metric"
 			(at 242.57 133.35 0)
 			(effects
@@
 			)
 		)
-		(property "Footprint" ""
+		(property "Footprint" "Resistor_SMD:R_0402_1005Metric"
 			(at 242.57 125.73 0)
 			(effects
@@
 			)
 		)
-		(property "Footprint" ""
+		(property "Footprint" "Resistor_SMD:R_0402_1005Metric"
 			(at 201.93 120.65 0)
 			(effects
@@
 			)
 		)
-		(property "Footprint" ""
+		(property "Footprint" "Resistor_SMD:R_0402_1005Metric"
 			(at 242.57 171.45 0)
 			(effects
@@
 			)
 		)
-		(property "Footprint" ""
+		(property "Footprint" "Resistor_SMD:R_0402_1005Metric"
 			(at 242.57 123.19 0)
 			(effects
@@
 			)
 		)
-		(property "Footprint" ""
+		(property "Footprint" "Resistor_SMD:R_0402_1005Metric"
 			(at 242.57 138.43 0)
 			(effects
@@
 			)
 		)
-		(property "Footprint" ""
+		(property "Footprint" "Resistor_SMD:R_0402_1005Metric"
 			(at 242.57 163.83 0)
 			(effects
@@
 			)
 		)
-		(property "Footprint" ""
+		(property "Footprint" "Resistor_SMD:R_0402_1005Metric"
 			(at 242.57 158.75 0)
 			(effects
@@
 			)
 		)
-		(property "Footprint" ""
+		(property "Footprint" "Resistor_SMD:R_0402_1005Metric"
 			(at 242.57 151.13 0)
 			(effects
@@
 			)
 		)
-		(property "Footprint" ""
+		(property "Footprint" "Resistor_SMD:R_0402_1005Metric"
 			(at 201.93 118.11 0)
 			(effects
@@
 			)
 		)
-		(property "Footprint" ""
+		(property "Footprint" "Resistor_SMD:R_0402_1005Metric"
 			(at 201.93 163.83 0)
 			(effects
@@
 			)
 		)
-		(property "Footprint" ""
+		(property "Footprint" "Resistor_SMD:R_0402_1005Metric"
 			(at 201.93 148.59 0)
 			(effects
@@
 			)
 		)
-		(property "Footprint" ""
+		(property "Footprint" "Resistor_SMD:R_0402_1005Metric"
 			(at 242.57 102.87 0)
 			(effects
@@
 			)
 		)
-		(property "Footprint" ""
+		(property "Footprint" "Resistor_SMD:R_0402_1005Metric"
 			(at 242.57 113.03 0)
 			(effects
@@
 			)
 		)
-		(property "Footprint" ""
+		(property "Footprint" "Resistor_SMD:R_0402_1005Metric"
 			(at 201.93 115.57 0)
 			(effects
@@
 			)
 		)
-		(property "Footprint" ""
+		(property "Footprint" "Resistor_SMD:R_0402_1005Metric"
 			(at 81.28 107.95 0)
 			(effects
@@
 			)
 		)
-		(property "Footprint" ""
+		(property "Footprint" "Resistor_SMD:R_0402_1005Metric"
 			(at 201.93 140.97 0)
 			(effects
@@
 			)
 		)
-		(property "Footprint" ""
+		(property "Footprint" "Resistor_SMD:R_0402_1005Metric"
 			(at 242.57 97.79 0)
 			(effects
@@
 			)
 		)
-		(property "Footprint" ""
+		(property "Footprint" "Resistor_SMD:R_0402_1005Metric"
 			(at 201.93 105.41 0)
 			(effects
@@
 			)
 		)
-		(property "Footprint" ""
+		(property "Footprint" "Resistor_SMD:R_0402_1005Metric"
 			(at 242.57 146.05 0)
 			(effects
@@
 			)
 		)
-		(property "Footprint" ""
+		(property "Footprint" "Resistor_SMD:R_0402_1005Metric"
 			(at 242.57 120.65 0)
 			(effects
@@
 			)
 		)
-		(property "Footprint" ""
+		(property "Footprint" "Resistor_SMD:R_0402_1005Metric"
 			(at 201.93 156.21 0)
 			(effects
@@
 			)
 		)
-		(property "Footprint" ""
+		(property "Footprint" "Resistor_SMD:R_0402_1005Metric"
 			(at 242.57 166.37 0)
 			(effects
@@
 			)
 		)
-		(property "Footprint" ""
+		(property "Footprint" "Resistor_SMD:R_0402_1005Metric"
 			(at 242.57 173.99 0)
 			(effects
@@
 			)
 		)
-		(property "Footprint" ""
+		(property "Footprint" "Resistor_SMD:R_0402_1005Metric"
 			(at 201.93 107.95 0)
 			(effects
@@
 			)
 		)
-		(property "Footprint" ""
+		(property "Footprint" "Resistor_SMD:R_0402_1005Metric"
 			(at 242.57 143.51 0)
 			(effects
@@
 			)
 		)
-		(property "Footprint" ""
+		(property "Footprint" "Resistor_SMD:R_0402_1005Metric"
 			(at 242.57 130.81 0)
 			(effects
@@
 			)
 		)
-		(property "Footprint" ""
+		(property "Footprint" "Resistor_SMD:R_0402_1005Metric"
 			(at 242.57 168.91 0)
 			(effects
@@
 			)
 		)
-		(property "Footprint" ""
+		(property "Footprint" "Resistor_SMD:R_0402_1005Metric"
 			(at 93.98 104.14 0)
 			(effects
@@
 			)
 		)
-		(property "Footprint" ""
+		(property "Footprint" "Resistor_SMD:R_0402_1005Metric"
 			(at 201.93 102.87 0)
 			(effects
@@
 			)
 		)
-		(property "Footprint" ""
+		(property "Footprint" "Resistor_SMD:R_0402_1005Metric"
 			(at 201.93 128.27 0)
 			(effects
@@
 			)
 		)
-		(property "Footprint" ""
+		(property "Footprint" "Resistor_SMD:R_0402_1005Metric"
 			(at 242.57 153.67 0)
 			(effects
@@
 			)
 		)
-		(property "Footprint" ""
+		(property "Footprint" "Resistor_SMD:R_0402_1005Metric"
 			(at 201.93 161.29 0)
 			(effects
@@
 			)
 		)
-		(property "Footprint" ""
+		(property "Footprint" "Resistor_SMD:R_0402_1005Metric"
 			(at 201.93 130.81 0)
 			(effects
@@
 			)
 		)
-		(property "Footprint" ""
+		(property "Footprint" "Resistor_SMD:R_0402_1005Metric"
 			(at 201.93 123.19 0)
 			(effects
@@
 			)
 		)
-		(property "Footprint" ""
+		(property "Footprint" "Resistor_SMD:R_0402_1005Metric"
 			(at 201.93 146.05 0)
 			(effects
@@
 			)
 		)
-		(property "Footprint" ""
+		(property "Footprint" "Resistor_SMD:R_0402_1005Metric"
 			(at 201.93 113.03 0)
 			(effects
@@
 			)
 		)
-		(property "Footprint" ""
+		(property "Footprint" "Resistor_SMD:R_0402_1005Metric"
 			(at 201.93 138.43 0)
 			(effects
@@
 			)
 		)
-		(property "Footprint" ""
+		(property "Footprint" "Resistor_SMD:R_0402_1005Metric"
 			(at 242.57 135.89 0)
 			(effects
@@
 			)
 		)
-		(property "Footprint" ""
+		(property "Footprint" "Resistor_SMD:R_0402_1005Metric"
 			(at 242.57 115.57 0)
 			(effects
@@
 			)
 		)
-		(property "Footprint" ""
+		(property "Footprint" "Resistor_SMD:R_0402_1005Metric"
 			(at 242.57 95.25 0)
 			(effects
@@
 			)
 		)
-		(property "Footprint" ""
+		(property "Footprint" "Resistor_SMD:R_0402_1005Metric"
 			(at 242.57 118.11 0)
 			(effects
@@
 			)
 		)
-		(property "Footprint" ""
+		(property "Footprint" "Resistor_SMD:R_0402_1005Metric"
 			(at 242.57 100.33 0)
 			(effects
@@
 			)
 		)
-		(property "Footprint" ""
+		(property "Footprint" "Resistor_SMD:R_0402_1005Metric"
 			(at 201.93 143.51 0)
 			(effects
@@
 			)
 		)
-		(property "Footprint" ""
+		(property "Footprint" "Resistor_SMD:R_0402_1005Metric"
 			(at 242.57 161.29 0)
 			(effects
@@
 			)
 		)
-		(property "Footprint" ""
+		(property "Footprint" "Resistor_SMD:R_0402_1005Metric"
 			(at 242.57 105.41 0)
 			(effects
@@
 			)
 		)
-		(property "Footprint" ""
+		(property "Footprint" "Resistor_SMD:R_0402_1005Metric"
 			(at 201.93 95.25 0)
 			(effects
@@
 			)
 		)
-		(property "Footprint" ""
+		(property "Footprint" "Resistor_SMD:R_0402_1005Metric"
 			(at 242.57 156.21 0)
 			(effects
@@
 			)
 		)
-		(property "Footprint" ""
+		(property "Footprint" "Resistor_SMD:R_0402_1005Metric"
 			(at 201.93 100.33 0)
 			(effects
@@
 			)
 		)
-		(property "Footprint" "SOP50P1176X120-86N"
+		(property "Footprint" "SamacSys_Parts:SOP50P1176X120-86N"
 			(at 384.81 77.47 0)
 			(effects
@@
 			)
 		)
-		(property "Footprint" ""
+		(property "Footprint" "Resistor_SMD:R_0402_1005Metric"
 			(at 242.57 140.97 0)
 			(effects
@@
 			)
 		)
-		(property "Footprint" ""
+		(property "Footprint" "Resistor_SMD:R_0402_1005Metric"
 			(at 201.93 110.49 0)
 			(effects
@@
 			)
 		)
-		(property "Footprint" ""
+		(property "Footprint" "Resistor_SMD:R_0402_1005Metric"
 			(at 201.93 97.79 0)
 			(effects
@@
 			)
 		)
-		(property "Footprint" ""
+		(property "Footprint" "Resistor_SMD:R_0402_1005Metric"
 			(at 242.57 107.95 0)
 			(effects

Commit message: 핀 배치 완료
Parts:
- removed R100, R99: 10k/0.063w, Resistor_SMD:R_0402_1005Metric, symbol Device:R_Small_US
Changed lines of the file:
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@@
 	)
 	(junction
-		(at 93.98 96.52)
-		(diameter 0)
-		(color 0 0 0 0)
-	)
-	(junction
 		(at 140.97 96.52)
 		(diameter 0)
@@
 	(wire
 		(pts
-			(xy 93.98 106.68) (xy 93.98 124.46)
-		)
-		(stroke
-			(width 0)
-			(type default)
-		)
-	)
-	(wire
-		(pts
 			(xy 204.47 72.39) (xy 204.47 74.93)
 		)
@@
 	(wire
 		(pts
-			(xy 93.98 96.52) (xy 107.95 96.52)
+			(xy 81.28 96.52) (xy 107.95 96.52)
 		)
 		(stroke
@@
 	(wire
 		(pts
-			(xy 93.98 96.52) (xy 93.98 101.6)
-		)
-		(stroke
-			(width 0)
-			(type default)
-		)
-	)
-	(wire
-		(pts
 			(xy 350.52 146.05) (xy 355.6 146.05)
 		)
@@
 	(wire
 		(pts
-			(xy 81.28 127) (xy 97.79 127)
-		)
-		(stroke
-			(width 0)
-			(type default)
-		)
-	)
-	(wire
-		(pts
 			(xy 300.99 99.06) (xy 300.99 92.71)
 		)
@@
 	(wire
 		(pts
-			(xy 81.28 105.41) (xy 81.28 96.52)
-		)
-		(stroke
-			(width 0)
-			(type default)
-		)
-	)
-	(wire
-		(pts
 			(xy 200.66 72.39) (xy 204.47 72.39)
 		)
@@
 	(wire
 		(pts
-			(xy 81.28 110.49) (xy 81.28 127)
-		)
-		(stroke
-			(width 0)
-			(type default)
-		)
-	)
-	(wire
-		(pts
 			(xy 350.52 135.89) (xy 355.6 135.89)
 		)
@@
 	(wire
 		(pts
-			(xy 81.28 96.52) (xy 93.98 96.52)
-		)
-		(stroke
-			(width 0)
-			(type default)
-		)
-	)
-	(wire
-		(pts
 			(xy 236.22 130.81) (xy 240.03 130.81)
 		)
@@
 	(wire
 		(pts
-			(xy 93.98 124.46) (xy 97.79 124.46)
-		)
-		(stroke
-			(width 0)
-			(type default)
-		)
-	)
-	(wire
-		(pts
 			(xy 285.75 121.92) (xy 288.29 121.92)
 		)
@@
 	(symbol
 		(lib_id "Device:R_Small_US")
-		(at 81.28 107.95 0)
-		(unit 1)
-		(exclude_from_sim no)
-		(in_bom yes)
-		(on_board yes)
-		(dnp no)
-		(property "Reference" "R100"
-			(at 81.28 105.156 0)
-			(effects
-				(font
-					(size 1.27 1.27)
-				)
-				(justify left)
-			)
-		)
-		(property "Value" "10k/0.063w"
-			(at 81.534 109.982 0)
-			(effects
-				(font
-					(size 1.27 1.27)
-				)
-				(justify left)
-			)
-		)
-		(property "Footprint" "Resistor_SMD:R_0402_1005Metric"
-			(at 81.28 107.95 0)
-			(effects
-				(font
-					(size 1.27 1.27)
-				)
-				(hide yes)
-			)
-		)
-		(property "Datasheet" "~"
-			(at 81.28 107.95 0)
-			(effects
-				(font
-					(size 1.27 1.27)
-				)
-				(hide yes)
-			)
-		)
-		(property "Description" "Resistor, small US symbol"
-			(at 81.28 107.95 0)
-			(effects
-				(font
-					(size 1.27 1.27)
-				)
-				(hide yes)
-			)
-		)
-		(pin "1"
-		)
-		(pin "2"
-		)
-		(instances
-			(project "bldc_motor_controller"
-				(path "/a25adab6-a8c3-4e0e-8ba9-baac00aaa394/9f644060-1b86-41d4-818c-d38193d04e6e"
-					(reference "R100")
-					(unit 1)
-				)
-			)
-		)
-	)
-	(symbol
-		(lib_id "Device:R_Small_US")
 		(at 201.93 140.97 90)
 		(unit 1)
@@
 					(unit 1)
 				)
-			)
-		)
-	)
-	(symbol
-		(lib_id "Device:R_Small_US")
-		(at 93.98 104.14 0)
-		(unit 1)
-		(exclude_from_sim no)
-		(in_bom yes)
-		(on_board yes)
-		(dnp no)
-		(property "Reference" "R99"
-			(at 94.488 101.6 0)
-			(effects
-				(font
-					(size 1.27 1.27)
-				)
-				(justify left)
-			)
-		)
-		(property "Value" "10k/0.063w"
-			(at 94.234 106.426 0)
-			(effects
-				(font
-					(size 1.27 1.27)
-				)
-				(justify left)
-			)
-		)
-		(property "Footprint" "Resistor_SMD:R_0402_1005Metric"
-			(at 93.98 104.14 0)
-			(effects
-				(font
-					(size 1.27 1.27)
-				)
-				(hide yes)
-			)
-		)
-		(property "Datasheet" "~"
-			(at 93.98 104.14 0)
-			(effects
-				(font
-					(size 1.27 1.27)
-				)
-				(hide yes)
-			)
-		)
-		(property "Description" "Resistor, small US symbol"
-			(at 93.98 104.14 0)
-			(effects
-				(font
-					(size 1.27 1.27)
-				)
-				(hide yes)
-			)
-		)
-		(pin "1"
-		)
-		(pin "2"
-		)
-		(instances
-			(project "bldc_motor_controller"
-				(path "/a25adab6-a8c3-4e0e-8ba9-baac00aaa394/9f644060-1b86-41d4-818c-d38193d04e6e"
-					(reference "R99")
-					(unit 1)
-				)
