File: 1.hardware/memory.kicad_sch (KiCad schematic)
At the start: 90 parts, among them IC3 IS42S32800J-6TLI, U10 W25Q128JVS, U11 4D02WGJ0330T, U12 4D02WGJ0330T, U13 4D02WGJ0330T, U14 4D02WGJ0330T, U15 4D02WGJ0330T, U16 4D02WGJ0330T, U17 NC_IS42S16400J-xC, U18 4D02WGJ0330T, U19 4D02WGJ0330T, U20 4D02WGJ0330T, U21 4D02WGJ0330T, U6 4D02WGJ0330T, U7 4D02WGJ0330T, U8 4D02WGJ0330T, U9 4D02WGJ0330T

Commit message: 발주 최종버전
Parts:
- U11, U12, U13, U14, U15, U16, U18, U19, U20, U21, U6, U7, U8, U9: footprint footprints:4D02_2X1_ROH -> Library:4D02WGJ0330TCE
Changed lines of the file:
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@@
 			)
 		)
-		(property "Footprint" "footprints:4D02_2X1_ROH"
+		(property "Footprint" "Library:4D02WGJ0330TCE"
 			(at 173.99 50.8 0)
 			(effects
@@
 			)
 		)
-		(property "Footprint" "footprints:4D02_2X1_ROH"
+		(property "Footprint" "Library:4D02WGJ0330TCE"
 			(at 173.99 74.93 0)
 			(effects
@@
 			)
 		)
-		(property "Footprint" "footprints:4D02_2X1_ROH"
+		(property "Footprint" "Library:4D02WGJ0330TCE"
 			(at 250.19 49.53 0)
 			(effects
@@
 			)
 		)
-		(property "Footprint" "footprints:4D02_2X1_ROH"
+		(property "Footprint" "Library:4D02WGJ0330TCE"
 			(at 250.19 99.06 0)
 			(effects
@@
 			)
 		)
-		(property "Footprint" "footprints:4D02_2X1_ROH"
+		(property "Footprint" "Library:4D02WGJ0330TCE"
 			(at 250.19 73.66 0)
 			(effects
@@
 			)
 		)
-		(property "Footprint" "footprints:4D02_2X1_ROH"
+		(property "Footprint" "Library:4D02WGJ0330TCE"
 			(at 173.99 171.45 0)
 			(effects
@@
 			)
 		)
-		(property "Footprint" "footprints:4D02_2X1_ROH"
+		(property "Footprint" "Library:4D02WGJ0330TCE"
 			(at 251.46 147.32 0)
 			(effects
@@
 			)
 		)
-		(property "Footprint" "footprints:4D02_2X1_ROH"
+		(property "Footprint" "Library:4D02WGJ0330TCE"
 			(at 173.99 147.32 0)
 			(effects
@@
 			)
 		)
-		(property "Footprint" "footprints:4D02_2X1_ROH"
+		(property "Footprint" "Library:4D02WGJ0330TCE"
 			(at 227.33 223.52 0)
 			(effects
@@
 			)
 		)
-		(property "Footprint" "footprints:4D02_2X1_ROH"
+		(property "Footprint" "Library:4D02WGJ0330TCE"
 			(at 251.46 123.19 0)
 			(effects
@@
 			)
 		)
-		(property "Footprint" "footprints:4D02_2X1_ROH"
+		(property "Footprint" "Library:4D02WGJ0330TCE"
 			(at 173.99 195.58 0)
 			(effects
@@
 			)
 		)
-		(property "Footprint" "footprints:4D02_2X1_ROH"
+		(property "Footprint" "Library:4D02WGJ0330TCE"
 			(at 251.46 171.45 0)
 			(effects
@@
 			)
 		)
-		(property "Footprint" "footprints:4D02_2X1_ROH"
+		(property "Footprint" "Library:4D02WGJ0330TCE"
 			(at 173.99 99.06 0)
 			(effects
@@
 			)
 		)
-		(property "Footprint" "footprints:4D02_2X1_ROH"
+		(property "Footprint" "Library:4D02WGJ0330TCE"
 			(at 173.99 123.19 0)
 			(effects
