File: 1.hardware/motor_sense.kicad_sch (KiCad schematic)
At the start: 0 parts

Commit message: 중간 저장
Parts:
- added C80, C81, C82, C83, C84, C85, C86, C87, C88, C89, C90, C91, C92, C93, C94, C95, C96, C97, C98: 0.1uF/16V, symbol Device:C_Small_US
- added IC4, IC5: SN74HC266DRG4, SOIC127P600X175-14N, symbol SamacSys_Parts:SN74HC266DRG4
- added IC6: SN74LVC3G17DCTRG4, SOP65P400X130-8N, symbol SamacSys_Parts:SN74LVC3G17DCTRG4
- added IC9: SN74HC74PWRG4, SOP65P640X120-14N, symbol SamacSys_Parts:SN74HC74PWRG4
- added R126, R127, R128, R156, R157, R158: 22/0.063w, Resistor_SMD:R_0402_1005Metric, symbol Device:R_Small_US
- added R129, R130, R131, R132, R134, R136, R159, R160: 100k/0.063w, Resistor_SMD:R_0402_1005Metric, symbol Device:R_Small_US
- added R133, R135, R137, R153, R154, R155: 5k/0.063w, Resistor_SMD:R_0402_1005Metric, symbol Device:R_Small_US
- added R161, R162, R163, R164, R165, R166: 10k/0.063w, Resistor_SMD:R_0402_1005Metric, symbol Device:R_Small_US
- added R167, R168, R169: 10k/0.125w, Resistor_SMD:R_0402_1005Metric, symbol Device:R_Small_US
- added U12, U7, U8: TLV9064, symbol Amplifier_Operational:TLV9064
- added U6: TLV9064, PCM_4ms_Package_SSOP:TSSOP-14_4.4x5mm_P0.65mm, symbol Amplifier_Operational:TLV9064
Connections:
- new net: R128.1, U8.8
- new net: C90.1, R131.2, R155.1, U12.6 (-), U12.9 (-)
- new net: C86.1, R134.2, R135.1, U8.10 (+), U8.2 (-)
- new net: C87.1, R136.2, R137.1, U8.6 (-), U8.9 (-)
- new net: C96.1, R161.2, U7.3 (+)
- new net: C93.1, IC6.1 (1A), R159.2
- new net: C94.1, IC6.3 (2A), R160.2
- new net: IC5.3 (1Y), IC5.5 (2A)
- new net: IC4.3 (1Y), IC4.5 (2A)
- new net: C88.1, R129.2, R153.1, U12.3 (+), U12.5 (+)
- new net: R157.1, U12.7
- new net: C85.1, R132.2, R133.1, U8.3 (+), U8.5 (+)
- new net: R127.1, U8.7
- new net: R156.1, U12.1
- new net: R167.2, U7.1
- new net: R162.2, R167.1, U7.2 (-)
- new net: R164.2, R168.1, U7.6 (-)
- new net: R168.2, U7.7
- new net: C98.1, R165.2, U7.10 (+)
- new net: R166.2, R169.1, U7.9 (-)
- new net: C89.1, R130.2, R154.1, U12.10 (+), U12.2 (-)
- new net: R158.1, U12.8
- new net: R126.1, U8.1
- new net: R169.2, U7.8
- new net: C97.1, R163.2, U7.5 (+)
- new net 3V3_MCU: C83.1, C84.1, C91.1, C92.1, C95.1, IC4.14 (VCC), IC5.14 (VCC), IC6.8 (VCC), U12.4 (V+), U8.4 (V+)
- new net 5V: C82.1, IC9.1 (~{1CLR}), IC9.10 (2~{PRE}), IC9.13 (2~{CLR}), IC9.14 (VCC), IC9.4 (1~{PRE})
- new net ADC_VREF_2V5: C80.1, C81.1, U6.4 (V+), U7.4 (V+)
- new net GND: C80.2, C81.2, C82.2, C83.2, C84.2, C85.2, C86.2, C87.2, C88.2, C89.2, C90.2, C91.2, C92.2, C93.2, C94.2, C95.2, C96.2, C97.2, C98.2, IC4.7 (GND), IC5.7 (GND), IC6.4 (GND), IC9.7 (GND), R133.2, R135.2, R137.2, R153.2, R154.2, R155.2, U12.11 (V-), U6.11 (V-), U7.11 (V-), U8.11 (V-)
- new net HALL1_3x_Late_Sig: IC5.9 (3B), IC6.7 (1Y)
- new net HALL1_3x_Sig: IC5.4 (2Y), IC5.8 (3A), R159.1
- new net HALL1_6x_Pulse_Sig: IC5.10 (3Y)
- new net HALL1_A: IC5.1 (1A), IC9.2 (1D)
- new net HALL1_B: IC5.2 (1B), IC9.3 (1CLK)
- new net HALL1_C: IC5.6 (2B)
- new net HALL2_3x_Late_Sig: IC4.9 (3B), IC6.5 (2Y)
- new net HALL2_3x_Sig: IC4.4 (2Y), IC4.8 (3A), R160.1
- new net HALL2_6x_Pulse_Sig: IC4.10 (3Y)
- new net HALL2_A: IC4.1 (1A), IC9.12 (2D)
- new net HALL2_B: IC4.2 (1B), IC9.11 (2CLK)
- new net HALL2_C: IC4.6 (2B)
- new net MOTOR1_DIR: IC9.5 (1Q)
- new net MOTOR1_U: R132.1
- new net MOTOR1_U_SHUNT_M: R162.1
- new net MOTOR1_U_SHUNT_P: R161.1
- new net MOTOR1_V: R134.1
- new net MOTOR1_V_SHUNT_M: R164.1
- new net MOTOR1_V_SHUNT_P: R163.1
- new net MOTOR1_W: R136.1
- new net MOTOR1_W_SHUNT_M: R166.1
- new net MOTOR1_W_SHUNT_P: R165.1
- new net MOTOR2_DIR: IC9.9 (2Q)
- new net MOTOR2_U: R129.1
- new net MOTOR2_V: R130.1
- new net MOTOR2_W: R131.1
- new net ZC_UV1_1: R126.2
- new net ZC_UV2_1: R156.2
- new net ZC_UW1_2: R127.2
- new net ZC_UW2_2: R157.2
- new net ZC_VW1_3: R128.2
- new net ZC_VW2_3: R158.2
- no-connect marks 0 -> 22
Other:
- note added: "MOTOR_CURRENT_SENSE"
- note added: "MOTOR_DIR_SENSE"
- note added: "MOTOR_SPEED_SENSE"
- note added: "MOTOR_ZEROCROSS_SENSE"

Commit message: 중간 저장
Parts:
- added C101, C102, C103: 39nF/16V, symbol Device:C_Small_US
- added R171, R172, R173, R183, R184, R185: 100/0.1w, Resistor_SMD:R_0402_1005Metric, symbol Device:R_Small_US
- added R174, R175, R177, R178, R180, R181: 10k/0.063w, Resistor_SMD:R_0402_1005Metric, symbol Device:R_Small_US
- added R176, R179, R182: 47k/0.125w, Resistor_SMD:R_0402_1005Metric, symbol Device:R_Small_US
- added R186, R187: 22/0.1w, Resistor_SMD:R_0402_1005Metric, symbol Device:R_Small_US
- added TP19, TP20, TP21, TP22, TP23, TP24, TP25, TP26, TP27, TP28, TP29, TP30, TP31: TestPoint, symbol Connector:TestPoint
- C96, C97, C98: value 0.1uF/16V -> 39nF/16V
- R167, R168, R169: value 10k/0.125w -> 47k/0.125w
Connections:
- net 3V3_MCU: no longer C91.1, C92.1, C95.1, IC4.14 (VCC), IC5.14 (VCC), IC6.8 (VCC)
- net 5V: now also C91.1, C92.1, C95.1, IC4.14 (VCC), IC5.14 (VCC), IC6.8 (VCC)
- net GND: now also C101.2, C102.2, C103.2
- net HALL1_3x_Sig: now also TP21.1
- net HALL1_6x_Pulse_Sig: now also U8.12 (+)
- net HALL2_3x_Sig: now also TP22.1
- net HALL2_6x_Pulse_Sig: now also U12.12 (+)
- net MOTOR2_U_SHUNT_M: now also R175.1
- net MOTOR2_U_SHUNT_P: now also R174.1
- net MOTOR2_V_SHUNT_M: now also R178.1
- net MOTOR2_V_SHUNT_P: now also R177.1
- net MOTOR2_W_SHUNT_M: now also R181.1
- net MOTOR2_W_SHUNT_P: now also R180.1
- net ZC_UV1_1: now also TP23.1
- net ZC_UW1_2: now also TP24.1
- net ZC_VW1_3: now also TP25.1
- net at R161.2, U7.3 (+): no longer C96.1
- net at U6.5 (+): now also R177.2
- net at U6.6 (-): now also R178.2, R179.1
- net at U6.7: now also R179.2, R184.1
- net at U8.13 (-): now also U8.14, R186.1
- net at R167.2, U7.1: now also R173.1
- net at R168.2, U7.7: now also R172.1
- net at R165.2, U7.10 (+): no longer C98.1
- net at U6.10 (+): now also R180.2
- net at U6.8: now also R182.2, R185.1
- net at U6.9 (-): now also R181.2, R182.1
- net at U12.13 (-): now also U12.14, R187.1
- net at R169.2, U7.8: now also R171.1
- net at U6.1: now also R176.2, R183.1
- net at U6.2 (-): now also R175.2, R176.1
- net at U6.3 (+): now also R174.2
- net at R163.2, U7.5 (+): no longer C97.1
- new net HALL1_6x_Pulse_Sig_Follow: R186.2, TP19.1
- new net HALL2_6x_Pulse_Sig_Follow: R187.2, TP20.1
- new net MOTOR1_U_SHUNT_ADC: C98.1, R173.2, TP26.1
- new net MOTOR1_V_SHUNT_ADC: C97.1, R172.2, TP27.1
- new net MOTOR1_W_SHUNT_ADC: C96.1, R171.2, TP28.1
- new net MOTOR2_V_SHUNT_ADC: C102.1, R184.2, TP29.1
- new net MOTOR2_W_SHUNT_ADC: C101.1, C103.1, R183.2, R185.2, TP30.1, TP31.1
- no-connect marks 22 -> 16
Other:
- note added: "fc = 1/(2pi*R/8C)"
- moved on the sheet: U12D, U6A, U6B, U6C, U8D

Commit message: 중간저장
Parts:
- added TP37: TP_ZC_UV2_1, symbol Connector:TestPoint
- added TP38: TP_ZC_UW2_2, symbol Connector:TestPoint
- added TP39: TP_ZC_VW2_3, symbol Connector:TestPoint
- added TP40: TP_MOTOR1_DIR, symbol Connector:TestPoint
- added TP41: TP_MOTOR2_DIR, symbol Connector:TestPoint
- TP19: value TestPoint -> TP_HALL1_6x
- TP20: value TestPoint -> TP_HALL2_6x
- TP21: value TestPoint -> TP_HALL1_3x_Sig
- TP22: value TestPoint -> TP_HALL2_3x_Sig
- TP23: value TestPoint -> TP_ZC_UV1_1
- TP24: value TestPoint -> TP_ZC_UW1_2
- TP25: value TestPoint -> TP_ZC_VW1_3
- TP26: value TestPoint -> TP_MOTOR1_U_SHUNT_ADC
- TP27: value TestPoint -> TP_MOTOR1_V_SHUNT_ADC
- TP28: value TestPoint -> TP_MOTOR1_W_SHUNT_ADC
- TP29: value TestPoint -> TP_MOTOR2_V_SHUNT_ADC
- TP30, TP31: value TestPoint -> TP_MOTOR2_W_SHUNT_ADC
Connections:
- net MOTOR1_DIR: now also TP40.1
- net MOTOR2_DIR: now also TP41.1
- net ZC_UV2_1: now also TP37.1
- net ZC_UW2_2: now also TP38.1
- net ZC_VW2_3: now also TP39.1

Commit message: 중간 저장
Parts:
- removed C101, C102, C103: 39nF/16V, symbol Device:C_Small_US
- removed C80, C84, C88, C89, C90, C94, C95: 0.1uF/16V, symbol Device:C_Small_US
- removed IC4: SN74HC266DRG4, SOIC127P600X175-14N, symbol SamacSys_Parts:SN74HC266DRG4
- removed R129, R130, R131, R160: 100k/0.063w, Resistor_SMD:R_0402_1005Metric, symbol Device:R_Small_US
- removed R153, R154, R155: 5k/0.063w, Resistor_SMD:R_0402_1005Metric, symbol Device:R_Small_US
- removed R156, R157, R158: 22/0.063w, Resistor_SMD:R_0402_1005Metric, symbol Device:R_Small_US
- removed R174, R175, R177, R178, R180, R181: 10k/0.063w, Resistor_SMD:R_0402_1005Metric, symbol Device:R_Small_US
- removed R176, R179, R182: 47k/0.125w, Resistor_SMD:R_0402_1005Metric, symbol Device:R_Small_US
- removed R183, R184, R185: 100/0.1w, Resistor_SMD:R_0402_1005Metric, symbol Device:R_Small_US
- removed R187: 22/0.1w, Resistor_SMD:R_0402_1005Metric, symbol Device:R_Small_US
- removed TP20: TP_HALL2_6x, symbol Connector:TestPoint
- removed TP22: TP_HALL2_3x_Sig, symbol Connector:TestPoint
- removed TP29: TP_MOTOR2_V_SHUNT_ADC, symbol Connector:TestPoint
- removed TP30, TP31: TP_MOTOR2_W_SHUNT_ADC, symbol Connector:TestPoint
- removed TP37: TP_ZC_UV2_1, symbol Connector:TestPoint
- removed TP38: TP_ZC_UW2_2, symbol Connector:TestPoint
- removed TP39: TP_ZC_VW2_3, symbol Connector:TestPoint
- removed TP41: TP_MOTOR2_DIR, symbol Connector:TestPoint
- removed U12: TLV9064, symbol Amplifier_Operational:TLV9064
- removed U6: TLV9064, PCM_4ms_Package_SSOP:TSSOP-14_4.4x5mm_P0.65mm, symbol Amplifier_Operational:TLV9064
- TP19: value TP_HALL1_6x -> TP_HALL_6x
- TP21: value TP_HALL1_3x_Sig -> TP_HALL_3x_Sig
- TP23: value TP_ZC_UV1_1 -> TP_ZC_UV_1
- TP24: value TP_ZC_UW1_2 -> TP_ZC_UW_2
- TP25: value TP_ZC_VW1_3 -> TP_ZC_VW_3
- TP26: value TP_MOTOR1_U_SHUNT_ADC -> TP_MOTOR_U_SHUNT_ADC
- TP27: value TP_MOTOR1_V_SHUNT_ADC -> TP_MOTOR_V_SHUNT_ADC
- TP28: value TP_MOTOR1_W_SHUNT_ADC -> TP_MOTOR_W_SHUNT_ADC
Connections:
- net 5V: no longer IC9.10 (2~{PRE}), IC9.13 (2~{CLR})
- net HALL1_3x_Late_Sig renamed HALL_3x_Late_Sig
- net HALL1_3x_Sig renamed HALL_3x_Sig
- net HALL1_6x_Pulse_Sig renamed HALL_6x_Pulse_Sig
- net HALL1_6x_Pulse_Sig_Follow renamed HALL_6x_Pulse_Sig_Follow
- net HALL1_A renamed HALL_A
- net HALL1_B renamed HALL_B
- net HALL1_C renamed HALL_C
- net HALL2_3x_Late_Sig: no longer names the net of IC6.5 (2Y)
- net HALL2_A: no longer names the net of IC9.12 (2D)
- net HALL2_B: no longer names the net of IC9.11 (2CLK)
- net MOTOR1_DIR renamed MOTOR_DIR
- net MOTOR1_U renamed MOTOR_U
- net MOTOR1_U_SHUNT_ADC renamed MOTOR_U_SHUNT_ADC
- net MOTOR1_U_SHUNT_M renamed MOTOR_U_SHUNT_M
- net MOTOR1_U_SHUNT_P renamed MOTOR_U_SHUNT_P
- net MOTOR1_V renamed MOTOR_V
- net MOTOR1_V_SHUNT_ADC renamed MOTOR_V_SHUNT_ADC
- net MOTOR1_V_SHUNT_M renamed MOTOR_V_SHUNT_M
- net MOTOR1_V_SHUNT_P renamed MOTOR_V_SHUNT_P
- net MOTOR1_W renamed MOTOR_W
- net MOTOR1_W_SHUNT_ADC renamed MOTOR_W_SHUNT_ADC
- net MOTOR1_W_SHUNT_M renamed MOTOR_W_SHUNT_M
- net MOTOR1_W_SHUNT_P renamed MOTOR_W_SHUNT_P
- net MOTOR2_DIR: no longer names the net of IC9.9 (2Q)
- net ZC_UV1_1 renamed ZC_UV_1
- net ZC_UW1_2 renamed ZC_UW_2
- net ZC_VW1_3 renamed ZC_VW_3
- no-connect marks 16 -> 17
Other:
- moved on the sheet: C93

Commit message: 중간 저장
Parts:
- removed IC5: SN74HC266DRG4, SOIC127P600X175-14N, symbol SamacSys_Parts:SN74HC266DRG4
- removed IC6: SN74LVC3G17DCTRG4, SOP65P400X130-8N, symbol SamacSys_Parts:SN74LVC3G17DCTRG4
- removed R186: 22/0.1w, Resistor_SMD:R_0402_1005Metric, symbol Device:R_Small_US
- removed TP19: TP_HALL_6x, symbol Connector:TestPoint
- added IC4: SN74HCS266QDRQ1, SOIC127P600X175-14N, symbol SamacSys_Parts:SN74HCS266QDRQ1
- added IC5: SN74LVC3G17DCURG4, SOP50P310X90-8N, symbol SamacSys_Parts:SN74LVC3G17DCURG4
- added R130, R131, R153: 10k/0.063w, Resistor_SMD:R_0402_1005Metric, symbol Device:R_Small_US
Connections:
- net 3V3_MCU: now also R153.2
- net 5V: now also IC4.14 (VCC), IC5.8 (VCC), R130.2, R131.2
- net GND: now also IC4.7 (GND), IC5.4 (GND)
- net HALL_3x_Late_Sig: now also IC4.9 (3B), IC5.7 (1Y)
- net HALL_3x_Sig: now also IC4.4 (2Y), IC4.8 (3A), R131.1
- net HALL_6x_Pulse_Sig: now also IC4.10 (3Y), R153.1; no longer U8.12 (+)
- net HALL_A: now also IC4.1 (1A)
- net HALL_B: now also IC4.2 (1B)
- net HALL_C: now also IC4.6 (2B)
- net at C93.1, R159.2: now also IC5.1 (1A)
- net at U8.13 (-): no longer U8.14
- new net: IC4.3 (1Y), IC4.5 (2A), R130.1
- no-connect marks 17 -> 20
Other:
- moved on the sheet: C82, C91, U8D

Commit message: 핀 배치 완료
Parts:
- added C95: 0.22uF/50V, symbol Device:C_Small_US
- added R113: 10k/0.063w, Resistor_SMD:R_0402_1005Metric, symbol Device:R_Small_US
- C81, C82, C85, C86, C87, C91, C92, C93: value 0.1uF/16V -> 0.1uF/50V
- C96, C97, C98: value 39nF/16V -> 39nF/50V
Connections:
- net 5V: now also R113.2; no longer IC9.1 (~{1CLR})
- net GND: now also C95.2
- new net: C95.1, IC9.1 (~{1CLR}), R113.1
Other:
- moved on the sheet: C82, IC9, TP40

Commit message: 중간 저장
Parts:
- C112: renamed from C95; footprint (none) -> Capacitor_SMD:C_0603_1608Metric
- C113: renamed from C93; footprint (none) -> Capacitor_SMD:C_0603_1608Metric
- C114: renamed from C91; footprint (none) -> Capacitor_SMD:C_0603_1608Metric
- C115: renamed from C92; footprint (none) -> Capacitor_SMD:C_0603_1608Metric
- C116: renamed from C82; footprint (none) -> Capacitor_SMD:C_0603_1608Metric
- C117: renamed from C81; footprint (none) -> Capacitor_SMD:C_0603_1608Metric
- C118: renamed from C83; value 0.1uF/16V -> 0.1uF/50V; footprint (none) -> Capacitor_SMD:C_0603_1608Metric
- C119: renamed from C85; footprint (none) -> Capacitor_SMD:C_0603_1608Metric
- C120: renamed from C86; footprint (none) -> Capacitor_SMD:C_0603_1608Metric
- C121: renamed from C87; footprint (none) -> Capacitor_SMD:C_0603_1608Metric
- C122: renamed from C98; footprint (none) -> Capacitor_SMD:C_0402_1005Metric
- C123: renamed from C97; footprint (none) -> Capacitor_SMD:C_0402_1005Metric
- C124: renamed from C96; footprint (none) -> Capacitor_SMD:C_0402_1005Metric
- TP18: renamed from TP21; footprint (none) -> TestPoint:TestPoint_Pad_D1.5mm
- TP19: renamed from TP40; footprint (none) -> TestPoint:TestPoint_Pad_D1.5mm
- TP20: renamed from TP26; footprint (none) -> TestPoint:TestPoint_Pad_D1.5mm
- TP21: renamed from TP27; footprint (none) -> TestPoint:TestPoint_Pad_D1.5mm
- TP22: renamed from TP28; footprint (none) -> TestPoint:TestPoint_Pad_D1.5mm
- TP23, TP24, TP25: footprint (none) -> TestPoint:TestPoint_Pad_D1.5mm
- renumbered IC4 to IC7, IC9 to IC8, IC5 to IC9, R131 to R171, R113 to R172, R130 to R173, R159 to R174, R153 to R175, R161 to R176, R162 to R177, R163 to R178, R164 to R179, R165 to R180, R166 to R181, R132 to R182, R134 to R183, R136 to R184, R167 to R185, R168 to R186, R169 to R187, R133 to R188, R135 to R189, R137 to R190, R173 to R191, R172 to R192, R171 to R193, R126 to R194, R127 to R195, R128 to R196, U8 to U10, U7 to U9

Commit message: 중간 저장
Parts:
- IC7: footprint SOIC127P600X175-14N -> SamacSys_Parts:SOIC127P600X175-14N
- IC8: footprint SOP65P640X120-14N -> SamacSys_Parts:SOP65P640X120-14N
- IC9: footprint SOP50P310X90-8N -> SamacSys_Parts:SOP50P310X90-8N
Changed lines of the file:
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@@
 			)
 		)
-		(property "Footprint" "SOIC127P600X175-14N"
+		(property "Footprint" "SamacSys_Parts:SOIC127P600X175-14N"
 			(at 58.42 44.45 0)
 			(effects
@@
 			)
 		)
-		(property "Footprint" "SOP65P640X120-14N"
+		(property "Footprint" "SamacSys_Parts:SOP65P640X120-14N"
 			(at 83.82 157.48 0)
 			(effects
@@
 			)
 		)
-		(property "Footprint" "SOP50P310X90-8N"
+		(property "Footprint" "SamacSys_Parts:SOP50P310X90-8N"
 			(at 80.01 95.25 0)
 			(effects
