File: 1.hardware/motor_control.kicad_sch (KiCad schematic)
At the start: 19 parts, among them IC1 UCC27712QDRQ1, J10 MOTOR_1_UVW, J11 MOTOR_1_HALL_SENSOR, Q10 STL130N6F7, Q2 STL130N6F7, Q3 STL130N6F7, Q4 STL130N6F7, Q8 STL130N6F7, Q9 STL130N6F7

Commit message: 중간저장
Parts:
- added C104, C105: 33pF/50V, symbol Device:C_Small_US
- added C106, C108: 0.1uF/50V, symbol Device:C_Small_US
- added C107: 1uF/25V, symbol Device:C_Small_US
- added D14, D15, D16: D_Schottky_Generic, symbol PCM_Diode_Schottky_AKL:D_Schottky_Generic
- added D17: SS14, PCM_Diode_SMD_AKL:D_SMA, symbol PCM_Diode_Schottky_AKL:SS14
- added R188, R189: 49.9/0.1w, symbol Device:R_Small_US
- added R190, R191: 3.3/0.125w, symbol Device:R_Small_US
- added R192, R193: 2.2/0.125w, symbol Device:R_Small_US
- added R194, R195: R_Small_US, symbol Device:R_Small_US
- TP13: value TP_HA2 -> TP_HALL1_A
- TP14: value TP_HB2 -> TP_HALL1_B
- TP15: value TP_HC2 -> TP_HALL1_C
- TP16: value TP_U2 -> TP_MOTOR1_U
- TP17: value TP_V2 -> TP_MOTOR1_V
- TP18: value TP_W2 -> TP_MOTOR1_W
Connections:
- net 12V: now also IC1.3 (VDD), C106.1, R194.2
- net GND: now also C104.2, C105.2, C106.2
- net GNDPWR: now also IC1.4 (COM), Q3.1 (S_1), Q3.2 (S_2), Q3.3 (S_3)
- net MOTOR1_U: now also IC1.6 (HS), Q2.1 (S_1), Q2.2 (S_2), Q2.3 (S_3), Q3.5 (D_1), Q3.6 (D_2), Q3.7 (D_3), Q3.8 (D_4), Q3.9 (D_5), C107.2, C108.2, R195.2
- net PWR_INPUT(12V~48V): now also Q2.5 (D_1), Q2.6 (D_2), Q2.7 (D_3), Q2.8 (D_4), Q2.9 (D_5)
- net at IC1.1 (LI): now also C105.1, R188.1
- net at IC1.2 (HI): now also C104.1, R189.1
- net at IC1.5 (LO): now also R191.2, R193.2
- net at IC1.7 (HO): now also R190.2, R192.2
- net at IC1.8 (HB): now also C107.1, C108.1, D16.1 (K)
- net at Q2.4 (G): now also D14.2 (A), R190.1, R195.1
- net at Q3.4 (G): now also D15.2 (A), R191.1
- new net: D16.2 (A), R194.1
- new net: D15.1 (K), R193.1
- new net: D14.1 (K), R192.1
- new net MOTOR1_U_HI: R189.2
- new net MOTOR1_U_LI: R188.2
Other:
- note added: "1/(2*PI*R*C) = 100mhz"
- moved on the sheet: IC1, Q2, Q3

Commit message: 중간 저장
Parts:
- removed C107: 1uF/25V, symbol Device:C_Small_US
- removed D16: D_Schottky_Generic, symbol PCM_Diode_Schottky_AKL:D_Schottky_Generic
- removed D17: SS14, PCM_Diode_SMD_AKL:D_SMA, symbol PCM_Diode_Schottky_AKL:SS14
- added C109: 1uF/25V, symbol Device:C_Polarized_Small_US
- added D17: SS58c, Diode_SMD:D_SMC, symbol PCM_Diode_Schottky_AKL:D_Schottky_Generic
- added R196: 10/0.125w, symbol Device:R_Small_US
- C106: value 0.1uF/50V -> 10uF/25V
- R194: value R_Small_US -> 10/0.125w
Connections:
- net 12V: now also R196.1; no longer C106.1, IC1.3 (VDD)
- net GNDPWR: no longer Q3.1 (S_1), Q3.2 (S_2), Q3.3 (S_3)
- net MOTOR1_U: now also C109.2
- net at C108.1, IC1.8 (HB): now also C109.1, D17.1 (K)
- net at R194.1: now also D17.2 (A)
- net at R97.1: now also Q3.1 (S_1), Q3.2 (S_2), Q3.3 (S_3)
- new net: C106.1, IC1.3 (VDD), R196.2
Other:
- moved on the sheet: R97

Commit message: 중간 저장
Parts:
- removed C109: 1uF/25V, symbol Device:C_Polarized_Small_US
- removed D14, D15: D_Schottky_Generic, symbol PCM_Diode_Schottky_AKL:D_Schottky_Generic
- removed D17: SS58c, Diode_SMD:D_SMC, symbol PCM_Diode_Schottky_AKL:D_Schottky_Generic
- added C107, C113, C114, C121, C122: 10uF/25V, symbol Device:C_Small_US
- added C109, C110, C116, C118, C119, C124, C126, C127: 0.22uF/50V, symbol Device:C_Small_US
- added C111, C112, C120: 47uF/50V, symbol Device:C_Polarized_Small_US
- added C115, C117, C123, C125: 33pF/50V, symbol Device:C_Small_US
- added D14, D16, D18, D19, D21, D22: MBRM130LT1G, MBRM130LT1G, symbol SamacSys_Parts:MBRM130LT1G
- added D15, D17, D20: MURA160T3G, DIOM5226X220N, symbol SamacSys_Parts:MURA160T3G
- added IC11, IC7: UCC27712QDRQ1, SOIC127P600X175-8N, symbol SamacSys_Parts:UCC27712QDRQ1
- added R197, R206, R207, R216, R217: 5.1k/0.1w, symbol Device:R_Small_US
- added R198, R202, R208, R212: 2.2/0.25w, symbol Device:R_Small_US
- added R199, R200, R209, R210: 49.9/0.1w, symbol Device:R_Small_US
- added R201, R203, R211, R213: 2.2/0.125w, symbol Device:R_Small_US
- added R204, R205, R214, R215: 3.3/0.125w, symbol Device:R_Small_US
- C108: value 0.1uF/50V -> 0.22uF/50V
- J10: value MOTOR_1_UVW -> MOTOR_UVW
- J11: value MOTOR_1_HALL_SENSOR -> MOTOR_HALL_SENSOR
- R192: value 2.2/0.125w -> 2.2/0.25w
- R194: value 10/0.125w -> 2.2/0.125w
- R195: value R_Small_US -> 5.1k/0.1w
- R196: value 10/0.125w -> 2.2/0.25w
- TP13: value TP_HALL1_A -> TP_HALL_A
- TP14: value TP_HALL1_B -> TP_HALL_B
- TP15: value TP_HALL1_C -> TP_HALL_C
- TP16: value TP_MOTOR1_U -> TP_MOTOR_U
- TP17: value TP_MOTOR1_V -> TP_MOTOR_V
- TP18: value TP_MOTOR1_W -> TP_MOTOR_W
Connections:
- net MOTOR1_V is gone; now on net MOTOR_V: J10.2 (Pin_2), TP17.1
- net MOTOR1_W is gone; now on net MOTOR_W: J10.3 (Pin_3), TP18.1
- net 12V: now also R196.2, R198.2, R208.2; no longer R194.2, R196.1
- net GND: now also C107.2, C110.2, C111.2, C112.2, C113.2, C114.2, C115.2, C116.2, C117.2, C120.2, C121.2, C122.2, C123.2, C124.2, C125.2
- net GNDPWR: now also IC11.4 (COM), IC7.4 (COM), R197.2, R207.2, R217.2
- net PWR_INPUT(12V~48V): now also Q4.5 (D_1), Q4.6 (D_2), Q4.7 (D_3), Q4.8 (D_4), Q4.9 (D_5), Q9.5 (D_1), Q9.6 (D_2), Q9.7 (D_3), Q9.8 (D_4), Q9.9 (D_5)
- net at Q8.1 (S_1): now also Q8.2 (S_2), Q8.3 (S_3), R1.1
- net at Q8.4 (G): now also D19.2, R205.1, R207.1
- net MOTOR_V: now reaches Q8.5 (D_1)
- net MOTOR_V: now also Q4.1 (S_1), Q4.2 (S_2), Q4.3 (S_3), Q8.6 (D_2), Q8.7 (D_3), Q8.8 (D_4), Q8.9 (D_5), C118.2, C119.2, IC7.6 (HS), R206.2
- net at C106.1, IC1.3 (VDD): now also R194.2, R196.1, C107.1, C110.1, C111.1; no longer R196.2
- net at C108.1, IC1.8 (HB): now also C109.1, D15.1
- net at Q2.4 (G), R190.1, R195.1: now also D14.2
- net at R98.1: now also Q10.1 (S_1), Q10.2 (S_2), Q10.3 (S_3)
- net at R193.1: now also D16.1
- net MOTOR_W: now reaches Q9.1 (S_1)
- net MOTOR_W: now also Q10.5 (D_1), Q10.6 (D_2), Q10.7 (D_3), Q10.8 (D_4), Q10.9 (D_5), Q9.2 (S_2), Q9.3 (S_3), C126.2, C127.2, IC11.6 (HS), R216.2
- net at Q9.4 (G): now also D21.2, R214.1, R216.1
- net at R194.1: now also D15.2
- net at Q3.4 (G), R191.1: now also D16.2, R197.1
- net at R192.1: now also D14.1
- net at Q4.4 (G): now also D18.2, R204.1, R206.1
- net at Q10.4 (G): now also D22.2, R215.1, R217.1
- net HALL1_A renamed HALL_A
- net HALL1_B renamed HALL_B
- net HALL1_C renamed HALL_C
- net MOTOR1_U renamed MOTOR_U
- net MOTOR_U: now also C109.2
- net MOTOR1_U_HI renamed MOTOR_U_HI
- net MOTOR1_U_LI renamed MOTOR_U_LI
- net MOTOR1_U_SHUNT_M renamed MOTOR_U_SHUNT_M
- net MOTOR1_U_SHUNT_P renamed MOTOR_U_SHUNT_P
- net MOTOR1_V_SHUNT_M renamed MOTOR_V_SHUNT_M
- net MOTOR1_V_SHUNT_P renamed MOTOR_V_SHUNT_P
- net MOTOR1_W_SHUNT_M renamed MOTOR_W_SHUNT_M
- net MOTOR1_W_SHUNT_P renamed MOTOR_W_SHUNT_P
- new net: D18.1, R202.1
- new net: IC7.5 (LO), R203.2, R205.2
- new net: C117.1, IC7.1 (LI), R199.1
- new net: C126.1, C127.1, D20.1, IC11.8 (HB)
- new net: C118.1, C119.1, D17.1, IC7.8 (HB)
- new net: D17.2, R201.1
- new net: IC11.5 (LO), R213.2, R215.2
- new net: D20.2, R211.1
- new net: C120.1, C121.1, C122.1, C124.1, IC11.3 (VDD), R208.1, R211.2
- new net: C123.1, IC11.2 (HI), R210.1
- new net: D22.1, R213.1
- new net: D21.1, R212.1
- new net: C112.1, C113.1, C114.1, C116.1, IC7.3 (VDD), R198.1, R201.2
- new net: D19.1, R203.1
- new net: IC11.7 (HO), R212.2, R214.2
- new net: C115.1, IC7.2 (HI), R200.1
- new net: IC7.7 (HO), R202.2, R204.2
- new net: C125.1, IC11.1 (LI), R209.1
- new net MOTOR_V_HI: R200.2
- new net MOTOR_V_LI: R199.2
- new net MOTOR_W_HI: R210.2
- new net MOTOR_W_LI: R209.2
Other:
- moved on the sheet: C104, C105, C106, C108, IC1, Q2, Q3, R1, R188, R189, R190, R191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

Commit message: 중간 저장
Parts:
- added C89, C90, C94: 22uF/100V, symbol Device:C_Polarized_Small_US
Connections:
- net GNDPWR: now also C89.2, C90.2, C94.2
- net PWR_INPUT(12V~48V): now also C89.1, C90.1, C94.1

Commit message: 중간 저장
Parts:
- C100: renamed from C105; footprint (none) -> Capacitor_SMD:C_0402_1005Metric
- C101: renamed from C117; footprint (none) -> Capacitor_SMD:C_0402_1005Metric
- C102: renamed from C125; footprint (none) -> Capacitor_SMD:C_0402_1005Metric
- C103: renamed from C109; footprint (none) -> Capacitor_SMD:C_0603_1608Metric
- C104: renamed from C118; footprint (none) -> Capacitor_SMD:C_0603_1608Metric
- C105: renamed from C126; footprint (none) -> Capacitor_SMD:C_0603_1608Metric
- C106: renamed from C108; footprint (none) -> Capacitor_SMD:C_0603_1608Metric
- C107: renamed from C119; footprint (none) -> Capacitor_SMD:C_0603_1608Metric
- C108: renamed from C127; footprint (none) -> Capacitor_SMD:C_0603_1608Metric
- C109: renamed from C89; footprint (none) -> Capacitor_SMD:C_Elec_8x10.2
- C110: renamed from C90; footprint (none) -> Capacitor_SMD:C_Elec_8x10.2
- C111: renamed from C94; footprint (none) -> Capacitor_SMD:C_Elec_8x10.2
- C84: renamed from C17; footprint (none) -> Capacitor_SMD:C_0603_1608Metric
- C85: renamed from C111; footprint (none) -> Capacitor_SMD:C_Elec_6.3x7.7
- C86: renamed from C112; footprint (none) -> Capacitor_SMD:C_Elec_6.3x7.7
- C87: renamed from C120; footprint (none) -> Capacitor_SMD:C_Elec_6.3x7.7
- C88: renamed from C106; footprint (none) -> Capacitor_SMD:C_Elec_4x5.4
- C89: renamed from C113; footprint (none) -> Capacitor_SMD:C_Elec_4x5.4
- C90: renamed from C121; footprint (none) -> Capacitor_SMD:C_Elec_4x5.4
- C91: renamed from C107; footprint (none) -> Capacitor_SMD:C_Elec_4x5.4
- C92: renamed from C114; footprint (none) -> Capacitor_SMD:C_Elec_4x5.4
- C93: renamed from C122; footprint (none) -> Capacitor_SMD:C_Elec_4x5.4
- C94: renamed from C104; footprint (none) -> Capacitor_SMD:C_0402_1005Metric
- C95: renamed from C115; footprint (none) -> Capacitor_SMD:C_0402_1005Metric
- C96: renamed from C123; footprint (none) -> Capacitor_SMD:C_0402_1005Metric
- C97: renamed from C110; footprint (none) -> Capacitor_SMD:C_0603_1608Metric
- C98: renamed from C116; footprint (none) -> Capacitor_SMD:C_0603_1608Metric
- C99: renamed from C124; footprint (none) -> Capacitor_SMD:C_0603_1608Metric
- R138: renamed from R196; footprint (none) -> Resistor_SMD:R_1206_3216Metric
- R139: renamed from R198; footprint (none) -> Resistor_SMD:R_1206_3216Metric
- R140: renamed from R208; footprint (none) -> Resistor_SMD:R_1206_3216Metric
- R141: renamed from R188; footprint (none) -> Resistor_SMD:R_0603_1608Metric
- R142: renamed from R189; footprint (none) -> Resistor_SMD:R_0603_1608Metric
- R143: renamed from R199; footprint (none) -> Resistor_SMD:R_0603_1608Metric
- R144: renamed from R200; footprint (none) -> Resistor_SMD:R_0603_1608Metric
- R145: renamed from R209; footprint (none) -> Resistor_SMD:R_0603_1608Metric
- R146: renamed from R210; footprint (none) -> Resistor_SMD:R_0603_1608Metric
- R147: renamed from R194; footprint (none) -> Resistor_SMD:R_0805_2012Metric
- R148: renamed from R201; footprint (none) -> Resistor_SMD:R_0805_2012Metric
- R149: renamed from R211; footprint (none) -> Resistor_SMD:R_0805_2012Metric
- R150: renamed from R192; footprint (none) -> Resistor_SMD:R_1206_3216Metric
- R151: renamed from R193; footprint (none) -> Resistor_SMD:R_0805_2012Metric
- R152: renamed from R202; footprint (none) -> Resistor_SMD:R_1206_3216Metric
- R153: renamed from R203; footprint (none) -> Resistor_SMD:R_0805_2012Metric
- R154: renamed from R212; footprint (none) -> Resistor_SMD:R_1206_3216Metric
- R155: renamed from R213; footprint (none) -> Resistor_SMD:R_0805_2012Metric
- R156: renamed from R190; footprint (none) -> Resistor_SMD:R_0805_2012Metric
- R157: renamed from R191; footprint (none) -> Resistor_SMD:R_0805_2012Metric
- R158: renamed from R204; footprint (none) -> Resistor_SMD:R_0805_2012Metric
- R159: renamed from R205; footprint (none) -> Resistor_SMD:R_0805_2012Metric
- R160: renamed from R214; footprint (none) -> Resistor_SMD:R_0805_2012Metric
- R161: renamed from R215; footprint (none) -> Resistor_SMD:R_0805_2012Metric
- R162: renamed from R195; footprint (none) -> Resistor_SMD:R_0603_1608Metric
- R163: renamed from R197; footprint (none) -> Resistor_SMD:R_0603_1608Metric
- R164: renamed from R206; footprint (none) -> Resistor_SMD:R_0603_1608Metric
- R165: renamed from R207; footprint (none) -> Resistor_SMD:R_0603_1608Metric
- R166: renamed from R216; footprint (none) -> Resistor_SMD:R_0603_1608Metric
- R167: renamed from R217; footprint (none) -> Resistor_SMD:R_0603_1608Metric
- R168: renamed from R97; footprint (none) -> Resistor_SMD:R_2512_6332Metric
- R169: renamed from R1; footprint (none) -> Resistor_SMD:R_2512_6332Metric
- R170: renamed from R98; footprint (none) -> Resistor_SMD:R_2512_6332Metric
- TP12: renamed from TP16; footprint (none) -> TestPoint:TestPoint_Pad_D1.5mm
- TP13: footprint (none) -> TestPoint:TestPoint_Pad_D1.5mm
- TP14: renamed from TP17; footprint (none) -> TestPoint:TestPoint_Pad_D1.5mm
- TP15: renamed from TP14; footprint (none) -> TestPoint:TestPoint_Pad_D1.5mm
- TP16: renamed from TP18; footprint (none) -> TestPoint:TestPoint_Pad_D1.5mm
- TP17: renamed from TP15; footprint (none) -> TestPoint:TestPoint_Pad_D1.5mm
- renumbered D15 to D14, D17 to D15, D20 to D16, D14 to D17, D16 to D18, D18 to D19, D19 to D20, IC1 to IC4, IC7 to IC5, IC11 to IC6, J10 to J13, J11 to J14, Q9 to Q10, Q10 to Q11, Q2 to Q6, Q3 to Q7, Q4 to Q8, Q8 to Q9

Commit message: 중간 저장
Parts:
- IC4, IC5, IC6: footprint SOIC127P600X175-8N -> SamacSys_Parts:SOIC127P600X175-8N
- Q10, Q11, Q6, Q7, Q8, Q9: footprint FERD20U50DJFTR -> SamacSys_Parts:FERD20U50DJFTR
- R147, R148, R149: value 2.2/0.125w -> 2.2/0.25w
Changed lines of the file:
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@@
 			)
 		)
-		(property "Footprint" "SOIC127P600X175-8N"
+		(property "Footprint" "SamacSys_Parts:SOIC127P600X175-8N"
 			(at 190.5 45.72 0)
 			(effects
@@
 			)
 		)
-		(property "Footprint" "FERD20U50DJFTR"
+		(property "Footprint" "SamacSys_Parts:FERD20U50DJFTR"
 			(at 261.62 24.13 0)
 			(effects
@@
 			)
 		)
-		(property "Value" "2.2/0.125w"
+		(property "Value" "2.2/0.25w"
 			(at 172.72 181.102 90)
 			(effects
@@
 			)
 		)
-		(property "Footprint" "FERD20U50DJFTR"
+		(property "Footprint" "SamacSys_Parts:FERD20U50DJFTR"
 			(at 262.89 177.8 0)
 			(effects
@@
 			)
 		)
-		(property "Value" "2.2/0.125w"
+		(property "Value" "2.2/0.25w"
 			(at 172.72 104.902 90)
 			(effects
@@
 			)
 		)
-		(property "Footprint" "FERD20U50DJFTR"
+		(property "Footprint" "SamacSys_Parts:FERD20U50DJFTR"
 			(at 262.89 207.01 0)
 			(effects
@@
 			)
 		)
-		(property "Footprint" "FERD20U50DJFTR"
+		(property "Footprint" "SamacSys_Parts:FERD20U50DJFTR"
 			(at 262.89 130.81 0)
 			(effects
@@
 			)
 		)
-		(property "Footprint" "FERD20U50DJFTR"
+		(property "Footprint" "SamacSys_Parts:FERD20U50DJFTR"
 			(at 262.89 101.6 0)
 			(effects
@@
 			)
 		)
-		(property "Footprint" "FERD20U50DJFTR"
+		(property "Footprint" "SamacSys_Parts:FERD20U50DJFTR"
 			(at 261.62 53.34 0)
 			(effects
@@
 			)
 		)
-		(property "Value" "2.2/0.125w"
+		(property "Value" "2.2/0.25w"
 			(at 171.45 27.432 90)
 			(effects
@@
 			)
 		)
-		(property "Footprint" "SOIC127P600X175-8N"
+		(property "Footprint" "SamacSys_Parts:SOIC127P600X175-8N"
 			(at 191.77 199.39 0)
 			(effects
@@
 			)
 		)
-		(property "Footprint" "SOIC127P600X175-8N"
+		(property "Footprint" "SamacSys_Parts:SOIC127P600X175-8N"
 			(at 191.77 123.19 0)
 			(effects
